File: microcontroller.sch (KiCad schematic (older format))
At the start: 0 parts

Commit message: Micro and Environment Schematic Copy
Copied over the microcontroller and environment sheets from smart-regulator project. Also modified the power section.
Parts:
- added C4: C_10uF, Capacitors_SMD:C_0603_HandSoldering, symbol C_10uF
- added C6: C_1uF, Capacitors_SMD:C_0603_HandSoldering, symbol C_1uF
- added J1: Conn_02x05_Odd_Even, Pin_Headers:Pin_Header_Straight_2x05_Pitch2.54mm, symbol Conn_02x05_Odd_Even
- added R10, R6, R9: R_10k, Resistors_SMD:R_0603_HandSoldering, symbol R_10k
- added U1: ESP-WROOM-32, smart-regulator:ESP-WROOM-32, symbol ESP-WROOM-32
Connections:
- net labels added: 3V3, EN, FACTORY, GND, IO2, Microcontroller, PANEL_SW, POWER_EN, PROG, RXD, SCL, SDA, TXD, V_USB
- wire segments 0 -> 39
Other:
- note added: "Bypass CAPs"

Commit message: Power Schematic Update
Test commit and minior power schematic update.
Connections:
- net labels added: 5V
- net labels removed: V_USB
Changed lines of the file:
@@
 EESchema Schematic File Version 2
 LIBS:device
-LIBS:smart-regulator-cache
 LIBS:open-dash-daughterboard-cache
 EELAYER 25 0
@@
 TXD
 Text GLabel 8800 3650 2    60   Input ~ 0
-V_USB
+5V
 $Comp
 L GND #PWR013

Commit message: Backup Before SEPIC Design
Parts:
- U1: footprint smart-regulator:ESP-WROOM-32 -> open-automation:ESP-WROOM-32
Changed lines of the file:
@@
 F 0 "U1" H 6325 2350 60  0000 C CNN
 F 1 "ESP-WROOM-32" H 5775 4250 60  0000 C CNN
-F 2 "smart-regulator:ESP-WROOM-32" H 5425 4050 60  0001 C CNN
+F 2 "open-automation:ESP-WROOM-32" H 5425 4050 60  0001 C CNN
 F 3 "https://www.espressif.com/sites/default/files/documentation/esp_wroom_32_datasheet_en.pdf" H 5425 4050 60  0001 C CNN
 	1    5775 3450

Commit message: Updated Power Schematic
Power Schematic Updated for 3.3V, 5V, and 8V Buck Regulators. All regulator parts have correct footprints and selected components.

Prelim orgainization of PCB - grouped parts by section.
Parts:
- renumbered C4 to C7, C6 to C8, R9 to R6, R10 to R7, R6 to R8, U1 to U4
Connections:
- net labels added: EN_5V_POWER, EN_8V_POWER
- wire segments 39 -> 41
Changed lines of the file:
@@
 $EndDescr
 $Comp
-L GND #PWR011
+L GND #PWR015
 U 1 1 59097974
 P 4825 2750
-F 0 "#PWR011" H 4825 2500 50  0001 C CNN
+F 0 "#PWR015" H 4825 2500 50  0001 C CNN
 F 1 "GND" H 4825 2600 50  0000 C CNN
 F 2 "" H 4825 2750 50  0000 C CNN
@@
 IO2
 $Comp
-L ESP-WROOM-32 U1
+L ESP-WROOM-32 U4
 U 1 1 590979AF
 P 5775 3450
-F 0 "U1" H 6325 2350 60  0000 C CNN
+F 0 "U4" H 6325 2350 60  0000 C CNN
 F 1 "ESP-WROOM-32" H 5775 4250 60  0000 C CNN
 F 2 "open-automation:ESP-WROOM-32" H 5425 4050 60  0001 C CNN
@@
 SDA
 $Comp
-L GND #PWR012
+L GND #PWR016
 U 1 1 590979B0
 P 8150 3500
-F 0 "#PWR012" H 8150 3250 50  0001 C CNN
+F 0 "#PWR016" H 8150 3250 50  0001 C CNN
 F 1 "GND" H 8150 3350 50  0000 C CNN
 F 2 "" H 8150 3500 50  0000 C CNN
@@
 5V
 $Comp
-L GND #PWR013
+L GND #PWR017
 U 1 1 590979B2
 P 8750 3500
-F 0 "#PWR013" H 8750 3250 50  0001 C CNN
+F 0 "#PWR017" H 8750 3250 50  0001 C CNN
 F 1 "GND" H 8750 3350 50  0000 C CNN
 F 2 "" H 8750 3500 50  0000 C CNN
@@
 Microcontroller
 $Comp
-L C_1uF C6
+L C_1uF C8
 U 1 1 59C55B03
 P 2825 3775
-F 0 "C6" H 2825 3875 50  0000 L CNN
+F 0 "C8" H 2825 3875 50  0000 L CNN
 F 1 "C_1uF" H 2575 3675 50  0000 L CNN
 F 2 "Capacitors_SMD:C_0603_HandSoldering" H 2925 4075 50  0001 C CNN
@@
 $EndComp
 $Comp
-L GND #PWR014
+L GND #PWR018
 U 1 1 59C55B05
 P 2625 4025
-F 0 "#PWR014" H 2625 3775 50  0001 C CNN
+F 0 "#PWR018" H 2625 3775 50  0001 C CNN
 F 1 "GND" H 2625 3875 50  0000 C CNN
 F 2 "" H 2625 4025 50  0000 C CNN
@@
 	8100 3750 8200 3750
 $Comp
-L R_10k R6
+L R_10k R8
 U 1 1 59C609F8
 P 6400 4700
-F 0 "R6" V 6400 4700 50  0000 C CNN
+F 0 "R8" V 6400 4700 50  0000 C CNN
 F 1 "R_10k" V 6325 4700 50  0000 C CNN
 F 2 "Resistors_SMD:R_0603_HandSoldering" V 6330 4700 50  0001 C CNN
@@
 Connection ~ 6175 4700
 $Comp
-L GND #PWR015
+L GND #PWR019
 U 1 1 59C60A9D
 P 6600 4700
-F 0 "#PWR015" H 6600 4450 50  0001 C CNN
+F 0 "#PWR019" H 6600 4450 50  0001 C CNN
 F 1 "GND" H 6600 4550 50  0000 C CNN
 F 2 "" H 6600 4700 50  0000 C CNN
@@
 SDA
 $Comp
-L R_10k R10
+L R_10k R7
 U 1 1 59C83F25
 P 3450 3700
-F 0 "R10" V 3450 3700 50  0000 C CNN
+F 0 "R7" V 3450 3700 50  0000 C CNN
 F 1 "R_10k" H 3325 3850 50  0000 C CNN
 F 2 "Resistors_SMD:R_0603_HandSoldering" V 3380 3700 50  0001 C CNN
@@
 $EndComp
 $Comp
-L R_10k R9
+L R_10k R6
 U 1 1 59C83F7C
 P 3350 3700
-F 0 "R9" V 3350 3700 50  0000 C CNN
+F 0 "R6" V 3350 3700 50  0000 C CNN
 F 1 "R_10k" H 3475 3850 50  0000 C CNN
 F 2 "Resistors_SMD:R_0603_HandSoldering" V 3280 3700 50  0001 C CNN
@@
 3V3
 $Comp
-L C_10uF C4
+L C_10uF C7
 U 1 1 5A10664F
 P 2425 3775
-F 0 "C4" H 2450 3875 50  0000 L CNN
+F 0 "C7" H 2450 3875 50  0000 L CNN
 F 1 "C_10uF" H 2125 3675 50  0000 L CNN
 F 2 "Capacitors_SMD:C_0603_HandSoldering" H 2525 4075 50  0001 C CNN
@@
 Wire Notes Line
 	3000 4275 2075 4275
+Text GLabel 4850 5250 0    60   Input ~ 0
+EN_5V_POWER
+Text GLabel 4850 5400 0    60   Input ~ 0
+EN_8V_POWER
+Wire Wire Line
+	4850 5250 5150 5250
+Wire Wire Line
+	4850 5400 5150 5400
 $EndSCHEMATC

Commit message: Update Power Schematic and directed parts to open-automation library
Change 3.3V and 5V buck regulator to adjustable chip version.

Directed multiple parts from -cache.lib to open-automation.lib.
Parts:
- renumbered R6 to R10, R7 to R11, R8 to R12
Changed lines of the file:
@@
 EESchema Schematic File Version 2
 LIBS:device
+LIBS:open-automation
 LIBS:open-dash-daughterboard-cache
 EELAYER 25 0
@@
 $EndDescr
 $Comp
-L GND #PWR015
+L GND #PWR20
 U 1 1 59097974
 P 4825 2750
-F 0 "#PWR015" H 4825 2500 50  0001 C CNN
+F 0 "#PWR20" H 4825 2500 50  0001 C CNN
 F 1 "GND" H 4825 2600 50  0000 C CNN
 F 2 "" H 4825 2750 50  0000 C CNN
@@
 SDA
 $Comp
-L GND #PWR016
+L GND #PWR22
 U 1 1 590979B0
 P 8150 3500
-F 0 "#PWR016" H 8150 3250 50  0001 C CNN
+F 0 "#PWR22" H 8150 3250 50  0001 C CNN
 F 1 "GND" H 8150 3350 50  0000 C CNN
 F 2 "" H 8150 3500 50  0000 C CNN
@@
 5V
 $Comp
-L GND #PWR017
+L GND #PWR23
 U 1 1 590979B2
 P 8750 3500
-F 0 "#PWR017" H 8750 3250 50  0001 C CNN
+F 0 "#PWR23" H 8750 3250 50  0001 C CNN
 F 1 "GND" H 8750 3350 50  0000 C CNN
 F 2 "" H 8750 3500 50  0000 C CNN
@@
 $EndComp
 $Comp
-L GND #PWR018
+L GND #PWR19
 U 1 1 59C55B05
 P 2625 4025
-F 0 "#PWR018" H 2625 3775 50  0001 C CNN
+F 0 "#PWR19" H 2625 3775 50  0001 C CNN
 F 1 "GND" H 2625 3875 50  0000 C CNN
 F 2 "" H 2625 4025 50  0000 C CNN
@@
 	8100 3750 8200 3750
 $Comp
-L R_10k R8
+L R_10k R12
 U 1 1 59C609F8
 P 6400 4700
-F 0 "R8" V 6400 4700 50  0000 C CNN
+F 0 "R12" V 6400 4700 50  0000 C CNN
 F 1 "R_10k" V 6325 4700 50  0000 C CNN
 F 2 "Resistors_SMD:R_0603_HandSoldering" V 6330 4700 50  0001 C CNN
@@
 Connection ~ 6175 4700
 $Comp
-L GND #PWR019
+L GND #PWR21
 U 1 1 59C60A9D
 P 6600 4700
-F 0 "#PWR019" H 6600 4450 50  0001 C CNN
+F 0 "#PWR21" H 6600 4450 50  0001 C CNN
 F 1 "GND" H 6600 4550 50  0000 C CNN
 F 2 "" H 6600 4700 50  0000 C CNN
@@
 Wire Wire Line
 	6725 3900 6625 3900
-$Comp
-L Conn_02x05_Odd_Even J1
-U 1 1 59C6C1C0
-P 8400 3750
-F 0 "J1" H 8450 4050 50  0000 C CNN
-F 1 "Conn_02x05_Odd_Even" H 8450 3450 50  0000 C CNN
-F 2 "Pin_Headers:Pin_Header_Straight_2x05_Pitch2.54mm" H 8400 3750 50  0001 C CNN
-F 3 "" H 8400 3750 50  0001 C CNN
-	1    8400 3750
-	1    0    0    -1
-$EndComp
 Text GLabel 3450 3925 3    60   Input ~ 0
 SCL
@@
 SDA
 $Comp
-L R_10k R7
+L R_10k R11
 U 1 1 59C83F25
 P 3450 3700
-F 0 "R7" V 3450 3700 50  0000 C CNN
+F 0 "R11" V 3450 3700 50  0000 C CNN
 F 1 "R_10k" H 3325 3850 50  0000 C CNN
 F 2 "Resistors_SMD:R_0603_HandSoldering" V 3380 3700 50  0001 C CNN
@@
 $EndComp
 $Comp
-L R_10k R6
+L R_10k R10
 U 1 1 59C83F7C
 P 3350 3700
-F 0 "R6" V 3350 3700 50  0000 C CNN
+F 0 "R10" V 3350 3700 50  0000 C CNN
 F 1 "R_10k" H 3475 3850 50  0000 C CNN
 F 2 "Resistors_SMD:R_0603_HandSoldering" V 3280 3700 50  0001 C CNN
@@
 Wire Wire Line
 	4850 5400 5150 5400
+$Comp
+L Conn_02x05_Odd_Even J1
+U 1 1 5AC7372F
+P 8400 3750
+F 0 "J1" H 8450 4050 50  0000 C CNN
+F 1 "Conn_02x05_Odd_Even" H 8450 3450 50  0000 C CNN
+F 2 "Pin_Headers:Pin_Header_Straight_2x05_Pitch2.54mm" H 8400 3750 50  0001 C CNN
+F 3 "" H 8400 3750 50  0001 C CNN
+	1    8400 3750
+	1    0    0    -1
+$EndComp
 $EndSCHEMATC

Commit message: Schematic Work on Audio Amp
Audio amplifier implemented with selected components and footprints.
Connections:
- net labels added: MUTE_AUDIO_AMP, STBY_AUDIO_AMP
- wire segments 41 -> 43
Changed lines of the file:
@@
 $EndDescr
 $Comp
-L GND #PWR20
+L GND #PWR021
 U 1 1 59097974
 P 4825 2750
-F 0 "#PWR20" H 4825 2500 50  0001 C CNN
+F 0 "#PWR021" H 4825 2500 50  0001 C CNN
 F 1 "GND" H 4825 2600 50  0000 C CNN
 F 2 "" H 4825 2750 50  0000 C CNN
@@
 SDA
 $Comp
-L GND #PWR22
+L GND #PWR022
 U 1 1 590979B0
 P 8150 3500
-F 0 "#PWR22" H 8150 3250 50  0001 C CNN
+F 0 "#PWR022" H 8150 3250 50  0001 C CNN
 F 1 "GND" H 8150 3350 50  0000 C CNN
 F 2 "" H 8150 3500 50  0000 C CNN
@@
 5V
 $Comp
-L GND #PWR23
+L GND #PWR023
 U 1 1 590979B2
 P 8750 3500
-F 0 "#PWR23" H 8750 3250 50  0001 C CNN
+F 0 "#PWR023" H 8750 3250 50  0001 C CNN
 F 1 "GND" H 8750 3350 50  0000 C CNN
 F 2 "" H 8750 3500 50  0000 C CNN
@@
 	-1   0    0    1
 $EndComp
-Wire Wire Line
-	8750 3550 8750 3500
-Wire Wire Line
-	8700 3550 8750 3550
-Wire Wire Line
-	8150 3550 8200 3550
-Wire Wire Line
-	8150 3500 8150 3550
-Wire Wire Line
-	8700 3650 8800 3650
-Wire Wire Line
-	8800 3850 8700 3850
-Wire Wire Line
-	8700 3750 8800 3750
-Wire Wire Line
-	8100 3650 8200 3650
-Wire Wire Line
-	6625 3800 6725 3800
-Wire Wire Line
-	6725 3500 6625 3500
-Wire Wire Line
-	6625 3600 6725 3600
-Wire Wire Line
-	6725 3050 6625 3050
-Wire Wire Line
-	6625 2950 6725 2950
-Wire Wire Line
-	6625 4100 6725 4100
-Wire Wire Line
-	6175 4650 6175 4750
-Wire Wire Line
-	4775 3000 4875 3000
-Wire Wire Line
-	4875 2900 4775 2900
-Wire Wire Line
-	4825 2800 4875 2800
-Wire Wire Line
-	4825 2750 4825 2800
-Wire Wire Line
-	4775 4100 4875 4100
 Text GLabel 6725 3800 2    60   Input ~ 0
 POWER_EN
@@
 $EndComp
 $Comp
-L GND #PWR19
+L GND #PWR024
 U 1 1 59C55B05
 P 2625 4025
-F 0 "#PWR19" H 2625 3775 50  0001 C CNN
+F 0 "#PWR024" H 2625 3775 50  0001 C CNN
 F 1 "GND" H 2625 3875 50  0000 C CNN
 F 2 "" H 2625 4025 50  0000 C CNN
@@
 Text GLabel 2625 3400 1    60   Input ~ 0
 3V3
-Wire Wire Line
-	2425 3925 2425 3975
-Wire Wire Line
-	2425 3975 2825 3975
-Wire Wire Line
-	2825 3975 2825 3925
-Wire Wire Line
-	2625 4025 2625 3975
-Connection ~ 2625 3975
 Text Notes 2275 4400 0    60   ~ 0
 Bypass CAPs
@@
 Text GLabel 8100 3850 0    60   Input ~ 0
 FACTORY
-Wire Wire Line
-	8100 3850 8200 3850
-Wire Wire Line
-	8100 3750 8200 3750
 $Comp
 L R_10k R12
@@
 	0    1    1    0
 $EndComp
-Wire Wire Line
-	6250 4700 6175 4700
-Connection ~ 6175 4700
-$Comp
-L GND #PWR21
+$Comp
+L GND #PWR025
 U 1 1 59C60A9D
 P 6600 4700
-F 0 "#PWR21" H 6600 4450 50  0001 C CNN
+F 0 "#PWR025" H 6600 4450 50  0001 C CNN
 F 1 "GND" H 6600 4550 50  0000 C CNN
 F 2 "" H 6600 4700 50  0000 C CNN
@@
 	0    -1   -1   0
 $EndComp
-Wire Wire Line
-	6600 4700 6550 4700
 Text GLabel 4775 2900 0    60   Input ~ 0
 3V3
@@
 Text GLabel 8800 3950 2    60   Input ~ 0
 SDA
-Wire Wire Line
-	8100 3950 8200 3950
-Wire Wire Line
-	8700 3950 8800 3950
 Text GLabel 6725 3900 2    60   Input ~ 0
 PANEL_SW
-Wire Wire Line
-	6725 3900 6625 3900
 Text GLabel 3450 3925 3    60   Input ~ 0
 SCL
@@
 	-1   0    0    1
 $EndComp
-Wire Wire Line
-	3450 3850 3450 3925
-Wire Wire Line
-	3350 3925 3350 3850
-Wire Wire Line
-	3350 3550 3350 3425
-Wire Wire Line
-	3450 3425 3450 3550
 Text GLabel 3350 3425 1    60   Input ~ 0
 3V3
@@
 	1    0    0    -1
 $EndComp
-Wire Wire Line
-	2425 3625 2425 3525
-Wire Wire Line
-	2425 3525 2825 3525
-Wire Wire Line
-	2625 3525 2625 3400
-Wire Wire Line
-	2825 3525 2825 3625
-Connection ~ 2625 3525
-Wire Notes Line
-	2075 4275 2075 3150
-Wire Notes Line
-	2075 3150 3000 3150
-Wire Notes Line
-	3000 3150 3000 4275
-Wire Notes Line
-	3000 4275 2075 4275
 Text GLabel 4850 5250 0    60   Input ~ 0
 EN_5V_POWER
 Text GLabel 4850 5400 0    60   Input ~ 0
 EN_8V_POWER
-Wire Wire Line
-	4850 5250 5150 5250
-Wire Wire Line
-	4850 5400 5150 5400
 $Comp
 L Conn_02x05_Odd_Even J1
@@
 	1    0    0    -1
 $EndComp
+Text GLabel 4850 5550 0    60   Input ~ 0
+MUTE_AUDIO_AMP
+Text GLabel 4850 5700 0    60   Input ~ 0
+STBY_AUDIO_AMP
+Wire Wire Line
+	8750 3550 8750 3500
+Wire Wire Line
+	8700 3550 8750 3550
+Wire Wire Line
+	8150 3550 8200 3550
+Wire Wire Line
+	8150 3500 8150 3550
+Wire Wire Line
+	8700 3650 8800 3650
+Wire Wire Line
+	8800 3850 8700 3850
+Wire Wire Line
+	8700 3750 8800 3750
+Wire Wire Line
+	8100 3650 8200 3650
+Wire Wire Line
+	6625 3800 6725 3800
+Wire Wire Line
+	6725 3500 6625 3500
+Wire Wire Line
+	6625 3600 6725 3600
+Wire Wire Line
+	6725 3050 6625 3050
+Wire Wire Line
+	6625 2950 6725 2950
+Wire Wire Line
+	6625 4100 6725 4100
+Wire Wire Line
+	6175 4650 6175 4750
+Wire Wire Line
+	4775 3000 4875 3000
+Wire Wire Line
+	4875 2900 4775 2900
+Wire Wire Line
+	4825 2800 4875 2800
+Wire Wire Line
+	4825 2750 4825 2800
+Wire Wire Line
+	4775 4100 4875 4100
+Wire Wire Line
+	2425 3925 2425 3975
+Wire Wire Line
+	2425 3975 2825 3975
+Wire Wire Line
+	2825 3975 2825 3925
+Wire Wire Line
+	2625 4025 2625 3975
+Connection ~ 2625 3975
+Wire Wire Line
+	8100 3850 8200 3850
+Wire Wire Line
+	8100 3750 8200 3750
+Wire Wire Line
+	6250 4700 6175 4700
+Connection ~ 6175 4700
+Wire Wire Line
+	6600 4700 6550 4700
+Wire Wire Line
+	8100 3950 8200 3950
+Wire Wire Line
+	8700 3950 8800 3950
+Wire Wire Line
+	6725 3900 6625 3900
+Wire Wire Line
+	3450 3850 3450 3925
+Wire Wire Line
+	3350 3925 3350 3850
+Wire Wire Line
+	3350 3550 3350 3425
+Wire Wire Line
+	3450 3425 3450 3550
+Wire Wire Line
+	2425 3625 2425 3525
+Wire Wire Line
+	2425 3525 2825 3525
+Wire Wire Line
+	2625 3525 2625 3400
+Wire Wire Line
+	2825 3525 2825 3625
+Connection ~ 2625 3525
+Wire Notes Line
+	2075 4275 2075 3150
+Wire Notes Line
+	2075 3150 3000 3150
+Wire Notes Line
+	3000 3150 3000 4275
+Wire Notes Line
+	3000 4275 2075 4275
+Wire Wire Line
+	4850 5250 5150 5250
+Wire Wire Line
+	4850 5400 5150 5400
+Wire Wire Line
+	4850 5550 5150 5550
+Wire Wire Line
+	4850 5700 5150 5700
 $EndSCHEMATC
