File: microcontroller.sch (KiCad schematic (older format))
At the start: 7 parts, among them J1 Conn_02x05_Odd_Even, U4 ESP-WROOM-32

Commit message: added mainboard-interface
Parts:
- removed J1: Conn_02x05_Odd_Even, Pin_Headers:Pin_Header_Straight_2x05_Pitch2.54mm, symbol open-automation:Conn_02x05_Odd_Even
Connections:
- net labels added: SOFT_POWER
- net labels removed: 5V
- wire segments 46 -> 35
Changed lines of the file:
@@
 EESchema Schematic File Version 4
-LIBS:open-dash-daughterboard-cache
 EELAYER 26 0
 EELAYER END
 $Descr USLetter 11000 8500
 encoding utf-8
-Sheet 3 14
+Sheet 3 15
 Title ""
 Date ""
@@
 $Comp
 L open-automation:ESP-WROOM-32 U4
-U 1 1 590979AF
+U 1 1 5AF61D9A
 P 5775 3450
 F 0 "U4" H 6325 2350 60  0000 C CNN
@@
 	1    5775 3450
 	1    0    0    -1
-$EndComp
-$Comp
-L open-automation:GND #PWR022
-U 1 1 590979B0
-P 8150 3500
-F 0 "#PWR022" H 8150 3250 50  0001 C CNN
-F 1 "GND" H 8150 3350 50  0000 C CNN
-F 2 "" H 8150 3500 50  0000 C CNN
-F 3 "" H 8150 3500 50  0000 C CNN
-	1    8150 3500
-	-1   0    0    1
-$EndComp
-$Comp
-L open-automation:GND #PWR023
-U 1 1 590979B2
-P 8750 3500
-F 0 "#PWR023" H 8750 3250 50  0001 C CNN
-F 1 "GND" H 8750 3350 50  0000 C CNN
-F 2 "" H 8750 3500 50  0000 C CNN
-F 3 "" H 8750 3500 50  0000 C CNN
-	1    8750 3500
-	-1   0    0    1
 $EndComp
 Text Label 4200 1025 0    197  ~ 0
@@
 $Comp
 L open-automation:GND #PWR025
-U 1 1 59C60A9D
+U 1 1 5AF61DA0
 P 6600 4700
 F 0 "#PWR025" H 6600 4450 50  0001 C CNN
@@
 $Comp
 L open-automation:C_10uF C7
-U 1 1 5A10664F
+U 1 1 5AF61DA3
 P 2425 3775
 F 0 "C7" H 2450 3875 50  0000 L CNN
@@
 	1    0    0    -1
 $EndComp
-$Comp
-L open-automation:Conn_02x05_Odd_Even J1
-U 1 1 5AC7372F
-P 8400 3750
-F 0 "J1" H 8450 4050 50  0000 C CNN
-F 1 "Conn_02x05_Odd_Even" H 8450 3450 50  0000 C CNN
-F 2 "Pin_Headers:Pin_Header_Straight_2x05_Pitch2.54mm" H 8400 3750 50  0001 C CNN
-F 3 "" H 8400 3750 50  0001 C CNN
-	1    8400 3750
-	1    0    0    -1
-$EndComp
-Wire Wire Line
-	8750 3550 8750 3500
-Wire Wire Line
-	8700 3550 8750 3550
-Wire Wire Line
-	8150 3550 8200 3550
-Wire Wire Line
-	8150 3500 8150 3550
-Wire Wire Line
-	8700 3650 8800 3650
-Wire Wire Line
-	8800 3850 8700 3850
-Wire Wire Line
-	8700 3750 8800 3750
-Wire Wire Line
-	8100 3650 8200 3650
 Wire Wire Line
 	6625 3800 6725 3800
@@
 Connection ~ 2625 3975
 Wire Wire Line
-	8100 3850 8200 3850
-Wire Wire Line
-	8100 3750 8200 3750
-Wire Wire Line
 	6250 4700 6175 4700
 Connection ~ 6175 4700
 Wire Wire Line
 	6600 4700 6550 4700
-Wire Wire Line
-	8100 3950 8200 3950
-Wire Wire Line
-	8700 3950 8800 3950
 Wire Wire Line
 	6725 3900 6625 3900
@@
 Text HLabel 6725 2950 2    60   Input ~ 0
 TXD
-Text HLabel 8100 3650 0    60   Input ~ 0
-3V3
-Text HLabel 8100 3750 0    60   Input ~ 0
-PROG
-Text HLabel 8100 3850 0    60   Input ~ 0
-FACTORY
-Text HLabel 8100 3950 0    60   Input ~ 0
-SCL
-Text HLabel 8800 3650 2    60   Input ~ 0
-5V
-Text HLabel 8800 3750 2    60   Input ~ 0
-TXD
-Text HLabel 8800 3850 2    60   Input ~ 0
-RXD
-Text HLabel 8800 3950 2    60   Input ~ 0
-SDA
 Text HLabel 4775 4100 0    60   Input ~ 0
 FACTORY
@@
 Text HLabel 4775 3000 0    60   Input ~ 0
 ESP_EN
+Text HLabel 6725 4000 2    50   Output ~ 0
+SOFT_POWER
+Wire Wire Line
+	6625 4000 6725 4000
 $EndSCHEMATC

Commit message: organizing
Parts:
- removed U4: ESP-WROOM-32, open-automation:ESP-WROOM-32, symbol open-automation:ESP-WROOM-32
- added U14: ESP-WROOM-32, open-automation:ESP-WROOM-32, symbol open-automation:ESP-WROOM-32
Changed lines of the file:
@@
 	-1   0    0    1
-$EndComp
-$Comp
-L open-automation:ESP-WROOM-32 U4
-U 1 1 5AF61D9A
-P 5775 3450
-F 0 "U4" H 6325 2350 60  0000 C CNN
-F 1 "ESP-WROOM-32" H 5775 4250 60  0000 C CNN
-F 2 "open-automation:ESP-WROOM-32" H 5425 4050 60  0001 C CNN
-F 3 "https://www.espressif.com/sites/default/files/documentation/esp_wroom_32_datasheet_en.pdf" H 5425 4050 60  0001 C CNN
-	1    5775 3450
-	1    0    0    -1
 $EndComp
 Text Label 4200 1025 0    197  ~ 0
@@
 Wire Wire Line
 	6625 4000 6725 4000
+$Comp
+L open-automation:ESP-WROOM-32 U14
+U 1 1 5AFA4EFB
+P 5775 3450
+F 0 "U14" H 6325 2350 60  0000 C CNN
+F 1 "ESP-WROOM-32" H 5775 4250 60  0000 C CNN
+F 2 "open-automation:ESP-WROOM-32" H 5425 4050 60  0001 C CNN
+F 3 "https://www.espressif.com/sites/default/files/documentation/esp_wroom_32_datasheet_en.pdf" H 5425 4050 60  0001 C CNN
+	1    5775 3450
+	1    0    0    -1
+$EndComp
 $EndSCHEMATC

Commit message: update
Connections:
- net labels added: 3v3, EN_AUDIO, EN_ESP, EN_MAIN, MUTE_AUDIO, STBY_AUDIO
- net labels removed: 3V3, EN_5V_POWER, EN_8V_POWER, ESP_EN, IO2, MUTE_AUDIO_AMP, PANEL_SW, POWER_EN, STBY_AUDIO_AMP
- wire segments 35 -> 32
Changed lines of the file:
@@
 EESchema Schematic File Version 4
+LIBS:open-dash-daughterboard-cache
 EELAYER 26 0
 EELAYER END
 $Descr USLetter 11000 8500
 encoding utf-8
-Sheet 3 15
+Sheet 3 14
 Title ""
 Date ""
@@
 $EndComp
 Wire Wire Line
-	6625 3800 6725 3800
-Wire Wire Line
-	6725 3500 6625 3500
-Wire Wire Line
-	6625 3600 6725 3600
+	6625 3900 6725 3900
+Wire Wire Line
+	6725 3400 6625 3400
+Wire Wire Line
+	6625 3500 6725 3500
 Wire Wire Line
 	6725 3050 6625 3050
@@
 Wire Wire Line
 	6250 4700 6175 4700
-Connection ~ 6175 4700
 Wire Wire Line
 	6600 4700 6550 4700
-Wire Wire Line
-	6725 3900 6625 3900
 Wire Wire Line
 	3450 3850 3450 3925
@@
 	3000 4275 2075 4275
 Wire Wire Line
-	4850 5250 5150 5250
-Wire Wire Line
-	4850 5400 5150 5400
-Wire Wire Line
-	4850 5550 5150 5550
-Wire Wire Line
-	4850 5700 5150 5700
-Wire Wire Line
 	2625 3975 2825 3975
-Wire Wire Line
-	6175 4700 6175 4750
 Wire Wire Line
 	2625 3525 2825 3525
 Text HLabel 3350 3425 1    60   Input ~ 0
-3V3
+3v3
 Text HLabel 3450 3425 1    60   Input ~ 0
-3V3
+3v3
 Text HLabel 3450 3925 3    60   Input ~ 0
 SCL
@@
 SDA
 Text HLabel 2625 3400 1    60   Input ~ 0
-3V3
-Text HLabel 4850 5250 0    60   Input ~ 0
-EN_5V_POWER
-Text HLabel 4850 5400 0    60   Input ~ 0
-EN_8V_POWER
-Text HLabel 4850 5550 0    60   Input ~ 0
-MUTE_AUDIO_AMP
-Text HLabel 4850 5700 0    60   Input ~ 0
-STBY_AUDIO_AMP
-Text HLabel 6175 4750 3    60   Input ~ 0
-IO2
+3v3
+Text HLabel 6725 3600 2    60   Input ~ 0
+EN_MAIN
+Text HLabel 6725 3900 2    60   Input ~ 0
+EN_AUDIO
+Text HLabel 6725 3700 2    60   Input ~ 0
+MUTE_AUDIO
+Text HLabel 6725 3800 2    60   Input ~ 0
+STBY_AUDIO
 Text HLabel 6725 4100 2    60   Input ~ 0
 PROG
-Text HLabel 6725 3900 2    60   Input ~ 0
-PANEL_SW
-Text HLabel 6725 3800 2    60   Input ~ 0
-POWER_EN
-Text HLabel 6725 3600 2    60   Input ~ 0
+Text HLabel 6725 3500 2    60   Input ~ 0
 SDA
-Text HLabel 6725 3500 2    60   Input ~ 0
+Text HLabel 6725 3400 2    60   Input ~ 0
 SCL
 Text HLabel 6725 3050 2    60   Input ~ 0
@@
 FACTORY
 Text HLabel 4775 2900 0    60   Input ~ 0
-3V3
+3v3
 Text HLabel 4775 3000 0    60   Input ~ 0
-ESP_EN
+EN_ESP
 Text HLabel 6725 4000 2    50   Output ~ 0
 SOFT_POWER
@@
 	1    0    0    -1
 $EndComp
+Wire Wire Line
+	6625 3700 6725 3700
+Wire Wire Line
+	6725 3800 6625 3800
+Wire Wire Line
+	6625 3600 6725 3600
 $EndSCHEMATC

Commit message: update
Parts:
- C10: renamed from C7; footprint Capacitors_SMD:C_0603_HandSoldering -> Capacitor_SMD:C_0603_1608Metric_Pad0.99x1.00mm_HandSolder
- C11: renamed from C8; footprint Capacitors_SMD:C_0603_HandSoldering -> Capacitor_SMD:C_0603_1608Metric_Pad0.99x1.00mm_HandSolder
- R13: renamed from R10; footprint Resistors_SMD:R_0603_HandSoldering -> Resistor_SMD:R_0603_1608Metric_Pad0.99x1.00mm_HandSolder
- R14: renamed from R11; footprint Resistors_SMD:R_0603_HandSoldering -> Resistor_SMD:R_0603_1608Metric_Pad0.99x1.00mm_HandSolder
- R15: renamed from R12; footprint Resistors_SMD:R_0603_HandSoldering -> Resistor_SMD:R_0603_1608Metric_Pad0.99x1.00mm_HandSolder
- renumbered U14 to U6
Connections:
- net labels added: CAN_RX, CAN_TX, EN_DISPLAY
- wire segments 32 -> 35
Changed lines of the file:
@@
 $Descr USLetter 11000 8500
 encoding utf-8
-Sheet 3 14
+Sheet 3 13
 Title ""
 Date ""
@@
 $EndDescr
 $Comp
-L open-automation:GND #PWR021
+L open-automation:GND #PWR027
 U 1 1 59097974
 P 4825 2750
-F 0 "#PWR021" H 4825 2500 50  0001 C CNN
+F 0 "#PWR027" H 4825 2500 50  0001 C CNN
 F 1 "GND" H 4825 2600 50  0000 C CNN
 F 2 "" H 4825 2750 50  0000 C CNN
@@
 Microcontroller
 $Comp
-L open-automation:C_1uF C8
+L open-automation:C_1uF C11
 U 1 1 59C55B03
 P 2825 3775
-F 0 "C8" H 2825 3875 50  0000 L CNN
+F 0 "C11" H 2825 3875 50  0000 L CNN
 F 1 "C_1uF" H 2575 3675 50  0000 L CNN
-F 2 "Capacitors_SMD:C_0603_HandSoldering" H 2925 4075 50  0001 C CNN
+F 2 "Capacitor_SMD:C_0603_1608Metric_Pad0.99x1.00mm_HandSolder" H 2925 4075 50  0001 C CNN
 F 3 "https://www.digikey.com/product-detail/en/yageo/CC0603ZRY5V7BB105/311-1372-1-ND/2103156" H 2825 3525 50  0001 C CNN
 F 4 "CC0603ZRY5V7BB105" H 2950 3975 60  0001 C CNN "Part Number"
@@
 $EndComp
 $Comp
-L open-automation:GND #PWR024
+L open-automation:GND #PWR026
 U 1 1 59C55B05
 P 2625 4025
-F 0 "#PWR024" H 2625 3775 50  0001 C CNN
+F 0 "#PWR026" H 2625 3775 50  0001 C CNN
 F 1 "GND" H 2625 3875 50  0000 C CNN
 F 2 "" H 2625 4025 50  0000 C CNN
@@
 Bypass CAPs
 $Comp
-L open-automation:R_10k R12
+L open-automation:R_10k R15
 U 1 1 59C609F8
 P 6400 4700
-F 0 "R12" V 6400 4700 50  0000 C CNN
+F 0 "R15" V 6400 4700 50  0000 C CNN
 F 1 "R_10k" V 6325 4700 50  0000 C CNN
-F 2 "Resistors_SMD:R_0603_HandSoldering" V 6330 4700 50  0001 C CNN
+F 2 "Resistor_SMD:R_0603_1608Metric_Pad0.99x1.00mm_HandSolder" V 6330 4700 50  0001 C CNN
 F 3 "https://www.digikey.com/product-detail/en/yageo/RC0603JR-0710KL/311-10KGRCT-ND/729647" V 6480 4700 50  0001 C CNN
 F 4 "RC0603JR-0710KL" V 6580 4800 60  0001 C CNN "Part Number"
@@
 $EndComp
 $Comp
-L open-automation:GND #PWR025
+L open-automation:GND #PWR028
 U 1 1 5AF61DA0
 P 6600 4700
-F 0 "#PWR025" H 6600 4450 50  0001 C CNN
+F 0 "#PWR028" H 6600 4450 50  0001 C CNN
 F 1 "GND" H 6600 4550 50  0000 C CNN
 F 2 "" H 6600 4700 50  0000 C CNN
@@
 $EndComp
 $Comp
-L open-automation:R_10k R11
+L open-automation:R_10k R14
 U 1 1 59C83F25
 P 3450 3700
-F 0 "R11" V 3450 3700 50  0000 C CNN
+F 0 "R14" V 3450 3700 50  0000 C CNN
 F 1 "R_10k" H 3325 3850 50  0000 C CNN
-F 2 "Resistors_SMD:R_0603_HandSoldering" V 3380 3700 50  0001 C CNN
+F 2 "Resistor_SMD:R_0603_1608Metric_Pad0.99x1.00mm_HandSolder" V 3380 3700 50  0001 C CNN
 F 3 "https://www.digikey.com/product-detail/en/yageo/RC0603JR-0710KL/311-10KGRCT-ND/729647" V 3530 3700 50  0001 C CNN
 F 4 "RC0603JR-0710KL" V 3630 3800 60  0001 C CNN "Part Number"
@@
 $EndComp
 $Comp
-L open-automation:R_10k R10
+L open-automation:R_10k R13
 U 1 1 59C83F7C
 P 3350 3700
-F 0 "R10" V 3350 3700 50  0000 C CNN
+F 0 "R13" V 3350 3700 50  0000 C CNN
 F 1 "R_10k" H 3475 3850 50  0000 C CNN
-F 2 "Resistors_SMD:R_0603_HandSoldering" V 3280 3700 50  0001 C CNN
+F 2 "Resistor_SMD:R_0603_1608Metric_Pad0.99x1.00mm_HandSolder" V 3280 3700 50  0001 C CNN
 F 3 "https://www.digikey.com/product-detail/en/yageo/RC0603JR-0710KL/311-10KGRCT-ND/729647" V 3430 3700 50  0001 C CNN
 F 4 "RC0603JR-0710KL" V 3530 3800 60  0001 C CNN "Part Number"
@@
 $EndComp
 $Comp
-L open-automation:C_10uF C7
+L open-automation:C_10uF C10
 U 1 1 5AF61DA3
 P 2425 3775
-F 0 "C7" H 2450 3875 50  0000 L CNN
+F 0 "C10" H 2450 3875 50  0000 L CNN
 F 1 "C_10uF" H 2125 3675 50  0000 L CNN
-F 2 "Capacitors_SMD:C_0603_HandSoldering" H 2525 4075 50  0001 C CNN
+F 2 "Capacitor_SMD:C_0603_1608Metric_Pad0.99x1.00mm_HandSolder" H 2525 4075 50  0001 C CNN
 F 3 "https://www.digikey.com/product-detail/en/murata-electronics-north-america/GRM188R61A106ME69D/490-10475-1-ND/5026393" H 2425 3525 50  0001 C CNN
 F 4 "GRM188R61A106ME69D" H 2550 3975 60  0001 C CNN "Part Number"
@@
 Text HLabel 6725 3900 2    60   Input ~ 0
 EN_AUDIO
-Text HLabel 6725 3700 2    60   Input ~ 0
+Text HLabel 4775 3700 0    60   Input ~ 0
 MUTE_AUDIO
-Text HLabel 6725 3800 2    60   Input ~ 0
+Text HLabel 4775 3600 0    60   Input ~ 0
 STBY_AUDIO
 Text HLabel 6725 4100 2    60   Input ~ 0
@@
 Text HLabel 4775 3000 0    60   Input ~ 0
 EN_ESP
-Text HLabel 6725 4000 2    50   Output ~ 0
+Text HLabel 4765 4200 0    50   Output ~ 0
 SOFT_POWER
 Wire Wire Line
 	6625 4000 6725 4000
 $Comp
-L open-automation:ESP-WROOM-32 U14
+L open-automation:ESP-WROOM-32 U6
 U 1 1 5AFA4EFB
 P 5775 3450
-F 0 "U14" H 6325 2350 60  0000 C CNN
+F 0 "U6" H 6325 2350 60  0000 C CNN
 F 1 "ESP-WROOM-32" H 5775 4250 60  0000 C CNN
 F 2 "open-automation:ESP-WROOM-32" H 5425 4050 60  0001 C CNN
@@
 	6625 3700 6725 3700
 Wire Wire Line
-	6725 3800 6625 3800
-Wire Wire Line
 	6625 3600 6725 3600
+Text HLabel 6075 4725 3    60   Input ~ 0
+EN_DISPLAY
+Wire Wire Line
+	6075 4725 6075 4650
+Wire Wire Line
+	4875 4200 4765 4200
+Text HLabel 6720 4000 2    60   Input ~ 0
+CAN_RX
+Text HLabel 6720 3700 2    60   Input ~ 0
+CAN_TX
+Wire Wire Line
+	4775 3700 4875 3700
+Wire Wire Line
+	4775 3600 4875 3600
 $EndSCHEMATC

Commit message: update
Changed lines of the file:
@@
 Wire Wire Line
 	4875 4200 4765 4200
-Text HLabel 6720 4000 2    60   Input ~ 0
+Text HLabel 6725 4000 2    60   Input ~ 0
 CAN_RX
-Text HLabel 6720 3700 2    60   Input ~ 0
+Text HLabel 6725 3700 2    60   Input ~ 0
 CAN_TX
 Wire Wire Line

Commit message: starting next revision
Connections:
- net labels added: 3V3
- net labels removed: 3v3
Changed lines of the file:
@@
-EESchema Schematic File Version 4
-LIBS:open-dash-daughterboard-cache
-EELAYER 26 0
+EESchema Schematic File Version 5
+EELAYER 29 0
 EELAYER END
 $Descr USLetter 11000 8500
@@
 	2625 3525 2825 3525
 Text HLabel 3350 3425 1    60   Input ~ 0
-3v3
+3V3
 Text HLabel 3450 3425 1    60   Input ~ 0
-3v3
+3V3
 Text HLabel 3450 3925 3    60   Input ~ 0
 SCL
@@
 SDA
 Text HLabel 2625 3400 1    60   Input ~ 0
-3v3
+3V3
 Text HLabel 6725 3600 2    60   Input ~ 0
 EN_MAIN
@@
 FACTORY
 Text HLabel 4775 2900 0    60   Input ~ 0
-3v3
+3V3
 Text HLabel 4775 3000 0    60   Input ~ 0
 EN_ESP
