File: power.sch (KiCad schematic (older format))
At the start: 0 parts

Commit message: Ethan Initial Commit
Copy of power section from smart-regulator
Parts:
- added BATTERY1, PANEL1: CONN_01X02, open-automation:XT60, symbol CONN_01X02
- added C1: 100uF, Capacitors_THT:CP_Radial_D10.0mm_P3.50mm, symbol CP
- added C2: 1000uF, Capacitors_THT:CP_Radial_D10.0mm_P3.50mm, symbol CP
- added C3: 4.7uF, Capacitors_SMD:C_0603_HandSoldering, symbol C
- added C8: C_0.1uF, Capacitors_SMD:C_0603_HandSoldering, symbol C_0.1uF
- added D1: D_Schottky, Diodes_SMD:D_SMA, symbol D_Schottky
- added D4: LED, LEDs:LED_0603_HandSoldering, symbol LED
- added L1: 47uH, open-automation:L-RAD-7.4mm, symbol L
- added Q1: Q_NMOS_GSD_AOD4184A, TO_SOT_Packages_SMD:TO-252-2_Rectifier, symbol Q_NMOS_GSD_AOD4184A
- added R1: R_10m, Resistors_SMD:R_2512_HandSoldering, symbol R_10m
- added R11, R8: R_10k, Resistors_SMD:R_0603_HandSoldering, symbol R_10k
- added R7: 1K, Resistors_SMD:R_0603_HandSoldering, symbol R
- added U11: NCP1117LPST33T3G, TO_SOT_Packages_SMD:SOT-223, symbol NCP1117LPST33T3G
- added U3: LM2576, open-automation:Regulator-LM2576, symbol LM2576
- added U5: Power-Monitor-INA219, TO_SOT_Packages_SMD:SOT-23-8_Handsoldering, symbol Power-Monitor-INA219
Connections:
- net labels added: 3V3, BATTERY, GND, PANEL_SW, SCL, SDA, V_MAIN, V_PANEL, V_USB, power_EN
- wire segments 0 -> 56

Commit message: Micro and Environment Schematic Copy
Copied over the microcontroller and environment sheets from smart-regulator project. Also modified the power section.
Parts:
- removed C8: C_0.1uF, Capacitors_SMD:C_0603_HandSoldering, symbol C_0.1uF
- removed Q1: Q_NMOS_GSD_AOD4184A, TO_SOT_Packages_SMD:TO-252-2_Rectifier, symbol Q_NMOS_GSD_AOD4184A
- removed R1: R_10m, Resistors_SMD:R_2512_HandSoldering, symbol R_10m
- removed R7: 1K, Resistors_SMD:R_0603_HandSoldering, symbol R
- removed U5: Power-Monitor-INA219, TO_SOT_Packages_SMD:SOT-23-8_Handsoldering, symbol Power-Monitor-INA219
- added C7: 10 uF, symbol CP
- 12V_Out1: renamed from PANEL1; footprint open-automation:XT60 -> smart-regulator:XT60
- BATTERY1: footprint open-automation:XT60 -> smart-regulator:XT60
- L1: footprint open-automation:L-RAD-7.4mm -> smart-regulator:L-RAD-7.4mm
- U3: footprint open-automation:Regulator-LM2576 -> smart-regulator:Regulator-LM2576
Connections:
- net labels added: 12V, POWER_EN
- net labels removed: PANEL_SW, SCL, SDA, V_PANEL, V_USB, power_EN
- wire segments 56 -> 34
Other:
- note added: "12V Battery Input"
- note added: "Main Board Power Output"
- note added: "V_MAIN is after the current sense resistor."

Commit message: Power Schematic Update
Test commit and minior power schematic update.
Connections:
- net labels added: 5V
- wire segments 34 -> 35

Commit message: Backup Before SEPIC Design
Parts:
- removed U3: LM2576, smart-regulator:Regulator-LM2576, symbol LM2576
- added U?: LM2576SX-3.3, open-automation:Regulator-LM2576, symbol LM2576SX-3.3
- 12V_Out1, BATTERY1: footprint smart-regulator:XT60 -> open-automation:XT60
- L1: footprint smart-regulator:L-RAD-7.4mm -> open-automation:L-RAD-7.4mm
Connections:
- wire segments 35 -> 44
Changed lines of the file:
@@
 Comment4 ""
 $EndDescr
-$Comp
-L LM2576 U3
-U 1 1 5936E607
-P 4475 1075
-F 0 "U3" H 4825 1275 60  0000 C CNN
-F 1 "LM2576" H 4525 875 60  0000 C CNN
-F 2 "smart-regulator:Regulator-LM2576" H 4875 1025 60  0001 C CNN
-F 3 "https://www.digikey.com/product-detail/en/texas-instruments/LM2576SX-5.0-NOPB/LM2576SX-5.0-NOPBCT-ND/3440106" H 4875 1025 60  0001 C CNN
-F 4 "LM2576SX-5.0/NOPB" H 4475 1075 60  0001 C CNN "Part Number"
-	1    4475 1075
-	1    0    0    -1
-$EndComp
 Text GLabel 2650 975  0    60   Input ~ 0
 V_MAIN
@@
 F 0 "L1" V 5275 1075 50  0001 C CNN
 F 1 "47uH" V 5275 1075 50  0000 C CNN
-F 2 "smart-regulator:L-RAD-7.4mm" H 5325 1075 50  0001 C CNN
+F 2 "open-automation:L-RAD-7.4mm" H 5325 1075 50  0001 C CNN
 F 3 "https://www.digikey.com/product-detail/en/abracon-llc/AIUR-06-470K/535-13031-ND/2343602" H 5325 1075 50  0001 C CNN
 F 4 "AIUR-06-470K" V 5325 1075 10  0001 C CNN "Part Number"
@@
 F 1 "D_Schottky" H 5125 1175 50  0001 C CNN
 F 2 "Diodes_SMD:D_SMA" H 5125 1275 50  0001 C CNN
-F 3 "http://www.digikey.com/scripts/DkSearch/dksus.dll?Detail&itemSeq=233263850&uq=636356340886764109" H 5125 1275 50  0001 C CNN
+F 3 "https://www.digikey.com/product-detail/en/diodes-incorporated/B330A-13-F/B330A-FDICT-ND/815332" H 5125 1275 50  0001 C CNN
 F 4 "B330A-13-F" H 5125 1275 60  0001 C CNN "Part Number"
 	1    5125 1275
@@
 F 0 "BATTERY1" H 1228 1091 50  0000 L CNN
 F 1 "CONN_01X02" H 1228 1000 50  0000 L CNN
-F 2 "smart-regulator:XT60" H 1150 1050 50  0001 C CNN
+F 2 "open-automation:XT60" H 1150 1050 50  0001 C CNN
 F 3 "https://www.digikey.com/product-detail/en/phoenix-contact/1934861/277-1607-ND/568644" H 1150 1050 50  0001 C CNN
 	1    1150 1050
@@
 	4225 2550 4225 2500
 Wire Wire Line
-	2675 2400 3375 2400
+	2675 2400 2975 2400
+Wire Wire Line
+	2975 2400 3375 2400
 Wire Wire Line
 	3325 2600 3375 2600
 Wire Wire Line
-	3325 2600 3325 2825
-Wire Wire Line
-	4125 2500 4825 2500
+	3325 2600 3325 2800
+Wire Wire Line
+	3325 2800 3325 2825
+Wire Wire Line
+	4125 2500 4225 2500
+Wire Wire Line
+	4225 2500 4625 2500
+Wire Wire Line
+	4625 2500 4825 2500
 Wire Wire Line
 	5125 1125 5125 1075
@@
 	5475 1075 5525 1075
 Wire Wire Line
-	5075 1075 5175 1075
-Wire Wire Line
-	5075 975  6075 975
+	5075 1075 5125 1075
+Wire Wire Line
+	5125 1075 5175 1075
+Wire Wire Line
+	5075 975  5525 975
+Wire Wire Line
+	5525 975  5775 975
+Wire Wire Line
+	5775 975  6075 975
 Wire Wire Line
 	8850 975  9175 975
@@
 	2900 1175 2900 975
 Wire Wire Line
-	2650 975  3975 975
+	2650 975  2900 975
+Wire Wire Line
+	2900 975  3975 975
 Connection ~ 2900 975
 Wire Wire Line
@@
 	3925 1175 3975 1175
 Wire Wire Line
-	3525 1075 3975 1075
+	3525 1075 3675 1075
+Wire Wire Line
+	3675 1075 3975 1075
 Wire Wire Line
 	1400 1150 1400 1100
@@
 F 0 "12V_Out1" H 9453 1066 50  0000 L CNN
 F 1 "CONN_01X02" H 9453 975 50  0000 L CNN
-F 2 "smart-regulator:XT60" H 9375 1025 50  0001 C CNN
+F 2 "open-automation:XT60" H 9375 1025 50  0001 C CNN
 F 3 "https://www.digikey.com/product-detail/en/phoenix-contact/1934861/277-1607-ND/568644" H 9375 1025 50  0001 C CNN
 	1    9375 1025
@@
 Text GLabel 8850 975  0    60   Input ~ 0
 12V
+$Comp
+L LM2576SX-3.3 U?
+U 1 1 5AC3E9C2
+P 4475 1075
+F 0 "U?" H 4825 1275 60  0000 C CNN
+F 1 "LM2576SX-3.3" H 4525 875 60  0000 C CNN
+F 2 "open-automation:Regulator-LM2576" H 4375 675 60  0001 C CNN
+F 3 "https://www.digikey.com/products/en?keywords=LM2576SX-3.3%2FNOPBCT-ND" H 4425 775 60  0001 C CNN
+	1    4475 1075
+	1    0    0    -1
+$EndComp
 $EndSCHEMATC

Commit message: Component Updates in Power Section
Parts:
- removed C3: 4.7uF, Capacitors_SMD:C_0603_HandSoldering, symbol C
- removed C7: 10 uF, symbol CP
- removed R8: R_10k, Resistors_SMD:R_0603_HandSoldering, symbol R_10k
- removed U11: NCP1117LPST33T3G, TO_SOT_Packages_SMD:SOT-223, symbol NCP1117LPST33T3G
- added C?: 100uF, Capacitors_THT:CP_Radial_D10.0mm_P3.50mm, symbol CP
- added C?: 1000uF, Capacitors_THT:CP_Radial_D10.0mm_P3.50mm, symbol CP
- added D?: D_Schottky, Diodes_SMD:D_SMA, symbol D_Schottky
- added L?: 47uH, open-automation:L-RAD-7.4mm, symbol L
- added R?: R_10k, Resistors_SMD:R_0603_HandSoldering, symbol R_10k
- added U?: LM2576SX-5.0, open-automation:Regulator-LM2576, symbol LM2576SX-3.3
- L1: value 47uH -> 68uH; footprint open-automation:L-RAD-7.4mm -> (none); Part Number AIUR-06-470K -> Wurth 7447709680
- R11: value R_10k -> R_1k4; Part Number RC0603JR-0710KL -> RC0603FR-071K4L
- U?: Part Number (none) -> LM2576SX-3.3/NOPB
Connections:
- net labels added: EN_5V_POWER
- net labels removed: POWER_EN
- wire segments 44 -> 43
Other:
- note added: "1mA current through LED"

Commit message: Updated Power Schematic
Power Schematic Updated for 3.3V, 5V, and 8V Buck Regulators. All regulator parts have correct footprints and selected components.

Prelim orgainization of PCB - grouped parts by section.
Parts:
- removed C?: 100uF, Capacitors_THT:CP_Radial_D10.0mm_P3.50mm, symbol CP
- removed C?: 1000uF, Capacitors_THT:CP_Radial_D10.0mm_P3.50mm, symbol CP
- removed D?: D_Schottky, Diodes_SMD:D_SMA, symbol D_Schottky
- added 5V_Out1: CONN_01X02, open-automation:XT60, symbol CONN_01X02
- added C2, C3: 180uF, Capacitors_THT:CP_Radial_D8.0mm_P3.50mm, symbol CP
- added C5, C6: 1000uF, Capacitors_THT:CP_Radial_D10.0mm_P5.00mm, symbol CP
- added D2, D3: D_Schottky, Diodes_SMD:D_SMA, symbol D_Schottky
- added L3: 100uH, open-automation:L_Toroid_Horizontal_D21.8mm_P20.06mm_Bourns_2100, symbol L
- added R2: R_10k, Resistors_SMD:R_0603_HandSoldering, symbol R_10k
- added R4: R_7.15k, Resistors_SMD:R_0603_HandSoldering, symbol R_10k
- added R5: R_1.3k, Resistors_SMD:R_0603_HandSoldering, symbol R_10k
- added U3: LM2576SX-ADJ, open-automation:Regulator-LM2576, symbol LM2576SX-3.3
- C1: value 100uF -> 180uF; footprint Capacitors_THT:CP_Radial_D10.0mm_P3.50mm -> Capacitors_THT:CP_Radial_D8.0mm_P3.50mm; Part Number UVR1H101MPD -> EKZN500ELL181MH20D
- C4: renamed from C2; footprint Capacitors_THT:CP_Radial_D10.0mm_P3.50mm -> Capacitors_THT:CP_Radial_D10.0mm_P5.00mm; Part Number UVR0J102MPD1TD -> 25YXJ1000M10X20
- D1: Part Number B330A-13-F -> CDBA540-HF
- L1: footprint (none) -> Inductors_SMD:L_12x12mm_h8mm
- L2: renamed from L?; value 47uH -> 100uH; footprint open-automation:L-RAD-7.4mm -> open-automation:L_Toroid_Horizontal_D21.8mm_P20.06mm_Bourns_2100; Part Number AIUR-06-470K -> 2100HT-101-H-RC
- gave numbers to parts that had none: 3
- renumbered R11 to R3
Connections:
- net labels added: 3.3V, 8V, 8V_FeedBack, EN_8V_POWER
- net labels removed: 12V
- wire segments 43 -> 66
Other:
- note added: "Battery Passthrough"
- note added: "Main Board 5V Supply"
- note added: "Main Board Connections"
- note removed: "Main Board Power Output"

Commit message: Update Power Schematic and directed parts to open-automation library
Change 3.3V and 5V buck regulator to adjustable chip version.

Directed multiple parts from -cache.lib to open-automation.lib.
Parts:
- removed 12V_Out1, 5V_Out1, BATTERY1: CONN_01X02, open-automation:XT60, symbol CONN_01X02
- removed U1: LM2576SX-3.3, open-automation:Regulator-LM2576, symbol LM2576SX-3.3
- removed U2: LM2576SX-5.0, open-automation:Regulator-LM2576, symbol LM2576SX-3.3
- removed U3: LM2576SX-ADJ, open-automation:Regulator-LM2576, symbol LM2576SX-3.3
- added 5V_OUT_1, BATT_IN_1, BATT_OUT_1: CONN_01X02, open-automation:XT60, symbol CONN_01X02
- added R3: R_3.92k, Resistors_SMD:R_0603_HandSoldering, symbol R_10k
- added R5, R7: R_7.15k, Resistors_SMD:R_0603_HandSoldering, symbol R_10k
- added R6: R_2.32k, Resistors_SMD:R_0603_HandSoldering, symbol R_10k
- added U1, U2, U3: LM2576-ADJ, open-automation:Regulator-LM2576, symbol LM2576
- R4: value R_7.15k -> R_2.32k; Part Number RC0603JR-0710KL -> RC0603FR-072K32L
- R8: renamed from R5; Part Number RC0603JR-0710KL -> RC0603FR-071K3L
- renumbered C3 to C1, C1 to C3, R3 to R9
Connections:
- net labels added: 3.3V_Feedback, 5V_Feedback, 8V_Feedback
- net labels removed: 8V_FeedBack
- wire segments 66 -> 71

Commit message: Schematic Work on Audio Amp
Audio amplifier implemented with selected components and footprints.
Parts:
- added D1: 26V Zener, Diodes_SMD:D_SMB, symbol D_Zener
- renumbered D1 to D2, D2 to D3, D3 to D4, D4 to D5
Connections:
- net labels added: AGND
- wire segments 71 -> 99
