File: audio-amplifier.sch (KiCad schematic (older format))
At the start: 0 parts

Commit message: Schematic Work on Audio Amp
Audio amplifier implemented with selected components and footprints.
Parts:
- added C12, C13: 0.22uF, Capacitors_SMD:C_0603_HandSoldering, symbol C
- added C14: 470uF, Capacitors_THT:CP_Radial_D8.0mm_P3.50mm, symbol CP
- added C15: 1uF, Capacitors_SMD:C_0603_HandSoldering, symbol C
- added C16: 10uF, Capacitors_THT:CP_Radial_D5.0mm_P2.00mm, symbol CP
- added C17: 100nF, Capacitors_SMD:C_0603_HandSoldering, symbol C
- added R14, R15: R_10k, Resistors_SMD:R_0603_HandSoldering, symbol R
- added U8: TDA7297, TO_SOT_Packages_THT:TO-220-15_Vertical_StaggeredType1, symbol TDA7297
Connections:
- net labels added: 8V, AGND, GND, L_AUDIO_IN, L_AUDIO_OUT+, L_AUDIO_OUT-, MUTE_AUDIO_AMP, R_AUDIO_IN, R_AUDIO_OUT+, R_AUDIO_OUT-, STBY_AUDIO_AMP
- wire segments 0 -> 35

Commit message: Fixed Ethan Branch to actually merge "lawrence_test" branch
Had some clinfict issues that were handeled incorrectly. Problems now fixed.
Parts:
- C12, C13, C15, C17: symbol C -> Device:C
- C14, C16: symbol CP -> Device:C
- R14, R15: symbol R -> Device:R
- U8: symbol TDA7297 -> open-automation:TDA7297
Connections:
- wire segments 35 -> 50
Changed lines of the file:
@@
-EESchema Schematic File Version 2
-LIBS:device
-LIBS:open-automation
+EESchema Schematic File Version 4
 LIBS:open-dash-daughterboard-cache
-EELAYER 25 0
+EELAYER 26 0
 EELAYER END
 $Descr A4 11693 8268
 encoding utf-8
-Sheet 7 11
+Sheet 7 13
 Title ""
 Date ""
@@
 $EndDescr
 $Comp
-L TDA7297 U8
+L open-automation:TDA7297 U8
 U 1 1 5AC797FB
 P 4500 1750
@@
 	1    0    0    -1
 $EndComp
-Text GLabel 2725 1400 0    60   Input ~ 0
-8V
-$Comp
-L AGND #PWR033
+$Comp
+L open-automation:AGND #PWR033
 U 1 1 5AC7B29E
 P 3750 1800
@@
 $EndComp
 $Comp
-L GND #PWR034
+L open-automation:GND #PWR034
 U 1 1 5AC7B2BE
 P 2850 1850
@@
 $EndComp
 $Comp
-L CP C14
+L Device:C C14
 U 1 1 5AC7B472
 P 2850 1600
@@
 $EndComp
 $Comp
-L C C17
+L Device:C C17
 U 1 1 5AC7B4BE
 P 3175 1600
@@
 	1    0    0    -1
 $EndComp
-Text GLabel 2425 2875 0    60   Input ~ 0
-MUTE_AUDIO_AMP
-Text GLabel 2425 3650 0    60   Input ~ 0
-STBY_AUDIO_AMP
-$Comp
-L R R14
+$Comp
+L Device:R R14
 U 1 1 5AC7BCAE
 P 2700 2875
@@
 $EndComp
 $Comp
-L GND #PWR035
+L open-automation:GND #PWR035
 U 1 1 5AC7C381
 P 3025 3325
@@
 $EndComp
 $Comp
-L GND #PWR036
+L open-automation:GND #PWR036
 U 1 1 5AC7C45C
 P 3050 4125
@@
 $EndComp
 Wire Wire Line
-	3900 1500 3800 1500
+	3900 1500 3850 1500
 Wire Wire Line
 	3800 1400 3800 1500
 Wire Wire Line
-	2725 1400 3900 1400
+	2725 1400 2850 1400
 Connection ~ 3800 1400
 Wire Wire Line
-	3750 1800 3900 1800
-Wire Wire Line
-	3900 1700 3550 1700
+	3750 1800 3850 1800
+Wire Wire Line
+	3900 1700 3850 1700
 Wire Wire Line
 	2850 1450 2850 1400
@@
 Connection ~ 3175 1400
 Wire Wire Line
-	2850 1750 2850 1850
-Wire Wire Line
-	2850 1800 3550 1800
+	2850 1750 2850 1800
+Wire Wire Line
+	2850 1800 3175 1800
 Wire Wire Line
 	3175 1800 3175 1750
@@
 	2550 2875 2425 2875
 Wire Wire Line
-	2850 3650 3675 3650
+	2850 3650 3050 3650
 Wire Wire Line
 	3050 3650 3050 3725
 Connection ~ 3050 3650
 Wire Wire Line
-	2850 2875 3600 2875
+	2850 2875 3025 2875
 Wire Wire Line
 	3025 2875 3025 2950
@@
 	3050 4025 3050 4125
 Wire Wire Line
-	3675 2350 3900 2350
-Wire Wire Line
-	3600 2250 3900 2250
-$Comp
-L C C12
+	3675 2350 3850 2350
+Wire Wire Line
+	3600 2250 3850 2250
+$Comp
+L Device:C C12
 U 1 1 5AC7CAB7
 P 2750 2325
@@
 	3525 2575 3525 2100
 Wire Wire Line
-	3525 2100 3900 2100
-Wire Wire Line
-	3900 2000 3450 2000
+	3525 2100 3850 2100
+Wire Wire Line
+	3900 2000 3850 2000
 Wire Wire Line
 	3450 2000 3450 2325
@@
 Wire Wire Line
 	2600 2575 2400 2575
-Text GLabel 2400 2325 0    60   Input ~ 0
-L_AUDIO_IN
-Text GLabel 2400 2575 0    60   Input ~ 0
-R_AUDIO_IN
 Wire Wire Line
 	5050 1650 5225 1650
@@
 Wire Wire Line
 	5050 2100 5225 2100
-Text GLabel 5225 1650 2    60   Input ~ 0
-L_AUDIO_OUT+
-Text GLabel 5225 1750 2    60   Input ~ 0
-L_AUDIO_OUT-
-Text GLabel 5225 2000 2    60   Input ~ 0
-R_AUDIO_OUT+
-Text GLabel 5225 2100 2    60   Input ~ 0
-R_AUDIO_OUT-
 Wire Wire Line
 	3600 2875 3600 2250
@@
 	3675 3650 3675 2350
 $Comp
-L C C13
+L Device:C C13
 U 1 1 5AC80604
 P 2750 2575
@@
 $EndComp
 $Comp
-L C C15
+L Device:C C15
 U 1 1 5AC80ED0
 P 3025 3100
@@
 $EndComp
 $Comp
-L CP C16
+L Device:C C16
 U 1 1 5AC81549
 P 3050 3875
@@
 $EndComp
 $Comp
-L R R15
+L Device:R R15
 U 1 1 5AC82122
 P 2700 3650
@@
 	0    1    1    0
 $EndComp
+Wire Wire Line
+	3800 1400 3850 1400
+Wire Wire Line
+	2850 1400 3175 1400
+Wire Wire Line
+	3175 1400 3800 1400
+Wire Wire Line
+	2850 1800 2850 1850
+Wire Wire Line
+	3175 1800 3550 1800
+Wire Wire Line
+	3050 3650 3675 3650
+Wire Wire Line
+	3025 2875 3600 2875
+Text HLabel 2725 1400 0    60   Input ~ 0
+8V
+Text HLabel 2400 2325 0    60   Input ~ 0
+L_AUDIO_IN
+Text HLabel 2400 2575 0    60   Input ~ 0
+R_AUDIO_IN
+Text HLabel 2425 2875 0    60   Input ~ 0
+MUTE_AUDIO_AMP
+Text HLabel 5225 1650 2    60   Input ~ 0
+L_AUDIO_OUT+
+Text HLabel 5225 2000 2    60   Input ~ 0
+R_AUDIO_OUT+
+Text HLabel 5225 1750 2    60   Input ~ 0
+L_AUDIO_OUT-
+Text HLabel 5225 2100 2    60   Input ~ 0
+R_AUDIO_OUT-
+Text HLabel 2425 3650 0    60   Input ~ 0
+STBY_AUDIO_AMP
+Connection ~ 3850 1500
+Wire Wire Line
+	3850 1500 3800 1500
+Connection ~ 3850 2000
+Wire Wire Line
+	3850 2000 3450 2000
+Connection ~ 3850 2250
+Wire Wire Line
+	3850 2250 3900 2250
+Connection ~ 3850 2350
+Wire Wire Line
+	3850 2350 3900 2350
+Connection ~ 3850 1800
+Wire Wire Line
+	3850 1800 3900 1800
+Connection ~ 3850 1700
+Wire Wire Line
+	3850 1700 3550 1700
+Connection ~ 3850 2100
+Wire Wire Line
+	3850 2100 3900 2100
+Connection ~ 3850 1400
+Wire Wire Line
+	3850 1400 3900 1400
 $EndSCHEMATC

Commit message: Revert "Merge branch 'lawrence_test' into ethan"
This reverts commit 4dccd689ac590a7d6c1598150e10b9b87c6b396b, reversing
changes made to 5eeefb6d84a8db9381deb81c77fe1ec3b29fea69.
Parts:
- C12, C13, C15, C17: symbol Device:C -> C
- C14, C16: symbol Device:C -> CP
- R14, R15: symbol Device:R -> R
- U8: symbol open-automation:TDA7297 -> TDA7297
Connections:
- wire segments 50 -> 35
Changed lines of the file:
@@
 $Descr A4 11693 8268
 encoding utf-8
-Sheet 7 13
+Sheet 7 11
 Title ""
 Date ""
@@
 $EndDescr
 $Comp
-L open-automation:TDA7297 U8
+L TDA7297 U8
 U 1 1 5AC797FB
 P 4500 1750
@@
 	1    0    0    -1
 $EndComp
-$Comp
-L open-automation:AGND #PWR033
+Text GLabel 2725 1400 0    60   Input ~ 0
+8V
+$Comp
+L AGND #PWR033
 U 1 1 5AC7B29E
 P 3750 1800
@@
 $EndComp
 $Comp
-L open-automation:GND #PWR034
+L GND #PWR034
 U 1 1 5AC7B2BE
 P 2850 1850
@@
 $EndComp
 $Comp
-L Device:C C14
+L CP C14
 U 1 1 5AC7B472
 P 2850 1600
@@
 $EndComp
 $Comp
-L Device:C C17
+L C C17
 U 1 1 5AC7B4BE
 P 3175 1600
@@
 	1    0    0    -1
 $EndComp
-$Comp
-L Device:R R14
+Text GLabel 2425 2875 0    60   Input ~ 0
+MUTE_AUDIO_AMP
+Text GLabel 2425 3650 0    60   Input ~ 0
+STBY_AUDIO_AMP
+$Comp
+L R R14
 U 1 1 5AC7BCAE
 P 2700 2875
@@
 $EndComp
 $Comp
-L open-automation:GND #PWR035
+L GND #PWR035
 U 1 1 5AC7C381
 P 3025 3325
@@
 $EndComp
 $Comp
-L open-automation:GND #PWR036
+L GND #PWR036
 U 1 1 5AC7C45C
 P 3050 4125
@@
 $EndComp
 Wire Wire Line
-	3900 1500 3850 1500
+	3900 1500 3800 1500
 Wire Wire Line
 	3800 1400 3800 1500
 Wire Wire Line
-	2725 1400 2850 1400
+	2725 1400 3900 1400
 Connection ~ 3800 1400
 Wire Wire Line
-	3750 1800 3850 1800
-Wire Wire Line
-	3900 1700 3850 1700
+	3750 1800 3900 1800
+Wire Wire Line
+	3900 1700 3550 1700
 Wire Wire Line
 	2850 1450 2850 1400
@@
 Connection ~ 3175 1400
 Wire Wire Line
-	2850 1750 2850 1800
-Wire Wire Line
-	2850 1800 3175 1800
+	2850 1750 2850 1850
+Wire Wire Line
+	2850 1800 3550 1800
 Wire Wire Line
 	3175 1800 3175 1750
@@
 	2550 2875 2425 2875
 Wire Wire Line
-	2850 3650 3050 3650
+	2850 3650 3675 3650
 Wire Wire Line
 	3050 3650 3050 3725
 Connection ~ 3050 3650
 Wire Wire Line
-	2850 2875 3025 2875
+	2850 2875 3600 2875
 Wire Wire Line
 	3025 2875 3025 2950
@@
 	3050 4025 3050 4125
 Wire Wire Line
-	3675 2350 3850 2350
-Wire Wire Line
-	3600 2250 3850 2250
-$Comp
-L Device:C C12
+	3675 2350 3900 2350
+Wire Wire Line
+	3600 2250 3900 2250
+$Comp
+L C C12
 U 1 1 5AC7CAB7
 P 2750 2325
@@
 	3525 2575 3525 2100
 Wire Wire Line
-	3525 2100 3850 2100
-Wire Wire Line
-	3900 2000 3850 2000
+	3525 2100 3900 2100
+Wire Wire Line
+	3900 2000 3450 2000
 Wire Wire Line
 	3450 2000 3450 2325
@@
 Wire Wire Line
 	2600 2575 2400 2575
+Text GLabel 2400 2325 0    60   Input ~ 0
+L_AUDIO_IN
+Text GLabel 2400 2575 0    60   Input ~ 0
+R_AUDIO_IN
 Wire Wire Line
 	5050 1650 5225 1650
@@
 Wire Wire Line
 	5050 2100 5225 2100
+Text GLabel 5225 1650 2    60   Input ~ 0
+L_AUDIO_OUT+
+Text GLabel 5225 1750 2    60   Input ~ 0
+L_AUDIO_OUT-
+Text GLabel 5225 2000 2    60   Input ~ 0
+R_AUDIO_OUT+
+Text GLabel 5225 2100 2    60   Input ~ 0
+R_AUDIO_OUT-
 Wire Wire Line
 	3600 2875 3600 2250
@@
 	3675 3650 3675 2350
 $Comp
-L Device:C C13
+L C C13
 U 1 1 5AC80604
 P 2750 2575
@@
 $EndComp
 $Comp
-L Device:C C15
+L C C15
 U 1 1 5AC80ED0
 P 3025 3100
@@
 $EndComp
 $Comp
-L Device:C C16
+L CP C16
 U 1 1 5AC81549
 P 3050 3875
@@
 $EndComp
 $Comp
-L Device:R R15
+L R R15
 U 1 1 5AC82122
 P 2700 3650
@@
 	0    1    1    0
 $EndComp
-Wire Wire Line
-	3800 1400 3850 1400
-Wire Wire Line
-	2850 1400 3175 1400
-Wire Wire Line
-	3175 1400 3800 1400
-Wire Wire Line
-	2850 1800 2850 1850
-Wire Wire Line
-	3175 1800 3550 1800
-Wire Wire Line
-	3050 3650 3675 3650
-Wire Wire Line
-	3025 2875 3600 2875
-Text HLabel 2725 1400 0    60   Input ~ 0
-8V
-Text HLabel 2400 2325 0    60   Input ~ 0
-L_AUDIO_IN
-Text HLabel 2400 2575 0    60   Input ~ 0
-R_AUDIO_IN
-Text HLabel 2425 2875 0    60   Input ~ 0
-MUTE_AUDIO_AMP
-Text HLabel 5225 1650 2    60   Input ~ 0
-L_AUDIO_OUT+
-Text HLabel 5225 2000 2    60   Input ~ 0
-R_AUDIO_OUT+
-Text HLabel 5225 1750 2    60   Input ~ 0
-L_AUDIO_OUT-
-Text HLabel 5225 2100 2    60   Input ~ 0
-R_AUDIO_OUT-
-Text HLabel 2425 3650 0    60   Input ~ 0
-STBY_AUDIO_AMP
-Connection ~ 3850 1500
-Wire Wire Line
-	3850 1500 3800 1500
-Connection ~ 3850 2000
-Wire Wire Line
-	3850 2000 3450 2000
-Connection ~ 3850 2250
-Wire Wire Line
-	3850 2250 3900 2250
-Connection ~ 3850 2350
-Wire Wire Line
-	3850 2350 3900 2350
-Connection ~ 3850 1800
-Wire Wire Line
-	3850 1800 3900 1800
-Connection ~ 3850 1700
-Wire Wire Line
-	3850 1700 3550 1700
-Connection ~ 3850 2100
-Wire Wire Line
-	3850 2100 3900 2100
-Connection ~ 3850 1400
-Wire Wire Line
-	3850 1400 3900 1400
 $EndSCHEMATC
