File: audio-amplifier.sch (KiCad schematic (older format))
At the start: 56 parts

Commit message: audio
Connections:
- wire segments 232 -> 234
Changed lines of the file:
@@
 Wire Wire Line
 	3700 6300 3825 6300
+Wire Wire Line
+	5275 4100 5600 4100
+Wire Wire Line
+	5600 4100 5600 4650
+$Comp
+L open-automation:GND #PWR?
+U 1 1 5B6FB0D8
+P 5600 4650
+F 0 "#PWR?" H 5600 4400 50  0001 C CNN
+F 1 "GND" H 5605 4477 50  0000 C CNN
+F 2 "" H 5600 4650 50  0000 C CNN
+F 3 "" H 5600 4650 50  0000 C CNN
+	1    5600 4650
+	1    0    0    -1
+$EndComp
 $EndSCHEMATC

Commit message: almost there
Parts:
- removed C?: C_0.1uF, Capacitor_SMD:C_0603_1608Metric_Pad0.99x1.00mm_HandSolder, symbol open-automation:C_0.1uF
- removed J? (x2): Conn_01x02, Connector_PinHeader_1.00mm:PinHeader_1x02_P1.00mm_Vertical, symbol Connector_Generic:Conn_01x02
- removed LS? (x2): speaker-CVS-1508, open-automation:speaker-1508, symbol open-dash-daughterboard-rescue:speaker-CVS-1508-liger-rescue
- removed R?: R_100k, Resistors_SMD:R_0603_HandSoldering, symbol open-dash-daughterboard-rescue:R_100k-liger-rescue
- removed U?: MAX98357AETE+T, open-automation:MAX98357A, symbol open-dash-daughterboard-rescue:MAX98357AETE+T-liger-rescue
- added Q1, Q2: Q_NPN_BEC, Package_TO_SOT_SMD:SOT-23, symbol open-automation:Q_NPN_BEC
- added R39, R40, R41, R42, R43, R44: R_1k, Resistor_SMD:R_0603_1608Metric_Pad0.99x1.00mm_HandSolder, symbol open-automation:R_1k
- gave numbers to parts that had none: 49
Connections:
- net labels added: 5V
- net labels removed: I2S_DATA_OUT, V_IN
- wire segments 234 -> 228

Commit message: updated corrections
Parts:
- R30: footprint Resistors_SMD:R_0603 -> Resistor_SMD:R_0603_1608Metric_Pad0.99x1.00mm_HandSolder
Changed lines of the file:
@@
 F 0 "R30" H 4325 4275 50  0000 L CNN
 F 1 "R_100k" H 4320 4205 50  0000 L CNN
-F 2 "Resistors_SMD:R_0603" V 4180 4250 50  0001 C CNN
+F 2 "Resistor_SMD:R_0603_1608Metric_Pad0.99x1.00mm_HandSolder" V 4180 4250 50  0001 C CNN
 F 3 "https://www.digikey.com/product-detail/en/yageo/RC0603JR-07100KL/311-100KGRCT-ND/729645" V 4330 4250 50  0001 C CNN
 F 4 "RC0603JR-07100KL" V 4430 4350 60  0001 C CNN "Part Number"

Commit message: traces
Connections:
- net labels added: 3v3
- net labels removed: +3.3V
Changed lines of the file:
@@
-$EndComp
-$Comp
-L open-automation:+3.3V #PWR054
-U 1 1 5B435474
-P 5800 5400
-F 0 "#PWR054" H 5800 5250 50  0001 C CNN
-F 1 "+3.3V" H 5815 5573 50  0000 C CNN
-F 2 "" H 5800 5400 50  0000 C CNN
-F 3 "" H 5800 5400 50  0000 C CNN
-	1    5800 5400
-	1    0    0    -1
 $EndComp
 $Comp
@@
 Connection ~ 5600 5675
 $Comp
-L open-automation:+3.3V #PWR053
-U 1 1 5B463178
-P 5600 5600
-F 0 "#PWR053" H 5600 5450 50  0001 C CNN
-F 1 "+3.3V" H 5600 5725 50  0000 C CNN
-F 2 "" H 5600 5600 50  0000 C CNN
-F 3 "" H 5600 5600 50  0000 C CNN
-	1    5600 5600
-	1    0    0    -1
-$EndComp
-$Comp
 L open-automation:GND #PWR052
 U 1 1 5B46E7FE
@@
 	4175 6875 4250 6875
 $Comp
-L open-automation:+3.3V #PWR046
-U 1 1 5B4C02B5
-P 4175 6850
-F 0 "#PWR046" H 4175 6700 50  0001 C CNN
-F 1 "+3.3V" H 4190 7023 50  0000 C CNN
-F 2 "" H 4175 6850 50  0000 C CNN
-F 3 "" H 4175 6850 50  0000 C CNN
-	1    4175 6850
-	1    0    0    -1
-$EndComp
-$Comp
 L open-automation:C_0.1uF C22
 U 1 1 5B4C0634
@@
 Wire Wire Line
 	5025 5525 5025 5425
-$Comp
-L open-automation:+3.3V #PWR049
-U 1 1 5B5851A6
-P 5025 5425
-F 0 "#PWR049" H 5025 5275 50  0001 C CNN
-F 1 "+3.3V" H 5040 5598 50  0000 C CNN
-F 2 "" H 5025 5425 50  0000 C CNN
-F 3 "" H 5025 5425 50  0000 C CNN
-	1    5025 5425
-	1    0    0    -1
-$EndComp
 $Comp
 L open-automation:C_1uF C29
@@
 	5600 7275 6100 7275
 Connection ~ 6100 7275
+Text HLabel 5800 5400 1    60   Input ~ 0
+3v3
+Text HLabel 5025 5425 1    60   Input ~ 0
+3v3
+Text HLabel 4175 6850 1    60   Input ~ 0
+3v3
+Text HLabel 5600 5600 1    60   Input ~ 0
+3v3
 $EndSCHEMATC
