File: environment.sch (KiCad schematic (older format))
At the start: 0 parts

Commit message: Micro and Environment Schematic Copy
Copied over the microcontroller and environment sheets from smart-regulator project. Also modified the power section.
Parts:
- added C10, C5, C9: C_0.1uF, Capacitors_SMD:C_0603_HandSoldering, symbol C_0.1uF
- added R1: R_10m, Resistors_SMD:R_2512_HandSoldering, symbol R_10m
- added U2: TSL45315CL, smart-regulator:LIGHT-SENSOR-TSL45315CL, symbol TSL45315CL
- added U4: Power-Monitor-INA219, TO_SOT_Packages_SMD:SOT-23-8_Handsoldering, symbol Power-Monitor-INA219
- added U6: SI7020-A20, smart-regulator:SI7020-A20, symbol SI7020-A20
Connections:
- net labels added: 3V3, BATTERY, GND, Light-Level, SCL, SDA, Temp-Humidty, V_MAIN
- wire segments 0 -> 30

Commit message: Backup Before SEPIC Design
Parts:
- U2: footprint smart-regulator:LIGHT-SENSOR-TSL45315CL -> open-automation:LIGHT-SENSOR-TSL45315CL
- U6: footprint smart-regulator:SI7020-A20 -> open-automation:SI7020-A20
Changed lines of the file:
@@
 F 0 "U6" H 2550 1475 60  0000 C CNN
 F 1 "SI7020-A20" H 2350 1775 60  0000 C CNN
-F 2 "smart-regulator:SI7020-A20" H 2350 1275 60  0001 C CNN
+F 2 "open-automation:SI7020-A20" H 2350 1275 60  0001 C CNN
 F 3 "https://www.digikey.com/product-detail/en/silicon-labs/SI7020-A20-GM1R/336-3596-1-ND/5823452" H 2350 1375 60  0001 C CNN
 F 4 "SI7020-A20-GM1R" H 2450 1375 60  0001 C CNN "Part Number"
@@
 F 0 "U2" H 4925 1475 60  0000 C CNN
 F 1 "TSL45315CL" H 4725 1775 60  0000 C CNN
-F 2 "smart-regulator:LIGHT-SENSOR-TSL45315CL" H 4725 1275 60  0001 C CNN
+F 2 "open-automation:LIGHT-SENSOR-TSL45315CL" H 4725 1275 60  0001 C CNN
 F 3 "https://www.digikey.com/product-detail/en/ams/TSL45315CL/TSL45315-CLCT-ND/3095326" H 4725 1375 60  0001 C CNN
 F 4 "TSL45315CL" H 4725 1175 60  0001 C CNN "Part Number"

Commit message: Updated Power Schematic
Power Schematic Updated for 3.3V, 5V, and 8V Buck Regulators. All regulator parts have correct footprints and selected components.

Prelim orgainization of PCB - grouped parts by section.
Parts:
- renumbered C5 to C11, R1 to R9, U6 to U5, U2 to U6, U4 to U7
Changed lines of the file:
@@
 3V3
 $Comp
-L GND #PWR016
+L GND #PWR020
 U 1 1 59C50BD3
 P 1850 1625
-F 0 "#PWR016" H 1850 1375 50  0001 C CNN
+F 0 "#PWR020" H 1850 1375 50  0001 C CNN
 F 1 "GND" H 1850 1475 50  0000 C CNN
 F 2 "" H 1850 1625 50  0000 C CNN
@@
 SDA
 $Comp
-L SI7020-A20 U6
+L SI7020-A20 U5
 U 1 1 59C50BD4
 P 2350 1575
-F 0 "U6" H 2550 1475 60  0000 C CNN
+F 0 "U5" H 2550 1475 60  0000 C CNN
 F 1 "SI7020-A20" H 2350 1775 60  0000 C CNN
 F 2 "open-automation:SI7020-A20" H 2350 1275 60  0001 C CNN
@@
 $EndComp
 $Comp
-L GND #PWR017
+L GND #PWR021
 U 1 1 59C50BD6
 P 1550 1875
-F 0 "#PWR017" H 1550 1625 50  0001 C CNN
+F 0 "#PWR021" H 1550 1625 50  0001 C CNN
 F 1 "GND" H 1550 1725 50  0000 C CNN
 F 2 "" H 1550 1875 50  0000 C CNN
@@
 SCL
 $Comp
-L GND #PWR018
+L GND #PWR022
 U 1 1 59C50BD8
 P 4225 1625
-F 0 "#PWR018" H 4225 1375 50  0001 C CNN
+F 0 "#PWR022" H 4225 1375 50  0001 C CNN
 F 1 "GND" H 4225 1475 50  0000 C CNN
 F 2 "" H 4225 1625 50  0000 C CNN
@@
 Temp-Humidty
 $Comp
-L GND #PWR019
+L GND #PWR023
 U 1 1 59E2A131
 P 4000 1850
-F 0 "#PWR019" H 4000 1600 50  0001 C CNN
+F 0 "#PWR023" H 4000 1600 50  0001 C CNN
 F 1 "GND" H 4000 1700 50  0000 C CNN
 F 2 "" H 4000 1850 50  0000 C CNN
@@
 $EndComp
 $Comp
-L TSL45315CL U2
+L TSL45315CL U6
 U 1 1 59E41F23
 P 4725 1575
-F 0 "U2" H 4925 1475 60  0000 C CNN
+F 0 "U6" H 4925 1475 60  0000 C CNN
 F 1 "TSL45315CL" H 4725 1775 60  0000 C CNN
 F 2 "open-automation:LIGHT-SENSOR-TSL45315CL" H 4725 1275 60  0001 C CNN
@@
 3V3
 $Comp
-L C_0.1uF C5
+L C_0.1uF C11
 U 1 1 5AC2BC67
 P 6475 1725
-F 0 "C5" V 6550 1775 50  0000 L CNN
+F 0 "C11" V 6550 1775 50  0000 L CNN
 F 1 "C_0.1uF" V 6625 1575 50  0000 L CNN
 F 2 "Capacitors_SMD:C_0603_HandSoldering" H 6575 2025 50  0001 C CNN
@@
 $EndComp
 $Comp
-L GND #PWR020
+L GND #PWR024
 U 1 1 5AC2BC6E
 P 6475 1925
-F 0 "#PWR020" H 6475 1675 50  0001 C CNN
+F 0 "#PWR024" H 6475 1675 50  0001 C CNN
 F 1 "GND" V 6550 1850 50  0000 C CNN
 F 2 "" H 6475 1925 50  0000 C CNN
@@
 $EndComp
 $Comp
-L GND #PWR021
+L GND #PWR025
 U 1 1 5AC2BC85
 P 7675 1800
-F 0 "#PWR021" H 7675 1550 50  0001 C CNN
+F 0 "#PWR025" H 7675 1550 50  0001 C CNN
 F 1 "GND" H 7675 1650 50  0000 C CNN
 F 2 "" H 7675 1800 50  0000 C CNN
@@
 SCL
 $Comp
-L Power-Monitor-INA219 U4
+L Power-Monitor-INA219 U7
 U 1 1 5AC2BC90
 P 8200 1625
-F 0 "U4" H 8400 1375 60  0000 C CNN
+F 0 "U7" H 8400 1375 60  0000 C CNN
 F 1 "Power-Monitor-INA219" H 8225 1925 60  0000 C CNN
 F 2 "TO_SOT_Packages_SMD:SOT-23-8_Handsoldering" H 8300 1275 60  0001 C CNN
@@
 $EndComp
 $Comp
-L GND #PWR022
+L GND #PWR026
 U 1 1 5AC2BC97
 P 8800 1450
-F 0 "#PWR022" H 8800 1200 50  0001 C CNN
+F 0 "#PWR026" H 8800 1200 50  0001 C CNN
 F 1 "GND" H 8700 1450 50  0000 C CNN
 F 2 "" H 8800 1450 50  0000 C CNN
@@
 3V3
 $Comp
-L R_10m R1
+L R_10m R9
 U 1 1 5AC2BCA2
 P 7175 1800
-F 0 "R1" H 7150 1800 50  0000 C CNN
+F 0 "R9" H 7150 1800 50  0000 C CNN
 F 1 "R_10m" H 7150 1700 50  0000 C CNN
 F 2 "Resistors_SMD:R_2512_HandSoldering" H 7150 1625 50  0001 C CNN

Commit message: Update Power Schematic and directed parts to open-automation library
Change 3.3V and 5V buck regulator to adjustable chip version.

Directed multiple parts from -cache.lib to open-automation.lib.
Parts:
- removed R9: R_10m, Resistors_SMD:R_2512_HandSoldering, symbol R_10m
- added R13: R_10m, Resistors_SMD:R_2512_HandSoldering, symbol R_10m
Changed lines of the file:
@@
 EESchema Schematic File Version 2
 LIBS:device
+LIBS:open-automation
 LIBS:open-dash-daughterboard-cache
 EELAYER 25 0
@@
 3V3
 $Comp
-L GND #PWR020
+L GND #PWR25
 U 1 1 59C50BD3
 P 1850 1625
-F 0 "#PWR020" H 1850 1375 50  0001 C CNN
+F 0 "#PWR25" H 1850 1375 50  0001 C CNN
 F 1 "GND" H 1850 1475 50  0000 C CNN
 F 2 "" H 1850 1625 50  0000 C CNN
@@
 $EndComp
 $Comp
-L GND #PWR021
+L GND #PWR24
 U 1 1 59C50BD6
 P 1550 1875
-F 0 "#PWR021" H 1550 1625 50  0001 C CNN
+F 0 "#PWR24" H 1550 1625 50  0001 C CNN
 F 1 "GND" H 1550 1725 50  0000 C CNN
 F 2 "" H 1550 1875 50  0000 C CNN
@@
 	1    0    0    -1
 $EndComp
-Text Label 4475 1200 0    60   ~ 0
+Text Label 4475 1250 0    60   ~ 0
 Light-Level
 Text GLabel 5225 1575 2    60   Input ~ 0
@@
 SCL
 $Comp
-L GND #PWR022
+L GND #PWR27
 U 1 1 59C50BD8
 P 4225 1625
-F 0 "#PWR022" H 4225 1375 50  0001 C CNN
+F 0 "#PWR27" H 4225 1375 50  0001 C CNN
 F 1 "GND" H 4225 1475 50  0000 C CNN
 F 2 "" H 4225 1625 50  0000 C CNN
@@
 Temp-Humidty
 $Comp
-L GND #PWR023
+L GND #PWR26
 U 1 1 59E2A131
 P 4000 1850
-F 0 "#PWR023" H 4000 1600 50  0001 C CNN
+F 0 "#PWR26" H 4000 1600 50  0001 C CNN
 F 1 "GND" H 4000 1700 50  0000 C CNN
 F 2 "" H 4000 1850 50  0000 C CNN
 F 3 "" H 4000 1850 50  0000 C CNN
 	1    4000 1850
-	1    0    0    -1
-$EndComp
-$Comp
-L TSL45315CL U6
-U 1 1 59E41F23
-P 4725 1575
-F 0 "U6" H 4925 1475 60  0000 C CNN
-F 1 "TSL45315CL" H 4725 1775 60  0000 C CNN
-F 2 "open-automation:LIGHT-SENSOR-TSL45315CL" H 4725 1275 60  0001 C CNN
-F 3 "https://www.digikey.com/product-detail/en/ams/TSL45315CL/TSL45315-CLCT-ND/3095326" H 4725 1375 60  0001 C CNN
-F 4 "TSL45315CL" H 4725 1175 60  0001 C CNN "Part Number"
-	1    4725 1575
 	1    0    0    -1
 $EndComp
@@
 $EndComp
 $Comp
-L GND #PWR024
+L GND #PWR28
 U 1 1 5AC2BC6E
 P 6475 1925
-F 0 "#PWR024" H 6475 1675 50  0001 C CNN
+F 0 "#PWR28" H 6475 1675 50  0001 C CNN
 F 1 "GND" V 6550 1850 50  0000 C CNN
 F 2 "" H 6475 1925 50  0000 C CNN
@@
 $EndComp
 $Comp
-L GND #PWR025
+L GND #PWR29
 U 1 1 5AC2BC85
 P 7675 1800
-F 0 "#PWR025" H 7675 1550 50  0001 C CNN
+F 0 "#PWR29" H 7675 1550 50  0001 C CNN
 F 1 "GND" H 7675 1650 50  0000 C CNN
 F 2 "" H 7675 1800 50  0000 C CNN
@@
 $EndComp
 $Comp
-L GND #PWR026
+L GND #PWR30
 U 1 1 5AC2BC97
 P 8800 1450
-F 0 "#PWR026" H 8800 1200 50  0001 C CNN
+F 0 "#PWR30" H 8800 1200 50  0001 C CNN
 F 1 "GND" H 8700 1450 50  0000 C CNN
 F 2 "" H 8800 1450 50  0000 C CNN
@@
 Text GLabel 8775 1575 2    60   Input ~ 0
 3V3
-$Comp
-L R_10m R9
-U 1 1 5AC2BCA2
+Wire Wire Line
+	1400 1475 1900 1475
+Wire Wire Line
+	1900 1575 1850 1575
+Wire Wire Line
+	2850 1575 2750 1575
+Wire Wire Line
+	2750 1475 2850 1475
+Wire Wire Line
+	1550 1525 1550 1475
+Connection ~ 1550 1475
+Wire Wire Line
+	1550 1875 1550 1825
+Wire Wire Line
+	1850 1575 1850 1625
+Wire Wire Line
+	4225 1625 4225 1575
+Wire Wire Line
+	4225 1575 4275 1575
+Wire Wire Line
+	3900 1475 4275 1475
+Wire Wire Line
+	4000 1475 4000 1500
+Wire Wire Line
+	4000 1850 4000 1800
+Connection ~ 4000 1475
+Wire Wire Line
+	5225 1575 5125 1575
+Wire Wire Line
+	5125 1475 5225 1475
+Wire Wire Line
+	6200 1475 7725 1475
+Wire Wire Line
+	7350 2000 7350 1675
+Wire Wire Line
+	7675 1800 7675 1775
+Wire Wire Line
+	7675 1775 7725 1775
+Wire Wire Line
+	7100 2000 7350 2000
+Wire Wire Line
+	7175 2000 7175 1925
+Connection ~ 7175 2000
+Wire Wire Line
+	7175 1625 7175 1575
+Connection ~ 7175 1575
+Connection ~ 6475 1475
+Wire Wire Line
+	6475 1925 6475 1875
+Wire Wire Line
+	8650 1475 8800 1475
+Wire Wire Line
+	8775 1675 8650 1675
+Wire Wire Line
+	8775 1775 8650 1775
+Wire Wire Line
+	8800 1475 8800 1450
+Wire Wire Line
+	7100 1575 7725 1575
+Wire Wire Line
+	8775 1575 8650 1575
+Wire Wire Line
+	6475 1475 6475 1575
+Wire Wire Line
+	7350 1675 7725 1675
+$Comp
+L TSL45315CL U6
+U 1 1 5AC75DD5
+P 4725 1575
+F 0 "U6" H 4925 1475 60  0000 C CNN
+F 1 "TSL45315CL" H 4725 1775 60  0000 C CNN
+F 2 "open-automation:LIGHT-SENSOR-TSL45315CL" H 4725 1275 60  0001 C CNN
+F 3 "https://www.digikey.com/product-detail/en/ams/TSL45315CL/TSL45315-CLCT-ND/3095326" H 4725 1375 60  0001 C CNN
+F 4 "TSL45315CL" H 4725 1175 60  0001 C CNN "Part Number"
+	1    4725 1575
+	1    0    0    -1
+$EndComp
+$Comp
+L R_10m R13
+U 1 1 5AC78E3A
 P 7175 1800
-F 0 "R9" H 7150 1800 50  0000 C CNN
+F 0 "R13" H 7150 1800 50  0000 C CNN
 F 1 "R_10m" H 7150 1700 50  0000 C CNN
 F 2 "Resistors_SMD:R_2512_HandSoldering" H 7150 1625 50  0001 C CNN
@@
 	0    1    1    0
 $EndComp
-Wire Wire Line
-	1400 1475 1900 1475
-Wire Wire Line
-	1900 1575 1850 1575
-Wire Wire Line
-	2850 1575 2750 1575
-Wire Wire Line
-	2750 1475 2850 1475
-Wire Wire Line
-	1550 1525 1550 1475
-Connection ~ 1550 1475
-Wire Wire Line
-	1550 1875 1550 1825
-Wire Wire Line
-	1850 1575 1850 1625
-Wire Wire Line
-	4225 1625 4225 1575
-Wire Wire Line
-	4225 1575 4275 1575
-Wire Wire Line
-	3900 1475 4275 1475
-Wire Wire Line
-	4000 1475 4000 1500
-Wire Wire Line
-	4000 1850 4000 1800
-Connection ~ 4000 1475
-Wire Wire Line
-	5225 1575 5125 1575
-Wire Wire Line
-	5125 1475 5225 1475
-Wire Wire Line
-	6200 1475 7725 1475
-Wire Wire Line
-	7350 2000 7350 1675
-Wire Wire Line
-	7675 1800 7675 1775
-Wire Wire Line
-	7675 1775 7725 1775
-Wire Wire Line
-	7100 2000 7350 2000
-Wire Wire Line
-	7175 2000 7175 1925
-Connection ~ 7175 2000
-Wire Wire Line
-	7175 1625 7175 1575
-Connection ~ 7175 1575
-Connection ~ 6475 1475
-Wire Wire Line
-	6475 1925 6475 1875
-Wire Wire Line
-	8650 1475 8800 1475
-Wire Wire Line
-	8775 1675 8650 1675
-Wire Wire Line
-	8775 1775 8650 1775
-Wire Wire Line
-	8800 1475 8800 1450
-Wire Wire Line
-	7100 1575 7725 1575
-Wire Wire Line
-	8775 1575 8650 1575
-Wire Wire Line
-	6475 1475 6475 1575
-Wire Wire Line
-	7350 1675 7725 1675
 $EndSCHEMATC

Commit message: Removed Light Sensor from Enviornment Schematic
Parts:
- removed C10: C_0.1uF, Capacitors_SMD:C_0603_HandSoldering, symbol C_0.1uF
- removed U6: TSL45315CL, open-automation:LIGHT-SENSOR-TSL45315CL, symbol TSL45315CL
Connections:
- net labels removed: Light-Level
- wire segments 30 -> 23
Changed lines of the file:
@@
-	1    0    0    -1
-$EndComp
-Text Label 4475 1250 0    60   ~ 0
-Light-Level
-Text GLabel 5225 1575 2    60   Input ~ 0
-SDA
-Text GLabel 5225 1475 2    60   Input ~ 0
-SCL
-$Comp
-L GND #PWR028
-U 1 1 59C50BD8
-P 4225 1625
-F 0 "#PWR028" H 4225 1375 50  0001 C CNN
-F 1 "GND" H 4225 1475 50  0000 C CNN
-F 2 "" H 4225 1625 50  0000 C CNN
-F 3 "" H 4225 1625 50  0000 C CNN
-	1    4225 1625
-	1    0    0    -1
-$EndComp
-Text GLabel 3900 1475 0    60   Input ~ 0
-3V3
-$Comp
-L C_0.1uF C10
-U 1 1 59C50BDA
-P 4000 1650
-F 0 "C10" H 4025 1750 50  0000 L CNN
-F 1 "C_0.1uF" H 3700 1550 50  0000 L CNN
-F 2 "Capacitors_SMD:C_0603_HandSoldering" H 4100 1950 50  0001 C CNN
-F 3 "https://www.digikey.com/product-detail/en/kemet/C0603C104K5RACTU/399-5089-1-ND/1465623" H 4000 1400 50  0001 C CNN
-F 4 "C0603C104K5RACTU" H 4125 1850 60  0001 C CNN "Part Number"
-	1    4000 1650
 	1    0    0    -1
 $EndComp
 Text Label 2050 1250 0    60   ~ 0
 Temp-Humidty
-$Comp
-L GND #PWR029
-U 1 1 59E2A131
-P 4000 1850
-F 0 "#PWR029" H 4000 1600 50  0001 C CNN
-F 1 "GND" H 4000 1700 50  0000 C CNN
-F 2 "" H 4000 1850 50  0000 C CNN
-F 3 "" H 4000 1850 50  0000 C CNN
-	1    4000 1850
-	1    0    0    -1
-$EndComp
-Text GLabel 7100 1575 0    60   Input ~ 0
+Text GLabel 4825 1525 0    60   Input ~ 0
 BATTERY
-Text GLabel 7100 2000 0    60   Input ~ 0
+Text GLabel 4825 1950 0    60   Input ~ 0
 V_MAIN
-Text GLabel 6200 1475 0    60   Input ~ 0
+Text GLabel 3925 1425 0    60   Input ~ 0
 3V3
 $Comp
 L C_0.1uF C11
 U 1 1 5AC2BC67
-P 6475 1725
-F 0 "C11" V 6550 1775 50  0000 L CNN
-F 1 "C_0.1uF" V 6625 1575 50  0000 L CNN
-F 2 "Capacitors_SMD:C_0603_HandSoldering" H 6575 2025 50  0001 C CNN
-F 3 "https://www.digikey.com/product-detail/en/kemet/C0603C104K5RACTU/399-5089-1-ND/1465623" H 6475 1475 50  0001 C CNN
-F 4 "C0603C104K5RACTU" H 6600 1925 60  0001 C CNN "Part Number"
-	1    6475 1725
+P 4200 1675
+F 0 "C11" V 4275 1725 50  0000 L CNN
+F 1 "C_0.1uF" V 4350 1525 50  0000 L CNN
+F 2 "Capacitors_SMD:C_0603_HandSoldering" H 4300 1975 50  0001 C CNN
+F 3 "https://www.digikey.com/product-detail/en/kemet/C0603C104K5RACTU/399-5089-1-ND/1465623" H 4200 1425 50  0001 C CNN
+F 4 "C0603C104K5RACTU" H 4325 1875 60  0001 C CNN "Part Number"
+	1    4200 1675
 	-1   0    0    1
 $EndComp
@@
 L GND #PWR030
 U 1 1 5AC2BC6E
-P 6475 1925
-F 0 "#PWR030" H 6475 1675 50  0001 C CNN
-F 1 "GND" V 6550 1850 50  0000 C CNN
-F 2 "" H 6475 1925 50  0000 C CNN
-F 3 "" H 6475 1925 50  0000 C CNN
-	1    6475 1925
+P 4200 1875
+F 0 "#PWR030" H 4200 1625 50  0001 C CNN
+F 1 "GND" V 4275 1800 50  0000 C CNN
+F 2 "" H 4200 1875 50  0000 C CNN
+F 3 "" H 4200 1875 50  0000 C CNN
+	1    4200 1875
 	1    0    0    -1
 $EndComp
@@
 L GND #PWR031
 U 1 1 5AC2BC85
-P 7675 1800
-F 0 "#PWR031" H 7675 1550 50  0001 C CNN
-F 1 "GND" H 7675 1650 50  0000 C CNN
-F 2 "" H 7675 1800 50  0000 C CNN
-F 3 "" H 7675 1800 50  0000 C CNN
-	1    7675 1800
+P 5400 1750
+F 0 "#PWR031" H 5400 1500 50  0001 C CNN
+F 1 "GND" H 5400 1600 50  0000 C CNN
+F 2 "" H 5400 1750 50  0000 C CNN
+F 3 "" H 5400 1750 50  0000 C CNN
+	1    5400 1750
 	1    0    0    -1
 $EndComp
-Text GLabel 8775 1675 2    60   Input ~ 0
+Text GLabel 6500 1625 2    60   Input ~ 0
 SDA
-Text GLabel 8775 1775 2    60   Input ~ 0
+Text GLabel 6500 1725 2    60   Input ~ 0
 SCL
 $Comp
 L Power-Monitor-INA219 U7
 U 1 1 5AC2BC90
-P 8200 1625
-F 0 "U7" H 8400 1375 60  0000 C CNN
-F 1 "Power-Monitor-INA219" H 8225 1925 60  0000 C CNN
-F 2 "TO_SOT_Packages_SMD:SOT-23-8_Handsoldering" H 8300 1275 60  0001 C CNN
-F 3 "https://www.digikey.com/product-detail/en/texas-instruments/INA219AIDCNR/296-23770-1-ND/1952550" H 8400 1375 60  0001 C CNN
-F 4 "INA219AIDCNR" H 8500 1475 60  0001 C CNN "Part Number"
-	1    8200 1625
+P 5925 1575
+F 0 "U7" H 6125 1325 60  0000 C CNN
+F 1 "Power-Monitor-INA219" H 5950 1875 60  0000 C CNN
+F 2 "TO_SOT_Packages_SMD:SOT-23-8_Handsoldering" H 6025 1225 60  0001 C CNN
+F 3 "https://www.digikey.com/product-detail/en/texas-instruments/INA219AIDCNR/296-23770-1-ND/1952550" H 6125 1325 60  0001 C CNN
+F 4 "INA219AIDCNR" H 6225 1425 60  0001 C CNN "Part Number"
+	1    5925 1575
 	1    0    0    -1
 $EndComp
@@
 L GND #PWR032
 U 1 1 5AC2BC97
-P 8800 1450
-F 0 "#PWR032" H 8800 1200 50  0001 C CNN
-F 1 "GND" H 8700 1450 50  0000 C CNN
-F 2 "" H 8800 1450 50  0000 C CNN
-F 3 "" H 8800 1450 50  0000 C CNN
-	1    8800 1450
+P 6525 1400
+F 0 "#PWR032" H 6525 1150 50  0001 C CNN
+F 1 "GND" H 6425 1400 50  0000 C CNN
+F 2 "" H 6525 1400 50  0000 C CNN
+F 3 "" H 6525 1400 50  0000 C CNN
+	1    6525 1400
 	-1   0    0    1
 $EndComp
-Text GLabel 8775 1575 2    60   Input ~ 0
+Text GLabel 6500 1525 2    60   Input ~ 0
 3V3
 Wire Wire Line
@@
 	1850 1575 1850 1625
 Wire Wire Line
-	4225 1625 4225 1575
+	3925 1425 5450 1425
 Wire Wire Line
-	4225 1575 4275 1575
+	5075 1950 5075 1625
 Wire Wire Line
-	3900 1475 4275 1475
+	5400 1750 5400 1725
 Wire Wire Line
-	4000 1475 4000 1500
+	5400 1725 5450 1725
 Wire Wire Line
-	4000 1850 4000 1800
-Connection ~ 4000 1475
+	4825 1950 5075 1950
 Wire Wire Line
-	5225 1575 5125 1575
+	4900 1950 4900 1875
+Connection ~ 4900 1950
 Wire Wire Line
-	5125 1475 5225 1475
+	4900 1575 4900 1525
+Connection ~ 4900 1525
+Connection ~ 4200 1425
 Wire Wire Line
-	6200 1475 7725 1475
+	4200 1875 4200 1825
 Wire Wire Line
-	7350 2000 7350 1675
+	6375 1425 6525 1425
 Wire Wire Line
-	7675 1800 7675 1775
+	6500 1625 6375 1625
 Wire Wire Line
-	7675 1775 7725 1775
+	6500 1725 6375 1725
 Wire Wire Line
-	7100 2000 7350 2000
+	6525 1425 6525 1400
 Wire Wire Line
-	7175 2000 7175 1925
-Connection ~ 7175 2000
+	4825 1525 5450 1525
 Wire Wire Line
-	7175 1625 7175 1575
-Connection ~ 7175 1575
-Connection ~ 6475 1475
+	6500 1525 6375 1525
 Wire Wire Line
-	6475 1925 6475 1875
+	4200 1425 4200 1525
 Wire Wire Line
-	8650 1475 8800 1475
-Wire Wire Line
-	8775 1675 8650 1675
-Wire Wire Line
-	8775 1775 8650 1775
-Wire Wire Line
-	8800 1475 8800 1450
-Wire Wire Line
-	7100 1575 7725 1575
-Wire Wire Line
-	8775 1575 8650 1575
-Wire Wire Line
-	6475 1475 6475 1575
-Wire Wire Line
-	7350 1675 7725 1675
-$Comp
-L TSL45315CL U6
-U 1 1 5AC75DD5
-P 4725 1575
-F 0 "U6" H 4925 1475 60  0000 C CNN
-F 1 "TSL45315CL" H 4725 1775 60  0000 C CNN
-F 2 "open-automation:LIGHT-SENSOR-TSL45315CL" H 4725 1275 60  0001 C CNN
-F 3 "https://www.digikey.com/product-detail/en/ams/TSL45315CL/TSL45315-CLCT-ND/3095326" H 4725 1375 60  0001 C CNN
-F 4 "TSL45315CL" H 4725 1175 60  0001 C CNN "Part Number"
-	1    4725 1575
-	1    0    0    -1
-$EndComp
+	5075 1625 5450 1625
 $Comp
 L R_10m R13
 U 1 1 5AC78E3A
-P 7175 1800
-F 0 "R13" H 7150 1800 50  0000 C CNN
-F 1 "R_10m" H 7150 1700 50  0000 C CNN
-F 2 "Resistors_SMD:R_2512_HandSoldering" H 7150 1625 50  0001 C CNN
-F 3 "https://www.digikey.com/product-detail/en/bourns-inc/CRA2512-FZ-R010ELF/CRA2512-FZ-R010ELFCT-ND/1775054" H 7175 1550 50  0001 C CNN
-F 4 "CRA2512-FZ-R010ELF" H 7175 1875 60  0001 C CNN "Part Number"
-	1    7175 1800
+P 4900 1750
+F 0 "R13" H 4875 1750 50  0000 C CNN
+F 1 "R_10m" H 4875 1650 50  0000 C CNN
+F 2 "Resistors_SMD:R_2512_HandSoldering" H 4875 1575 50  0001 C CNN
+F 3 "https://www.digikey.com/product-detail/en/bourns-inc/CRA2512-FZ-R010ELF/CRA2512-FZ-R010ELFCT-ND/1775054" H 4900 1500 50  0001 C CNN
+F 4 "CRA2512-FZ-R010ELF" H 4900 1825 60  0001 C CNN "Part Number"
+	1    4900 1750
 	0    1    1    0
 $EndComp

Commit message: Fixed Ethan Branch to actually merge "lawrence_test" branch
Had some clinfict issues that were handeled incorrectly. Problems now fixed.
Parts:
- C11, C9: symbol C_0.1uF -> open-automation:C_0.1uF
- R13: symbol R_10m -> open-automation:R_10m
- U5: symbol SI7020-A20 -> open-automation:SI7020-A20
- U7: symbol Power-Monitor-INA219 -> open-automation:Power-Monitor-INA219
Connections:
- wire segments 23 -> 27
Changed lines of the file:
@@
-EESchema Schematic File Version 2
-LIBS:device
-LIBS:open-automation
+EESchema Schematic File Version 4
 LIBS:open-dash-daughterboard-cache
-EELAYER 25 0
+EELAYER 26 0
 EELAYER END
-$Descr A4 11693 8268
+$Descr USLetter 11000 8500
 encoding utf-8
-Sheet 6 11
+Sheet 6 13
 Title ""
 Date ""
@@
 Comment4 ""
 $EndDescr
-Text GLabel 1400 1475 0    60   Input ~ 0
-3V3
-$Comp
-L GND #PWR026
+$Comp
+L open-automation:GND #PWR026
 U 1 1 59C50BD3
 P 1850 1625
@@
 	1    0    0    -1
 $EndComp
-Text GLabel 2850 1475 2    60   Input ~ 0
-SCL
-Text GLabel 2850 1575 2    60   Input ~ 0
-SDA
-$Comp
-L SI7020-A20 U5
+$Comp
+L open-automation:SI7020-A20 U5
 U 1 1 59C50BD4
 P 2350 1575
@@
 $EndComp
 $Comp
-L C_0.1uF C9
+L open-automation:C_0.1uF C9
 U 1 1 59C50BD5
 P 1550 1675
@@
 $EndComp
 $Comp
-L GND #PWR027
+L open-automation:GND #PWR027
 U 1 1 59C50BD6
 P 1550 1875
@@
 Text Label 2050 1250 0    60   ~ 0
 Temp-Humidty
-Text GLabel 4825 1525 0    60   Input ~ 0
-BATTERY
-Text GLabel 4825 1950 0    60   Input ~ 0
-V_MAIN
-Text GLabel 3925 1425 0    60   Input ~ 0
-3V3
-$Comp
-L C_0.1uF C11
+$Comp
+L open-automation:C_0.1uF C11
 U 1 1 5AC2BC67
 P 4200 1675
@@
 $EndComp
 $Comp
-L GND #PWR030
+L open-automation:GND #PWR030
 U 1 1 5AC2BC6E
 P 4200 1875
@@
 $EndComp
 $Comp
-L GND #PWR031
+L open-automation:GND #PWR031
 U 1 1 5AC2BC85
 P 5400 1750
@@
 	1    0    0    -1
 $EndComp
-Text GLabel 6500 1625 2    60   Input ~ 0
-SDA
-Text GLabel 6500 1725 2    60   Input ~ 0
-SCL
-$Comp
-L Power-Monitor-INA219 U7
+$Comp
+L open-automation:Power-Monitor-INA219 U7
 U 1 1 5AC2BC90
 P 5925 1575
@@
 $EndComp
 $Comp
-L GND #PWR032
+L open-automation:GND #PWR032
 U 1 1 5AC2BC97
 P 6525 1400
@@
 	-1   0    0    1
 $EndComp
-Text GLabel 6500 1525 2    60   Input ~ 0
-3V3
-Wire Wire Line
-	1400 1475 1900 1475
+Wire Wire Line
+	1400 1475 1550 1475
 Wire Wire Line
 	1900 1575 1850 1575
@@
 	1850 1575 1850 1625
 Wire Wire Line
-	3925 1425 5450 1425
+	3925 1425 4200 1425
 Wire Wire Line
 	5075 1950 5075 1625
@@
 	5400 1725 5450 1725
 Wire Wire Line
-	4825 1950 5075 1950
+	4825 1950 4900 1950
 Wire Wire Line
 	4900 1950 4900 1875
@@
 	6525 1425 6525 1400
 Wire Wire Line
-	4825 1525 5450 1525
+	4825 1525 4900 1525
 Wire Wire Line
 	6500 1525 6375 1525
@@
 	5075 1625 5450 1625
 $Comp
-L R_10m R13
+L open-automation:R_10m R13
 U 1 1 5AC78E3A
 P 4900 1750
@@
 	0    1    1    0
 $EndComp
+Wire Wire Line
+	1550 1475 1900 1475
+Wire Wire Line
+	4900 1950 5075 1950
+Wire Wire Line
+	4900 1525 5450 1525
+Wire Wire Line
+	4200 1425 5450 1425
+Text HLabel 1400 1475 0    60   Input ~ 0
+3V3
+Text HLabel 2850 1475 2    60   Input ~ 0
+SCL
+Text HLabel 2850 1575 2    60   Input ~ 0
+SDA
+Text HLabel 3925 1425 0    60   Input ~ 0
+3V3
+Text HLabel 4825 1525 0    60   Input ~ 0
+BATTERY
+Text HLabel 4825 1950 0    60   Input ~ 0
+V_MAIN
+Text HLabel 6500 1525 2    60   Input ~ 0
+3V3
+Text HLabel 6500 1625 2    60   Input ~ 0
+SDA
+Text HLabel 6500 1725 2    60   Input ~ 0
+SCL
 $EndSCHEMATC
