File: environment.sch (KiCad schematic (older format))
At the start: 5 parts, among them U10 Power-Monitor-INA219, U9 SI7020-A20

Commit message: almost there
Parts:
- gave numbers to parts that had none: 1
- renumbered C18 to C16, C19 to C17, U9 to U8, U10 to U9
Changed lines of the file:
@@
 $Descr USLetter 11000 8500
 encoding utf-8
-Sheet 6 13
+Sheet 6 12
 Title ""
 Date ""
@@
 $EndDescr
 $Comp
-L open-automation:GND #PWR037
+L open-automation:GND #PWR040
 U 1 1 59C50BD3
 P 3325 3550
-F 0 "#PWR037" H 3325 3300 50  0001 C CNN
+F 0 "#PWR040" H 3325 3300 50  0001 C CNN
 F 1 "GND" H 3325 3400 50  0000 C CNN
 F 2 "" H 3325 3550 50  0000 C CNN
@@
 $EndComp
 $Comp
-L open-automation:SI7020-A20 U9
+L open-automation:SI7020-A20 U8
 U 1 1 59C50BD4
 P 3825 3500
-F 0 "U9" H 4025 3400 60  0000 C CNN
+F 0 "U8" H 4025 3400 60  0000 C CNN
 F 1 "SI7020-A20" H 3825 3700 60  0000 C CNN
 F 2 "open-automation:SI7020-A20" H 3825 3200 60  0001 C CNN
@@
 $EndComp
 $Comp
-L open-automation:GND #PWR036
+L open-automation:GND #PWR039
 U 1 1 59C50BD6
 P 3050 3800
-F 0 "#PWR036" H 3050 3550 50  0001 C CNN
+F 0 "#PWR039" H 3050 3550 50  0001 C CNN
 F 1 "GND" H 3050 3650 50  0000 C CNN
 F 2 "" H 3050 3800 50  0000 C CNN
@@
 Temp-Humidty
 $Comp
-L open-automation:GND #PWR038
+L open-automation:GND #PWR041
 U 1 1 5AC2BC6E
 P 5600 3800
-F 0 "#PWR038" H 5600 3550 50  0001 C CNN
+F 0 "#PWR041" H 5600 3550 50  0001 C CNN
 F 1 "GND" V 5675 3725 50  0000 C CNN
 F 2 "" H 5600 3800 50  0000 C CNN
@@
 $EndComp
 $Comp
-L open-automation:GND #PWR039
+L open-automation:GND #PWR042
 U 1 1 5AC2BC85
 P 6875 3675
-F 0 "#PWR039" H 6875 3425 50  0001 C CNN
+F 0 "#PWR042" H 6875 3425 50  0001 C CNN
 F 1 "GND" H 6875 3525 50  0000 C CNN
 F 2 "" H 6875 3675 50  0000 C CNN
@@
 $EndComp
 $Comp
-L open-automation:GND #PWR040
+L open-automation:GND #PWR043
 U 1 1 5AC2BC97
 P 8000 3325
-F 0 "#PWR040" H 8000 3075 50  0001 C CNN
+F 0 "#PWR043" H 8000 3075 50  0001 C CNN
 F 1 "GND" H 7900 3325 50  0000 C CNN
 F 2 "" H 8000 3325 50  0000 C CNN
@@
 SCL
 $Comp
-L open-automation:C_0.1uF C18
+L open-automation:C_0.1uF C16
 U 1 1 5B22240F
 P 3050 3600
-F 0 "C18" H 3165 3646 50  0000 L CNN
+F 0 "C16" H 3165 3646 50  0000 L CNN
 F 1 "C_0.1uF" H 3165 3555 50  0000 L CNN
 F 2 "Capacitor_SMD:C_0603_1608Metric_Pad0.99x1.00mm_HandSolder" H 3150 3900 50  0001 C CNN
@@
 	3050 3750 3050 3800
 $Comp
-L open-automation:C_0.1uF C19
+L open-automation:C_0.1uF C17
 U 1 1 5B223737
 P 5600 3600
-F 0 "C19" H 5715 3646 50  0000 L CNN
+F 0 "C17" H 5715 3646 50  0000 L CNN
 F 1 "C_0.1uF" H 5715 3555 50  0000 L CNN
 F 2 "Capacitor_SMD:C_0603_1608Metric_Pad0.99x1.00mm_HandSolder" H 5700 3900 50  0001 C CNN
@@
 	5600 3350 6925 3350
 $Comp
-L open-automation:Power-Monitor-INA219 U10
+L open-automation:Power-Monitor-INA219 U9
 U 1 1 5B2C37F2
 P 7400 3500
-F 0 "U10" H 7387 3897 60  0000 C CNN
+F 0 "U9" H 7387 3897 60  0000 C CNN
 F 1 "Power-Monitor-INA219" H 7387 3791 60  0000 C CNN
 F 2 "TO_SOT_Packages_SMD:SOT-23-8_Handsoldering" H 7500 3150 60  0001 C CNN
@@
 $EndComp
 $Comp
-L open-automation:R_10m R?
+L open-automation:R_10m R26
 U 1 1 5B3C5EA6
 P 6375 3675
-F 0 "R?" V 6304 3745 50  0000 L CNN
+F 0 "R26" V 6304 3745 50  0000 L CNN
 F 1 "R_10m" V 6395 3745 50  0000 L CNN
 F 2 "Resistors_SMD:R_2512_HandSoldering" H 6350 3500 50  0001 C CNN

Commit message: updated corrections
Parts:
- R26: footprint Resistors_SMD:R_2512_HandSoldering -> Resistor_SMD:R_2512_6332Metric_Pad1.49x3.40mm_HandSolder
- U9: footprint TO_SOT_Packages_SMD:SOT-23-8_Handsoldering -> Package_TO_SOT_SMD:SOT-23-8_Handsoldering
Changed lines of the file:
@@
 F 0 "U9" H 7387 3897 60  0000 C CNN
 F 1 "Power-Monitor-INA219" H 7387 3791 60  0000 C CNN
-F 2 "TO_SOT_Packages_SMD:SOT-23-8_Handsoldering" H 7500 3150 60  0001 C CNN
+F 2 "Package_TO_SOT_SMD:SOT-23-8_Handsoldering" H 7500 3150 60  0001 C CNN
 F 3 "https://www.digikey.com/product-detail/en/texas-instruments/INA219AIDCNT/296-26073-1-ND/2254846" H 7600 3250 60  0001 C CNN
 F 4 "INA219AIDCNT" H 7700 3350 60  0001 C CNN "Part Number"
@@
 F 0 "R26" V 6304 3745 50  0000 L CNN
 F 1 "R_10m" V 6395 3745 50  0000 L CNN
-F 2 "Resistors_SMD:R_2512_HandSoldering" H 6350 3500 50  0001 C CNN
+F 2 "Resistor_SMD:R_2512_6332Metric_Pad1.49x3.40mm_HandSolder" H 6350 3500 50  0001 C CNN
 F 3 "https://www.digikey.com/product-detail/en/bourns-inc/CRA2512-FZ-R010ELF/CRA2512-FZ-R010ELFCT-ND/1775054" H 6375 3425 50  0001 C CNN
 F 4 "CRA2512-FZ-R010ELF" H 6375 3750 60  0001 C CNN "Part Number"
