File: GPS interface.sch (KiCad schematic (older format))
At the start: 3 parts

Commit message: dangling commit
Parts:
- U?: symbol dk_RF-Receivers:A2235-H -> open-dash-daughterboard-rescue:A2235-H-dk_RF-Receivers
Changed lines of the file:
@@
 SCL
 $Comp
-L dk_RF-Receivers:A2235-H U?
+L open-dash-daughterboard-rescue:A2235-H-dk_RF-Receivers U?
 U 1 1 5AE2F0AB
 P 9150 3250

Commit message: adding and cleaning lables
Connections:
- net labels added: GPS_Ant
- wire segments 23 -> 24
Changed lines of the file:
@@
 Wire Wire Line
 	6850 3600 8200 3600
+Text HLabel 8050 3850 0    50   Input ~ 0
+GPS_Ant
+Wire Wire Line
+	8350 3850 8050 3850
 $EndSCHEMATC
