File: switches.sch (KiCad schematic (older format))
At the start: 12 parts, among them P5 USB_A_2, U10 touchpad, U4 housing-mounts

Commit message: added footprints  and merged from main branch and
Parts:
- D2, D3, D5: symbol open-automation:LED -> open-dash-daughterboard-rescue:LED-open-automation
- FACTORY1, PROG1, REBOOT1: symbol open-automation:SW_PUSH -> open-dash-daughterboard-rescue:SW_PUSH-open-automation
- P5: symbol open-automation:USB_A_2 -> open-dash-daughterboard-rescue:USB_A_2-open-automation
- R2, R3, R4: symbol open-automation:R_10k -> open-dash-daughterboard-rescue:R_10k-open-automation
- U10: symbol open-automation:touchpad -> open-dash-daughterboard-rescue:touchpad-open-automation
- U4: symbol open-automation:housing-mounts -> open-dash-daughterboard-rescue:housing-mounts-open-automation
Changed lines of the file:
@@
 EESchema Schematic File Version 4
+LIBS:open-dash-daughterboard-cache
 EELAYER 26 0
 EELAYER END
@@
 $EndDescr
 $Comp
-L open-automation:LED D2
+L open-dash-daughterboard-rescue:LED-open-automation D2
 U 1 1 59092D24
 P 3225 3325
@@
 $EndComp
 $Comp
-L open-automation:touchpad U10
+L open-dash-daughterboard-rescue:touchpad-open-automation U10
 U 1 1 590F8D3B
 P 7950 4800
@@
 $EndComp
 $Comp
-L open-automation:USB_A_2 P5
+L open-dash-daughterboard-rescue:USB_A_2-open-automation P5
 U 1 1 59693837
 P 7850 3000
@@
 $EndComp
 $Comp
-L open-automation:GND #PWR0121
+L open-dash-daughterboard-rescue:GND-open-automation #PWR0121
 U 1 1 5969393D
 P 8000 3400
@@
 	7400 3400 7350 3400
 $Comp
-L open-automation:housing-mounts U4
+L open-dash-daughterboard-rescue:housing-mounts-open-automation U4
 U 1 1 5978A2A6
 P 7925 4225
@@
 $EndComp
 $Comp
-L open-automation:SW_PUSH FACTORY1
+L open-dash-daughterboard-rescue:SW_PUSH-open-automation FACTORY1
 U 1 1 59C587B8
 P 3225 4175
@@
 $EndComp
 $Comp
-L open-automation:GND #PWR0122
+L open-dash-daughterboard-rescue:GND-open-automation #PWR0122
 U 1 1 59C59092
 P 3225 4550
@@
 	3225 4550 3225 4475
 $Comp
-L open-automation:R_10k R2
+L open-dash-daughterboard-rescue:R_10k-open-automation R2
 U 1 1 59E3E4D2
 P 3225 3675
@@
 Connection ~ 3225 3850
 $Comp
-L open-automation:LED D3
+L open-dash-daughterboard-rescue:LED-open-automation D3
 U 1 1 59E3EE41
 P 4175 3325
@@
 $EndComp
 $Comp
-L open-automation:SW_PUSH REBOOT1
+L open-dash-daughterboard-rescue:SW_PUSH-open-automation REBOOT1
 U 1 1 59E3EE49
 P 4175 4175
@@
 $EndComp
 $Comp
-L open-automation:GND #PWR0123
+L open-dash-daughterboard-rescue:GND-open-automation #PWR0123
 U 1 1 59E3EE50
 P 4175 4550
@@
 	4175 4550 4175 4475
 $Comp
-L open-automation:R_10k R3
+L open-dash-daughterboard-rescue:R_10k-open-automation R3
 U 1 1 59E3EE58
 P 4175 3675
@@
 Connection ~ 4175 3850
 $Comp
-L open-automation:LED D5
+L open-dash-daughterboard-rescue:LED-open-automation D5
 U 1 1 59E3F1C3
 P 5000 3325
@@
 $EndComp
 $Comp
-L open-automation:SW_PUSH PROG1
+L open-dash-daughterboard-rescue:SW_PUSH-open-automation PROG1
 U 1 1 59E3F1CB
 P 5000 4175
@@
 $EndComp
 $Comp
-L open-automation:GND #PWR0124
+L open-dash-daughterboard-rescue:GND-open-automation #PWR0124
 U 1 1 59E3F1D2
 P 5000 4550
@@
 	5000 4550 5000 4475
 $Comp
-L open-automation:R_10k R4
+L open-dash-daughterboard-rescue:R_10k-open-automation R4
 U 1 1 59E3F1DA
 P 5000 3675
