File: switches.sch (KiCad schematic (older format))
At the start: 12 parts, among them P5 USB_A_2, U10 touchpad, U4 housing-mounts

Commit message: update
Connections:
- net labels added: 3v3
- net labels removed: 3V3
Changed lines of the file:
@@
 EESchema Schematic File Version 4
+LIBS:open-dash-daughterboard-cache
 EELAYER 26 0
 EELAYER END
 $Descr USLetter 11000 8500
 encoding utf-8
-Sheet 12 15
+Sheet 12 14
 Title ""
 Date ""
@@
 $Comp
 L open-automation:GND #PWR0121
-U 1 1 5969393D
+U 1 1 5B1799B0
 P 8000 3400
 F 0 "#PWR0121" H 8000 3150 50  0001 C CNN
@@
 $Comp
 L open-automation:housing-mounts U4
-U 1 1 5978A2A6
+U 1 1 5B1799B1
 P 7925 4225
 F 0 "U4" H 8075 4125 60  0000 C CNN
@@
 $Comp
 L open-automation:GND #PWR0122
-U 1 1 59C59092
+U 1 1 5B1799B3
 P 3225 4550
 F 0 "#PWR0122" H 3225 4300 50  0001 C CNN
@@
 $Comp
 L open-automation:GND #PWR0124
-U 1 1 59E3F1D2
+U 1 1 5B1799BB
 P 5000 4550
 F 0 "#PWR0124" H 5000 4300 50  0001 C CNN
@@
 PROG
 Text HLabel 4175 3125 1    60   Input ~ 0
-3V3
+3v3
 Text HLabel 5000 3125 1    60   Input ~ 0
-3V3
+3v3
 Text HLabel 3225 3125 1    60   Input ~ 0
-3V3
+3v3
 $EndSCHEMATC
