File: audio-interface.sch (KiCad schematic (older format))
At the start: 21 parts

Commit message: organizing
Parts:
- gave numbers to parts that had none: 21
Changed lines of the file:
@@
 $EndDescr
 $Comp
-L open-automation:CM108AH U?
+L open-automation:CM108AH U13
 U 1 1 5AE40241
 P 5575 3675
-F 0 "U?" H 5600 5490 50  0000 C CNN
+F 0 "U13" H 5600 5490 50  0000 C CNN
 F 1 "CM108AH" H 5600 5399 50  0000 C CNN
 F 2 "" H 5575 3675 50  0001 C CNN
@@
 5v
 $Comp
-L Device:C_Small C?
+L Device:C_Small C51
 U 1 1 5AE44C69
 P 4075 2150
-F 0 "C?" H 4167 2196 50  0000 L CNN
+F 0 "C51" H 4167 2196 50  0000 L CNN
 F 1 "4.7uF" H 4167 2105 50  0000 L CNN
 F 2 "" H 4075 2150 50  0001 C CNN
@@
 	4075 2250 4075 2300
 $Comp
-L open-automation:GND #PWR?
+L open-automation:GND #PWR0138
 U 1 1 5AE44DC5
 P 4075 2350
-F 0 "#PWR?" H 4075 2100 50  0001 C CNN
+F 0 "#PWR0138" H 4075 2100 50  0001 C CNN
 F 1 "GND" H 4200 2275 50  0000 C CNN
 F 2 "" H 4075 2350 50  0000 C CNN
@@
 	4075 2300 4500 2300
 $Comp
-L Device:C_Small C?
+L Device:C_Small C52
 U 1 1 5AE457CC
 P 4500 2150
-F 0 "C?" H 4592 2196 50  0000 L CNN
+F 0 "C52" H 4592 2196 50  0000 L CNN
 F 1 "0.1uF" H 4592 2105 50  0000 L CNN
 F 2 "" H 4500 2150 50  0001 C CNN
@@
 5v
 $Comp
-L Device:C_Small C?
+L Device:C_Small C45
 U 1 1 5AE45EF6
 P 3075 2675
-F 0 "C?" H 3167 2721 50  0000 L CNN
+F 0 "C45" H 3167 2721 50  0000 L CNN
 F 1 "4.7uF" H 3167 2630 50  0000 L CNN
 F 2 "" H 3075 2675 50  0001 C CNN
@@
 	3075 2825 3500 2825
 $Comp
-L Device:C_Small C?
+L Device:C_Small C47
 U 1 1 5AE45F0B
 P 3500 2675
-F 0 "C?" H 3592 2721 50  0000 L CNN
+F 0 "C47" H 3592 2721 50  0000 L CNN
 F 1 "0.1uF" H 3592 2630 50  0000 L CNN
 F 2 "" H 3500 2675 50  0001 C CNN
@@
 	4875 2625 4875 2725
 $Comp
-L Device:C_Small C?
+L Device:C_Small C49
 U 1 1 5AE48B66
 P 3700 2975
-F 0 "C?" H 3775 3050 50  0000 L CNN
+F 0 "C49" H 3775 3050 50  0000 L CNN
 F 1 "4.7uF" H 3775 2975 50  0000 L CNN
 F 2 "" H 3700 2975 50  0001 C CNN
@@
 $EndComp
 $Comp
-L open-automation:GND #PWR?
+L open-automation:GND #PWR0139
 U 1 1 5AE48D0C
 P 4800 2325
-F 0 "#PWR?" H 4800 2075 50  0001 C CNN
+F 0 "#PWR0139" H 4800 2075 50  0001 C CNN
 F 1 "GND" V 4900 2275 50  0000 C CNN
 F 2 "" H 4800 2325 50  0000 C CNN
@@
 $EndComp
 $Comp
-L open-automation:AGND #PWR?
+L open-automation:AGND #PWR0140
 U 1 1 5AE49217
 P 4825 2625
-F 0 "#PWR?" H 4825 2375 50  0001 C CNN
+F 0 "#PWR0140" H 4825 2375 50  0001 C CNN
 F 1 "AGND" V 4925 2650 50  0000 R CNN
 F 2 "" H 4825 2625 50  0000 C CNN
@@
 	3700 2875 3700 2825
 $Comp
-L open-automation:AGND #PWR?
+L open-automation:AGND #PWR0141
 U 1 1 5AE4B09D
 P 3075 2875
-F 0 "#PWR?" H 3075 2625 50  0001 C CNN
+F 0 "#PWR0141" H 3075 2625 50  0001 C CNN
 F 1 "AGND" H 3325 2800 50  0000 R CNN
 F 2 "" H 3075 2875 50  0000 C CNN
@@
 $EndComp
 $Comp
-L open-automation:GND #PWR?
+L open-automation:GND #PWR0142
 U 1 1 5AE4B108
 P 3700 3225
-F 0 "#PWR?" H 3700 2975 50  0001 C CNN
+F 0 "#PWR0142" H 3700 2975 50  0001 C CNN
 F 1 "GND" H 3825 3150 50  0000 C CNN
 F 2 "" H 3700 3225 50  0000 C CNN
@@
 	3700 3225 3700 3075
 $Comp
-L Device:C_Small C?
+L Device:C_Small C50
 U 1 1 5AE4B5C6
 P 4025 3050
-F 0 "C?" H 4100 3100 50  0000 L CNN
+F 0 "C50" H 4100 3100 50  0000 L CNN
 F 1 "4.7uF" H 4100 3000 50  0000 L CNN
 F 2 "" H 4025 3050 50  0001 C CNN
@@
 $EndComp
 $Comp
-L Device:Crystal_Small Y?
+L Device:Crystal_Small Y2
 U 1 1 5AE4DDD9
 P 4750 3125
-F 0 "Y?" V 4800 3075 50  0000 R CNN
+F 0 "Y2" V 4800 3075 50  0000 R CNN
 F 1 "12MHz" V 4700 3075 50  0000 R CNN
 F 2 "" H 4750 3125 50  0001 C CNN
@@
 $EndComp
 $Comp
-L Device:C_Small C?
+L Device:C_Small C54
 U 1 1 5AE4EE03
 P 4550 3225
-F 0 "C?" V 4500 3125 50  0000 C CNN
+F 0 "C54" V 4500 3125 50  0000 C CNN
 F 1 "?" V 4600 3100 50  0000 C CNN
 F 2 "" H 4550 3225 50  0001 C CNN
@@
 $EndComp
 $Comp
-L Device:C_Small C?
+L Device:C_Small C53
 U 1 1 5AE50258
 P 4550 3000
-F 0 "C?" V 4500 2925 50  0000 C CNN
+F 0 "C53" V 4500 2925 50  0000 C CNN
 F 1 "?" V 4600 2925 50  0000 C CNN
 F 2 "" H 4550 3000 50  0001 C CNN
@@
 	4975 2000 4500 2000
 $Comp
-L Device:R_Small R?
+L Device:R_Small R36
 U 1 1 5AE684BB
 P 4500 3425
-F 0 "R?" V 4425 3425 50  0000 C CNN
+F 0 "R36" V 4425 3425 50  0000 C CNN
 F 1 "22" V 4575 3425 50  0000 C CNN
 F 2 "" V 4430 3425 50  0001 C CNN
@@
 	4600 3425 4975 3425
 $Comp
-L Device:R_Small R?
+L Device:R_Small R35
 U 1 1 5AE6995C
 P 4275 3525
-F 0 "R?" V 4200 3525 50  0000 C CNN
+F 0 "R35" V 4200 3525 50  0000 C CNN
 F 1 "22" V 4350 3525 50  0000 C CNN
 F 2 "" V 4205 3525 50  0001 C CNN
@@
 	2475 3525 2650 3525
 $Comp
-L Device:C_Small C?
+L Device:C_Small C46
 U 1 1 5AE6F10A
 P 3375 3675
-F 0 "C?" H 3450 3725 50  0000 L CNN
+F 0 "C46" H 3450 3725 50  0000 L CNN
 F 1 "47pF" H 3450 3625 50  0000 L CNN
 F 2 "" H 3375 3675 50  0001 C CNN
@@
 $EndComp
 $Comp
-L Device:C_Small C?
+L Device:C_Small C48
 U 1 1 5AE6F180
 P 3650 3675
-F 0 "C?" H 3725 3725 50  0000 L CNN
+F 0 "C48" H 3725 3725 50  0000 L CNN
 F 1 "47pF" H 3725 3625 50  0000 L CNN
 F 2 "" H 3650 3675 50  0001 C CNN
@@
 	3650 3425 4400 3425
 $Comp
-L open-automation:GND #PWR?
+L open-automation:GND #PWR0143
 U 1 1 5AE70A91
 P 3375 3850
-F 0 "#PWR?" H 3375 3600 50  0001 C CNN
+F 0 "#PWR0143" H 3375 3600 50  0001 C CNN
 F 1 "GND" H 3500 3775 50  0000 C CNN
 F 2 "" H 3375 3850 50  0000 C CNN
@@
 	3650 3850 3375 3850
 $Comp
-L Device:R_Small R?
+L Device:R_Small R34
 U 1 1 5AE72A98
 P 3225 3225
-F 0 "R?" V 3150 3225 50  0000 C CNN
+F 0 "R34" V 3150 3225 50  0000 C CNN
 F 1 "1k5" V 3300 3225 50  0000 C CNN
 F 2 "" V 3155 3225 50  0001 C CNN
@@
 audio_mute
 $Comp
-L open-automation:GND #PWR?
+L open-automation:GND #PWR0144
 U 1 1 5AE90C70
 P 4875 4325
-F 0 "#PWR?" H 4875 4075 50  0001 C CNN
+F 0 "#PWR0144" H 4875 4075 50  0001 C CNN
 F 1 "GND" H 5000 4250 50  0000 C CNN
 F 2 "" H 4875 4325 50  0000 C CNN
@@
 	4875 4825 4875 4925
 $Comp
-L open-automation:GND #PWR?
+L open-automation:GND #PWR0145
 U 1 1 5AEA5FA4
 P 4875 4925
-F 0 "#PWR?" H 4875 4675 50  0001 C CNN
+F 0 "#PWR0145" H 4875 4675 50  0001 C CNN
 F 1 "GND" H 5000 4850 50  0000 C CNN
 F 2 "" H 4875 4925 50  0000 C CNN
@@
 NoConn ~ 6225 3125
 $Comp
-L Device:CP_Small C?
+L Device:CP_Small C55
 U 1 1 5AEB573A
 P 6575 3225
-F 0 "C?" V 6625 3125 50  0000 C CNN
+F 0 "C55" V 6625 3125 50  0000 C CNN
 F 1 "470uF" V 6525 3075 50  0000 C CNN
 F 2 "" H 6575 3225 50  0001 C CNN
@@
 	6225 3225 6475 3225
 $Comp
-L Device:CP_Small C?
+L Device:CP_Small C56
 U 1 1 5AEBA252
 P 6875 3325
-F 0 "C?" V 6925 3225 50  0000 C CNN
+F 0 "C56" V 6925 3225 50  0000 C CNN
 F 1 "470uF" V 6825 3150 50  0000 C CNN
 F 2 "" H 6875 3325 50  0001 C CNN
@@
 NoConn ~ 6225 4425
 $Comp
-L Device:R_Small R?
+L Device:R_Small R37
 U 1 1 5AED144E
 P 6475 4325
-F 0 "R?" V 6400 4325 50  0000 C CNN
+F 0 "R37" V 6400 4325 50  0000 C CNN
 F 1 "?" V 6550 4325 50  0000 C CNN
 F 2 "" V 6405 4325 50  0001 C CNN
@@
 	6225 4325 6375 4325
 $Comp
-L open-automation:LED D?
+L open-automation:LED D11
 U 1 1 5AED9DFE
 P 6825 4325
-F 0 "D?" H 6825 4125 50  0000 C CNN
+F 0 "D11" H 6825 4125 50  0000 C CNN
 F 1 "LED" H 6825 4200 50  0000 C CNN
 F 2 "" H 6825 4325 50  0000 C CNN
@@
 	7100 4325 7100 4400
 $Comp
-L open-automation:GND #PWR?
+L open-automation:GND #PWR0146
 U 1 1 5AEDD835
 P 7100 4400
-F 0 "#PWR?" H 7100 4150 50  0001 C CNN
+F 0 "#PWR0146" H 7100 4150 50  0001 C CNN
 F 1 "GND" H 7225 4325 50  0000 C CNN
 F 2 "" H 7100 4400 50  0000 C CNN
@@
 dac_data_out
 $Comp
-L Device:D_TVS_ALT D?
+L Device:D_TVS_ALT D10
 U 1 1 5AEF3F02
 P 3025 3700
-F 0 "D?" V 2979 3779 50  0000 L CNN
+F 0 "D10" V 2979 3779 50  0000 L CNN
 F 1 "D_TVS" V 3070 3779 50  0000 L CNN
 F 2 "" H 3025 3700 50  0001 C CNN
@@
 $EndComp
 $Comp
-L Device:D_TVS_ALT D?
+L Device:D_TVS_ALT D9
 U 1 1 5AEF3F99
 P 2650 3700
-F 0 "D?" V 2604 3779 50  0000 L CNN
+F 0 "D9" V 2604 3779 50  0000 L CNN
 F 1 "D_TVS" V 2695 3779 50  0000 L CNN
 F 2 "" H 2650 3700 50  0001 C CNN

Commit message: added footprints  and merged from main branch and
Parts:
- C45, C46, C47, C48, C49, C50, C51, C52, C53, C54: footprint (none) -> Capacitors_SMD:C_0603_HandSoldering
- C55, C56: footprint (none) -> Capacitors_SMD:CP_Elec_5x4.5
- D11: footprint (none) -> smart-regulator:LED_0603; symbol open-automation:LED -> open-dash-daughterboard-rescue:LED-open-automation
- R34, R35, R36, R37: footprint (none) -> smart-regulator:R_0603_HandSoldering
- U13: symbol open-automation:CM108AH -> open-dash-daughterboard-rescue:CM108AH-open-automation
Changed lines of the file:
@@
 EESchema Schematic File Version 4
+LIBS:open-dash-daughterboard-cache
 EELAYER 26 0
 EELAYER END
@@
 $EndDescr
 $Comp
-L open-automation:CM108AH U13
+L open-dash-daughterboard-rescue:CM108AH-open-automation U13
 U 1 1 5AE40241
 P 5575 3675
@@
 F 0 "C51" H 4167 2196 50  0000 L CNN
 F 1 "4.7uF" H 4167 2105 50  0000 L CNN
-F 2 "" H 4075 2150 50  0001 C CNN
+F 2 "Capacitors_SMD:C_0603_HandSoldering" H 4075 2150 50  0001 C CNN
 F 3 "" H 4075 2150 50  0001 C CNN
 	1    4075 2150
@@
 	4075 2250 4075 2300
 $Comp
-L open-automation:GND #PWR0138
+L open-dash-daughterboard-rescue:GND-open-automation #PWR0138
 U 1 1 5AE44DC5
 P 4075 2350
@@
 F 0 "C52" H 4592 2196 50  0000 L CNN
 F 1 "0.1uF" H 4592 2105 50  0000 L CNN
-F 2 "" H 4500 2150 50  0001 C CNN
+F 2 "Capacitors_SMD:C_0603_HandSoldering" H 4500 2150 50  0001 C CNN
 F 3 "" H 4500 2150 50  0001 C CNN
 	1    4500 2150
@@
 F 0 "C45" H 3167 2721 50  0000 L CNN
 F 1 "4.7uF" H 3167 2630 50  0000 L CNN
-F 2 "" H 3075 2675 50  0001 C CNN
+F 2 "Capacitors_SMD:C_0603_HandSoldering" H 3075 2675 50  0001 C CNN
 F 3 "" H 3075 2675 50  0001 C CNN
 	1    3075 2675
@@
 F 0 "C47" H 3592 2721 50  0000 L CNN
 F 1 "0.1uF" H 3592 2630 50  0000 L CNN
-F 2 "" H 3500 2675 50  0001 C CNN
+F 2 "Capacitors_SMD:C_0603_HandSoldering" H 3500 2675 50  0001 C CNN
 F 3 "" H 3500 2675 50  0001 C CNN
 	1    3500 2675
@@
 F 0 "C49" H 3775 3050 50  0000 L CNN
 F 1 "4.7uF" H 3775 2975 50  0000 L CNN
-F 2 "" H 3700 2975 50  0001 C CNN
+F 2 "Capacitors_SMD:C_0603_HandSoldering" H 3700 2975 50  0001 C CNN
 F 3 "" H 3700 2975 50  0001 C CNN
 	1    3700 2975
@@
 $EndComp
 $Comp
-L open-automation:GND #PWR0139
+L open-dash-daughterboard-rescue:GND-open-automation #PWR0139
 U 1 1 5AE48D0C
 P 4800 2325
@@
 $EndComp
 $Comp
-L open-automation:AGND #PWR0140
+L open-dash-daughterboard-rescue:AGND-open-automation #PWR0140
 U 1 1 5AE49217
 P 4825 2625
@@
 	3700 2875 3700 2825
 $Comp
-L open-automation:AGND #PWR0141
+L open-dash-daughterboard-rescue:AGND-open-automation #PWR0141
 U 1 1 5AE4B09D
 P 3075 2875
@@
 $EndComp
 $Comp
-L open-automation:GND #PWR0142
+L open-dash-daughterboard-rescue:GND-open-automation #PWR0142
 U 1 1 5AE4B108
 P 3700 3225
@@
 F 0 "C50" H 4100 3100 50  0000 L CNN
 F 1 "4.7uF" H 4100 3000 50  0000 L CNN
-F 2 "" H 4025 3050 50  0001 C CNN
+F 2 "Capacitors_SMD:C_0603_HandSoldering" H 4025 3050 50  0001 C CNN
 F 3 "" H 4025 3050 50  0001 C CNN
 	1    4025 3050
@@
 F 0 "C54" V 4500 3125 50  0000 C CNN
 F 1 "?" V 4600 3100 50  0000 C CNN
-F 2 "" H 4550 3225 50  0001 C CNN
+F 2 "Capacitors_SMD:C_0603_HandSoldering" H 4550 3225 50  0001 C CNN
 F 3 "" H 4550 3225 50  0001 C CNN
 	1    4550 3225
@@
 F 0 "C53" V 4500 2925 50  0000 C CNN
 F 1 "?" V 4600 2925 50  0000 C CNN
-F 2 "" H 4550 3000 50  0001 C CNN
+F 2 "Capacitors_SMD:C_0603_HandSoldering" H 4550 3000 50  0001 C CNN
 F 3 "" H 4550 3000 50  0001 C CNN
 	1    4550 3000
@@
 F 0 "R36" V 4425 3425 50  0000 C CNN
 F 1 "22" V 4575 3425 50  0000 C CNN
-F 2 "" V 4430 3425 50  0001 C CNN
+F 2 "smart-regulator:R_0603_HandSoldering" V 4430 3425 50  0001 C CNN
 F 3 "" H 4500 3425 50  0001 C CNN
 	1    4500 3425
@@
 F 0 "R35" V 4200 3525 50  0000 C CNN
 F 1 "22" V 4350 3525 50  0000 C CNN
-F 2 "" V 4205 3525 50  0001 C CNN
+F 2 "smart-regulator:R_0603_HandSoldering" V 4205 3525 50  0001 C CNN
 F 3 "" H 4275 3525 50  0001 C CNN
 	1    4275 3525
@@
 F 0 "C46" H 3450 3725 50  0000 L CNN
 F 1 "47pF" H 3450 3625 50  0000 L CNN
-F 2 "" H 3375 3675 50  0001 C CNN
+F 2 "Capacitors_SMD:C_0603_HandSoldering" H 3375 3675 50  0001 C CNN
 F 3 "" H 3375 3675 50  0001 C CNN
 	1    3375 3675
@@
 F 0 "C48" H 3725 3725 50  0000 L CNN
 F 1 "47pF" H 3725 3625 50  0000 L CNN
-F 2 "" H 3650 3675 50  0001 C CNN
+F 2 "Capacitors_SMD:C_0603_HandSoldering" H 3650 3675 50  0001 C CNN
 F 3 "" H 3650 3675 50  0001 C CNN
 	1    3650 3675
@@
 	3650 3425 4400 3425
 $Comp
-L open-automation:GND #PWR0143
+L open-dash-daughterboard-rescue:GND-open-automation #PWR0143
 U 1 1 5AE70A91
 P 3375 3850
@@
 F 0 "R34" V 3150 3225 50  0000 C CNN
 F 1 "1k5" V 3300 3225 50  0000 C CNN
-F 2 "" V 3155 3225 50  0001 C CNN
+F 2 "smart-regulator:R_0603_HandSoldering" V 3155 3225 50  0001 C CNN
 F 3 "" H 3225 3225 50  0001 C CNN
 	1    3225 3225
@@
 audio_mute
 $Comp
-L open-automation:GND #PWR0144
+L open-dash-daughterboard-rescue:GND-open-automation #PWR0144
 U 1 1 5AE90C70
 P 4875 4325
@@
 	4875 4825 4875 4925
 $Comp
-L open-automation:GND #PWR0145
+L open-dash-daughterboard-rescue:GND-open-automation #PWR0145
 U 1 1 5AEA5FA4
 P 4875 4925
@@
 F 0 "C55" V 6625 3125 50  0000 C CNN
 F 1 "470uF" V 6525 3075 50  0000 C CNN
-F 2 "" H 6575 3225 50  0001 C CNN
+F 2 "Capacitors_SMD:CP_Elec_5x4.5" H 6575 3225 50  0001 C CNN
 F 3 "" H 6575 3225 50  0001 C CNN
 	1    6575 3225
@@
 F 0 "C56" V 6925 3225 50  0000 C CNN
 F 1 "470uF" V 6825 3150 50  0000 C CNN
-F 2 "" H 6875 3325 50  0001 C CNN
+F 2 "Capacitors_SMD:CP_Elec_5x4.5" H 6875 3325 50  0001 C CNN
 F 3 "" H 6875 3325 50  0001 C CNN
 	1    6875 3325
@@
 F 0 "R37" V 6400 4325 50  0000 C CNN
 F 1 "?" V 6550 4325 50  0000 C CNN
-F 2 "" V 6405 4325 50  0001 C CNN
+F 2 "smart-regulator:R_0603_HandSoldering" V 6405 4325 50  0001 C CNN
 F 3 "" H 6475 4325 50  0001 C CNN
 	1    6475 4325
@@
 	6225 4325 6375 4325
 $Comp
-L open-automation:LED D11
+L open-dash-daughterboard-rescue:LED-open-automation D11
 U 1 1 5AED9DFE
 P 6825 4325
 F 0 "D11" H 6825 4125 50  0000 C CNN
 F 1 "LED" H 6825 4200 50  0000 C CNN
-F 2 "" H 6825 4325 50  0000 C CNN
+F 2 "smart-regulator:LED_0603" H 6825 4325 50  0001 C CNN
 F 3 "" H 6825 4325 50  0000 C CNN
 	1    6825 4325
@@
 	7100 4325 7100 4400
 $Comp
-L open-automation:GND #PWR0146
+L open-dash-daughterboard-rescue:GND-open-automation #PWR0146
 U 1 1 5AEDD835
 P 7100 4400

Commit message: added new parts and started layout
Parts:
- U13: footprint (none) -> smart-regulator:QFP-48_7x7_Pitch0.5mm
Changed lines of the file:
@@
 F 0 "U13" H 5600 5490 50  0000 C CNN
 F 1 "CM108AH" H 5600 5399 50  0000 C CNN
-F 2 "" H 5575 3675 50  0001 C CNN
+F 2 "smart-regulator:QFP-48_7x7_Pitch0.5mm" H 5575 3675 50  0001 C CNN
 F 3 "" H 5575 3675 50  0001 C CNN
 	1    5575 3675
