File: _autosave-open-dash-daughterboard.kicad_pcb (KiCad board)
At the start: 2 copper layers, 150.1 x 127 mm, 110 parts, among them P5 USB_A_2, Q1 Q_NPN_BEC, Q2 Q_NJFET_DGS, Q3 Q_NJFET_DGS, U1 LM2576-ADJ, U10 touchpad, U14 ESP-WROOM-32, U2 LM2576-ADJ, U3 LM2576-ADJ, U4 housing-mounts, U5 SI7020-A20, U6 MCP2515-E_ST, U7 Power-Monitor-INA219, U8 TDA7297, U9 MCP2551-I_SN, Y1 16MHz

Commit message: update
Connections:
- net /mainboard-interface/3V3 renamed /mainboard-interface/3v3
- net /microcontroller/FACTORY renamed /FACTORY
- net /microcontroller/IO2 renamed Net-(R12-Pad2)
- net /microcontroller/MUTE_AUDIO_AMP renamed /MUTE_AUDIO_AMP
- net /microcontroller/PROG renamed /PROG
- net /microcontroller/RXD renamed /RXD
- net /microcontroller/SOFT_POWER renamed /SOFT_POWER
- net /microcontroller/STBY_AUDIO_AMP renamed /STBY_AUDIO_AMP
- net /microcontroller/TXD renamed /TXD
- net /power/AUDIO_POWER renamed /AUDIO_POWER
- net /power/MAIN_POWER renamed /MAIN_POWER
- net /power/V_MAIN renamed /V_MAIN
- net /switches/3V3 renamed /switches/3v3
- C1 pad 1: /power/BATTERY -> /BATTERY
- C3 pad 1: /power/BATTERY -> /BATTERY
- C4 pad 1: /power/3V3 -> /3v3
- C7 pad 1: /microcontroller/3V3 -> /3v3
- C8 pad 1: /microcontroller/3V3 -> /3v3
- D1 pad 1: /power/BATTERY -> /BATTERY
- D14 pad 2: /power/3V3 -> /3v3
- L1 pad 2: /power/3V3 -> /3v3
- R1 pad 1: /power/3V3 -> /3v3
- R1 pad 2: /power/EN_MAIN -> /EN_MAIN
- R10 pad 2: /microcontroller/3V3 -> /3v3
- R11 pad 2: /microcontroller/3V3 -> /3v3
- R39 pad 1: /power/3V3 -> /3v3
- R39 pad 2: /power/EN_AUDIO -> /EN_AUDIO
- R40 pad 1: /power/3V3 -> /3v3
- U1 pad 1: /power/BATTERY -> /BATTERY
- U14 pad 2: /microcontroller/3V3 -> /3v3
- U14 pad 27: /microcontroller/EN_AUDIO -> /EN_AUDIO
- U14 pad 30: /microcontroller/EN_MAIN -> /EN_MAIN
- U2 pad 5: /power/EN_MAIN -> /EN_MAIN
- U3 pad 1: /power/BATTERY -> /BATTERY
- U3 pad 5: /power/EN_AUDIO -> /EN_AUDIO
