File: interface.sch (KiCad schematic (older format))
At the start: 15 parts, among them J1 Conn_01x02, J2 Conn_01x02, P1 USB_A_2, U13 molex-2x4-5.7mm, U15 molex-2x4-5.7mm, U16 housing-mounts

Commit message: update
Parts:
- added P1, P2: CONN-BARREL-2x5.5mm, open-automation:CONN-BARREL_PJ-037A, symbol open-automation:CONN-BARREL-2x5.5mm
- D10: renamed from D9; footprint LEDs:LED_0603_HandSoldering -> LED_SMD:LED_0603_1608Metric_Pad0.82x1.00mm_HandSolder
- D11: renamed from D10; footprint LEDs:LED_0603_HandSoldering -> LED_SMD:LED_0603_1608Metric_Pad0.82x1.00mm_HandSolder
- D12: renamed from D11; footprint LEDs:LED_0603_HandSoldering -> LED_SMD:LED_0603_1608Metric_Pad0.82x1.00mm_HandSolder
- R38: renamed from R34; footprint Resistors_SMD:R_0603_HandSoldering -> Resistor_SMD:R_0603_1608Metric_Pad0.99x1.00mm_HandSolder
- R39: renamed from R35; footprint Resistors_SMD:R_0603_HandSoldering -> Resistor_SMD:R_0603_1608Metric_Pad0.99x1.00mm_HandSolder
- R40: renamed from R36; footprint Resistors_SMD:R_0603_HandSoldering -> Resistor_SMD:R_0603_1608Metric_Pad0.99x1.00mm_HandSolder
- renumbered FACTORY2 to FACTORY1, J1 to J4, J2 to J5, P1 to P3, PROG2 to PROG1, REBOOT2 to REBOOT1, U13 to U14
Connections:
- net labels added: 5V, DISPLAY_POWER, MAIN_POWER, SOFT_POWER
- net labels removed: V_USB
- wire segments 49 -> 56
Changed lines of the file:
@@
 $Descr A 11000 8500
 encoding utf-8
-Sheet 14 14
+Sheet 14 13
 Title ""
 Date ""
@@
 $EndDescr
 $Comp
-L Connector_Generic:Conn_01x02 J1
+L Connector_Generic:Conn_01x02 J4
 U 1 1 5AE24043
 P 8175 950
-F 0 "J1" H 8255 942 50  0000 L CNN
+F 0 "J4" H 8255 942 50  0000 L CNN
 F 1 "Conn_01x02" H 8255 851 50  0000 L CNN
 F 2 "" H 8175 950 50  0001 C CNN
@@
 $EndComp
 $Comp
-L Connector_Generic:Conn_01x02 J2
+L Connector_Generic:Conn_01x02 J5
 U 1 1 5AE240A7
 P 8225 1650
-F 0 "J2" H 8305 1642 50  0000 L CNN
+F 0 "J5" H 8305 1642 50  0000 L CNN
 F 1 "Conn_01x02" H 8305 1551 50  0000 L CNN
 F 2 "" H 8225 1650 50  0001 C CNN
@@
 GPS Antenna
 $Comp
-L power:GNDA #PWR0101
+L power:GNDA #PWR073
 U 1 1 5AE24110
 P 7775 1150
-F 0 "#PWR0101" H 7775 900 50  0001 C CNN
+F 0 "#PWR073" H 7775 900 50  0001 C CNN
 F 1 "GNDA" H 7780 977 50  0000 C CNN
 F 2 "" H 7775 1150 50  0001 C CNN
@@
 $EndComp
 $Comp
-L power:GNDA #PWR0111
+L power:GNDA #PWR074
 U 1 1 5AE24128
 P 7875 1850
-F 0 "#PWR0111" H 7875 1600 50  0001 C CNN
+F 0 "#PWR074" H 7875 1600 50  0001 C CNN
 F 1 "GNDA" H 7880 1677 50  0000 C CNN
 F 2 "" H 7875 1850 50  0001 C CNN
@@
 LF_AUDIO_OUT-
 $Comp
-L open-dash-daughterboard-rescue:LED-open-automation D9
+L open-dash-daughterboard-rescue:LED-open-automation D10
 U 1 1 5B1799AD
 P 1975 3750
-F 0 "D9" V 1950 3850 50  0000 C CNN
+F 0 "D10" V 1950 3850 50  0000 C CNN
 F 1 "LED" V 2075 3675 50  0000 C CNN
-F 2 "LEDs:LED_0603_HandSoldering" H 1975 3750 50  0001 C CNN
+F 2 "LED_SMD:LED_0603_1608Metric_Pad0.82x1.00mm_HandSolder" H 1975 3750 50  0001 C CNN
 F 3 "http://www.osram-os.com/Graphics/XPic9/00128792_0.pdf" H 1975 3750 50  0001 C CNN
 F 4 "475-2512-2-ND" H 1975 3750 60  0001 C CNN "Part Number"
@@
 $EndComp
 $Comp
-L open-automation:USB_A_2 P1
+L open-automation:USB_A_2 P3
 U 1 1 5B1799AF
 P 7850 3000
-F 0 "P1" H 8100 2800 50  0000 C CNN
+F 0 "P3" H 8100 2800 50  0000 C CNN
 F 1 "USB_A_2" H 7800 3200 50  0000 C CNN
 F 2 "open-automation:USB_A_2" V 7800 2900 50  0001 C CNN
@@
 $EndComp
 $Comp
-L open-automation:GND #PWR0112
+L open-automation:GND #PWR075
 U 1 1 5969393D
 P 8000 3400
-F 0 "#PWR0112" H 8000 3150 50  0001 C CNN
+F 0 "#PWR075" H 8000 3150 50  0001 C CNN
 F 1 "GND" H 8000 3250 50  0000 C CNN
 F 2 "" H 8000 3400 50  0000 C CNN
@@
 $EndComp
 $Comp
-L open-automation:SW_PUSH FACTORY2
+L open-automation:SW_PUSH FACTORY1
 U 1 1 5B1799B2
 P 1975 4600
-F 0 "FACTORY2" H 1975 4775 50  0000 C CNN
+F 0 "FACTORY1" H 1975 4775 50  0000 C CNN
 F 1 "SW_PUSH" H 1975 4520 50  0000 C CNN
 F 2 "Buttons_Switches_SMD:SW_SPST_KMR2" H 1975 4600 50  0001 C CNN
@@
 $EndComp
 $Comp
-L open-automation:GND #PWR0113
+L open-automation:GND #PWR067
 U 1 1 59C59092
 P 1975 4975
-F 0 "#PWR0113" H 1975 4725 50  0001 C CNN
+F 0 "#PWR067" H 1975 4725 50  0001 C CNN
 F 1 "GND" H 1975 4825 50  0000 C CNN
 F 2 "" H 1975 4975 50  0000 C CNN
@@
 	1975 4975 1975 4900
 $Comp
-L open-automation:R_10k R34
+L open-automation:R_10k R38
 U 1 1 5B1799B4
 P 1975 4100
-F 0 "R34" V 1975 4100 50  0000 C CNN
+F 0 "R38" V 1975 4100 50  0000 C CNN
 F 1 "R_10k" V 1875 4100 50  0000 C CNN
-F 2 "Resistors_SMD:R_0603_HandSoldering" V 1905 4100 50  0001 C CNN
+F 2 "Resistor_SMD:R_0603_1608Metric_Pad0.99x1.00mm_HandSolder" V 1905 4100 50  0001 C CNN
 F 3 "https://www.digikey.com/product-detail/en/yageo/RC0603JR-0710KL/311-10KGRCT-ND/729647" V 2055 4100 50  0001 C CNN
 F 4 "RC0603JR-0710KL" V 2155 4200 60  0001 C CNN "Part Number"
@@
 Connection ~ 1975 4275
 $Comp
-L open-dash-daughterboard-rescue:LED-open-automation D10
+L open-dash-daughterboard-rescue:LED-open-automation D11
 U 1 1 5B1799B5
 P 2925 3750
-F 0 "D10" V 2900 3850 50  0000 C CNN
+F 0 "D11" V 2900 3850 50  0000 C CNN
 F 1 "LED" V 3025 3675 50  0000 C CNN
-F 2 "LEDs:LED_0603_HandSoldering" H 2925 3750 50  0001 C CNN
+F 2 "LED_SMD:LED_0603_1608Metric_Pad0.82x1.00mm_HandSolder" H 2925 3750 50  0001 C CNN
 F 3 "http://www.osram-os.com/Graphics/XPic9/00128792_0.pdf" H 2925 3750 50  0001 C CNN
 F 4 "475-2512-2-ND" H 2925 3750 60  0001 C CNN "Part Number"
@@
 $EndComp
 $Comp
-L open-automation:SW_PUSH REBOOT2
+L open-automation:SW_PUSH REBOOT1
 U 1 1 5B1799B6
 P 2925 4600
-F 0 "REBOOT2" H 2925 4775 50  0000 C CNN
+F 0 "REBOOT1" H 2925 4775 50  0000 C CNN
 F 1 "SW_PUSH" H 2925 4520 50  0000 C CNN
 F 2 "Buttons_Switches_SMD:SW_SPST_KMR2" H 2925 4600 50  0001 C CNN
@@
 $EndComp
 $Comp
-L open-automation:GND #PWR0117
+L open-automation:GND #PWR069
 U 1 1 5B1799B7
 P 2925 4975
-F 0 "#PWR0117" H 2925 4725 50  0001 C CNN
+F 0 "#PWR069" H 2925 4725 50  0001 C CNN
 F 1 "GND" H 2925 4825 50  0000 C CNN
 F 2 "" H 2925 4975 50  0000 C CNN
@@
 	2925 4975 2925 4900
 $Comp
-L open-automation:R_10k R35
+L open-automation:R_10k R39
 U 1 1 5B1799B8
 P 2925 4100
-F 0 "R35" V 2925 4100 50  0000 C CNN
+F 0 "R39" V 2925 4100 50  0000 C CNN
 F 1 "R_10k" V 2825 4100 50  0000 C CNN
-F 2 "Resistors_SMD:R_0603_HandSoldering" V 2855 4100 50  0001 C CNN
+F 2 "Resistor_SMD:R_0603_1608Metric_Pad0.99x1.00mm_HandSolder" V 2855 4100 50  0001 C CNN
 F 3 "https://www.digikey.com/product-detail/en/yageo/RC0603JR-0710KL/311-10KGRCT-ND/729647" V 3005 4100 50  0001 C CNN
 F 4 "RC0603JR-0710KL" V 3105 4200 60  0001 C CNN "Part Number"
@@
 Connection ~ 2925 4275
 $Comp
-L open-dash-daughterboard-rescue:LED-open-automation D11
+L open-dash-daughterboard-rescue:LED-open-automation D12
 U 1 1 5B1799B9
 P 3750 3750
-F 0 "D11" V 3725 3850 50  0000 C CNN
+F 0 "D12" V 3725 3850 50  0000 C CNN
 F 1 "LED" V 3850 3675 50  0000 C CNN
-F 2 "LEDs:LED_0603_HandSoldering" H 3750 3750 50  0001 C CNN
+F 2 "LED_SMD:LED_0603_1608Metric_Pad0.82x1.00mm_HandSolder" H 3750 3750 50  0001 C CNN
 F 3 "http://www.osram-os.com/Graphics/XPic9/00128792_0.pdf" H 3750 3750 50  0001 C CNN
 F 4 "475-2512-2-ND" H 3750 3750 60  0001 C CNN "Part Number"
@@
 $EndComp
 $Comp
-L open-automation:SW_PUSH PROG2
+L open-automation:SW_PUSH PROG1
 U 1 1 5B1799BA
 P 3750 4600
-F 0 "PROG2" H 3750 4775 50  0000 C CNN
+F 0 "PROG1" H 3750 4775 50  0000 C CNN
 F 1 "SW_PUSH" H 3750 4520 50  0000 C CNN
 F 2 "Buttons_Switches_SMD:SW_SPST_KMR2" H 3750 4600 50  0001 C CNN
@@
 $EndComp
 $Comp
-L open-automation:GND #PWR0118
+L open-automation:GND #PWR070
 U 1 1 59E3F1D2
 P 3750 4975
-F 0 "#PWR0118" H 3750 4725 50  0001 C CNN
+F 0 "#PWR070" H 3750 4725 50  0001 C CNN
 F 1 "GND" H 3750 4825 50  0000 C CNN
 F 2 "" H 3750 4975 50  0000 C CNN
@@
 	3750 4975 3750 4900
 $Comp
-L open-automation:R_10k R36
+L open-automation:R_10k R40
 U 1 1 5B1799BC
 P 3750 4100
-F 0 "R36" V 3750 4100 50  0000 C CNN
+F 0 "R40" V 3750 4100 50  0000 C CNN
 F 1 "R_10k" V 3650 4100 50  0000 C CNN
-F 2 "Resistors_SMD:R_0603_HandSoldering" V 3680 4100 50  0001 C CNN
+F 2 "Resistor_SMD:R_0603_1608Metric_Pad0.99x1.00mm_HandSolder" V 3680 4100 50  0001 C CNN
 F 3 "https://www.digikey.com/product-detail/en/yageo/RC0603JR-0710KL/311-10KGRCT-ND/729647" V 3830 4100 50  0001 C CNN
 F 4 "RC0603JR-0710KL" V 3930 4200 60  0001 C CNN "Part Number"
@@
 	3750 4275 3750 4300
 Text HLabel 7350 3400 0    60   Input ~ 0
-V_USB
+5V
 Text HLabel 7550 3400 3    60   Input ~ 0
 TXD
@@
 3v3
 $Comp
-L open-automation:molex-2x4-5.7mm U13
+L open-automation:molex-2x4-5.7mm U14
 U 1 1 5B1A08B0
 P 2425 1900
-F 0 "U13" H 2425 2150 50  0000 C CNN
+F 0 "U14" H 2425 2150 50  0000 C CNN
 F 1 "molex-2x4-5.7mm" H 2450 1650 50  0000 C CNN
 F 2 "open-automation:molex-2x4-5.7mm" H 2425 1500 50  0001 C CNN
@@
 	5000 1775 4950 1775
 $Comp
-L open-automation:GND #PWR0138
+L open-automation:GND #PWR068
 U 1 1 5B1DA0DF
 P 2675 1750
-F 0 "#PWR0138" H 2675 1500 50  0001 C CNN
+F 0 "#PWR068" H 2675 1500 50  0001 C CNN
 F 1 "GND" V 2650 1575 50  0000 C CNN
 F 2 "" H 2675 1750 50  0000 C CNN
@@
 	0    -1   -1   0
 $EndComp
+Text HLabel 2175 1850 0    50   Input ~ 0
+SOFT_POWER
+Wire Wire Line
+	2225 1850 2175 1850
+$Comp
+L open-automation:CONN-BARREL-2x5.5mm P1
+U 1 1 5B0FBD41
+P 7700 4900
+F 0 "P1" H 7777 4941 50  0000 L CNN
+F 1 "CONN-BARREL-2x5.5mm" H 7777 4850 50  0000 L CNN
+F 2 "open-automation:CONN-BARREL_PJ-037A" H 7700 4650 50  0001 C CNN
+F 3 "https://www.digikey.com/product-detail/en/cui-inc/PJ-037A/CP-037A-ND/1644545" H 7700 4600 50  0001 C CNN
+F 4 "PJ-037A" H 7700 4500 50  0001 C CNN "Part Number"
+	1    7700 4900
+	1    0    0    -1
+$EndComp
+$Comp
+L open-automation:CONN-BARREL-2x5.5mm P2
+U 1 1 5B0FBEBD
+P 7700 5400
+F 0 "P2" H 7777 5441 50  0000 L CNN
+F 1 "CONN-BARREL-2x5.5mm" H 7777 5350 50  0000 L CNN
+F 2 "open-automation:CONN-BARREL_PJ-037A" H 7700 5150 50  0001 C CNN
+F 3 "https://www.digikey.com/product-detail/en/cui-inc/PJ-037A/CP-037A-ND/1644545" H 7700 5100 50  0001 C CNN
+F 4 "PJ-037A" H 7700 5000 50  0001 C CNN "Part Number"
+	1    7700 5400
+	1    0    0    -1
+$EndComp
+$Comp
+L open-automation:GND #PWR072
+U 1 1 5B0FC9F0
+P 7475 5475
+F 0 "#PWR072" H 7475 5225 50  0001 C CNN
+F 1 "GND" H 7475 5325 50  0000 C CNN
+F 2 "" H 7475 5475 50  0000 C CNN
+F 3 "" H 7475 5475 50  0000 C CNN
+	1    7475 5475
+	1    0    0    -1
+$EndComp
+Wire Wire Line
+	7475 5475 7475 5450
+Wire Wire Line
+	7475 5450 7500 5450
+$Comp
+L open-automation:GND #PWR071
+U 1 1 5B0FE113
+P 7475 4975
+F 0 "#PWR071" H 7475 4725 50  0001 C CNN
+F 1 "GND" H 7475 4825 50  0000 C CNN
+F 2 "" H 7475 4975 50  0000 C CNN
+F 3 "" H 7475 4975 50  0000 C CNN
+	1    7475 4975
+	1    0    0    -1
+$EndComp
+Wire Wire Line
+	7475 4975 7475 4950
+Wire Wire Line
+	7475 4950 7500 4950
+Text HLabel 7450 4850 0    60   Input ~ 0
+DISPLAY_POWER
+Wire Wire Line
+	7450 4850 7500 4850
+Text HLabel 7450 5350 0    60   Input ~ 0
+MAIN_POWER
+Wire Wire Line
+	7450 5350 7500 5350
 $EndSCHEMATC

Commit message: update
Parts:
- removed J4: Conn_01x02, symbol Connector_Generic:Conn_01x02
- removed R39: R_10k, Resistor_SMD:R_0603_1608Metric_Pad0.99x1.00mm_HandSolder, symbol open-automation:R_10k
- removed U16: housing-mounts, open-automation:enclosure-25x38, symbol open-automation:housing-mounts
- added J4: Conn_02x06_Odd_Even, symbol Connector_Generic:Conn_02x06_Odd_Even
- added J5: USB_B, open-automation:USB_B-B1HSB6, symbol open-automation:USB_B
- added J6: Conn_01x02, symbol Connector_Generic:Conn_01x02
- added R16, R17: R_10k, Resistor_SMD:R_0603_1608Metric_Pad0.99x1.00mm_HandSolder, symbol open-automation:R_10k
- added U15: radio-housing-mounts, open-automation:radio-housing-mounts, symbol open-automation:radio-housing-mounts
- added U16: USB_IC-CP2104, Package_DFN_QFN:QFN-20-1EP_3x3mm_P0.45mm_EP1.6x1.6mm, symbol open-automation:USB_IC-CP2104
- renumbered J5 to J7, R40 to R39, U15 to U14, U14 to U7
Connections:
- net labels added: SCL, SDA
- wire segments 56 -> 80
Other:
- moved on the sheet: D10

Commit message: update
Parts:
- removed J5: USB_B, open-automation:USB_B-B1HSB6, symbol open-automation:USB_B
- removed P1, P2: CONN-BARREL-2x5.5mm, open-automation:CONN-BARREL_PJ-037A, symbol open-automation:CONN-BARREL-2x5.5mm
- removed P3: USB_A_2, open-automation:USB_A_2, symbol open-automation:USB_A_2
- removed U16: USB_IC-CP2104, Package_DFN_QFN:QFN-20-1EP_3x3mm_P0.45mm_EP1.6x1.6mm, symbol open-automation:USB_IC-CP2104
- added J5: Conn_01x02, Connector_PinHeader_2.54mm:PinHeader_1x02_P2.54mm_Vertical, symbol Connector_Generic:Conn_01x02
- added U16: molex-2x4-5.7mm, open-automation:molex-2x4-5.7mm, symbol open-automation:molex-2x4-5.7mm
- J4: footprint (none) -> Connector_PinHeader_2.54mm:PinHeader_2x06_P2.54mm_Vertical
Connections:
- net labels added: L_AUDIO_IN, R_AUDIO_IN
- wire segments 80 -> 68
Other:
- moved on the sheet: D10, D11, D12

Commit message: update
Parts:
- J5: footprint Connector_PinHeader_2.54mm:PinHeader_1x02_P2.54mm_Vertical -> Pin_Headers:Pin_Header_Straight_1x02_Pitch2.54mm
- J6, J7: footprint (none) -> Pin_Headers:Pin_Header_Straight_1x02_Pitch2.54mm
Changed lines of the file:
@@
 F 0 "J6" H 7055 917 50  0000 L CNN
 F 1 "Conn_01x02" H 7055 826 50  0000 L CNN
-F 2 "" H 6975 925 50  0001 C CNN
+F 2 "Pin_Headers:Pin_Header_Straight_1x02_Pitch2.54mm" H 6975 925 50  0001 C CNN
 F 3 "~" H 6975 925 50  0001 C CNN
 	1    6975 925
@@
 F 0 "J7" H 8680 917 50  0000 L CNN
 F 1 "Conn_01x02" H 8680 826 50  0000 L CNN
-F 2 "" H 8600 925 50  0001 C CNN
+F 2 "Pin_Headers:Pin_Header_Straight_1x02_Pitch2.54mm" H 8600 925 50  0001 C CNN
 F 3 "~" H 8600 925 50  0001 C CNN
 	1    8600 925
@@
 F 0 "J5" H 7650 3637 50  0000 L CNN
 F 1 "Conn_01x02" H 7650 3546 50  0000 L CNN
-F 2 "Connector_PinHeader_2.54mm:PinHeader_1x02_P2.54mm_Vertical" H 7570 3645 50  0001 C CNN
+F 2 "Pin_Headers:Pin_Header_Straight_1x02_Pitch2.54mm" H 7570 3645 50  0001 C CNN
 F 3 "~" H 7570 3645 50  0001 C CNN
 	1    7570 3645
