File: interface.sch (KiCad schematic (older format))
At the start: 18 parts, among them J4 Conn_02x06_Odd_Even, U14 molex-2x4-5.7mm, U15 radio-housing-mounts, U16 molex-2x4-5.7mm, U7 molex-2x4-5.7mm

Commit message: update
Connections:
- net labels removed: GNDA
Changed lines of the file:
@@
 Text Notes 8350 725  0    50   ~ 0
 GPS Antenna
-$Comp
-L power:GNDA #PWR0102
-U 1 1 5AE24110
-P 6575 1125
-F 0 "#PWR0102" H 6575 875 50  0001 C CNN
-F 1 "GNDA" H 6580 952 50  0000 C CNN
-F 2 "" H 6575 1125 50  0001 C CNN
-F 3 "" H 6575 1125 50  0001 C CNN
-	1    6575 1125
-	1    0    0    -1
-$EndComp
-$Comp
-L power:GNDA #PWR0103
-U 1 1 5AE24128
-P 8250 1125
-F 0 "#PWR0103" H 8250 875 50  0001 C CNN
-F 1 "GNDA" H 8255 952 50  0000 C CNN
-F 2 "" H 8250 1125 50  0001 C CNN
-F 3 "" H 8250 1125 50  0001 C CNN
-	1    8250 1125
-	1    0    0    -1
-$EndComp
 Wire Wire Line
 	6575 1125 6575 1025
@@
 Wire Wire Line
 	3400 825  3450 825
+$Comp
+L open-automation:GND #PWR?
+U 1 1 5B1DCBD3
+P 6575 1125
+F 0 "#PWR?" H 6575 875 50  0001 C CNN
+F 1 "GND" H 6575 975 50  0000 C CNN
+F 2 "" H 6575 1125 50  0000 C CNN
+F 3 "" H 6575 1125 50  0000 C CNN
+	1    6575 1125
+	1    0    0    -1
+$EndComp
+$Comp
+L open-automation:GND #PWR?
+U 1 1 5B1DCC14
+P 8250 1125
+F 0 "#PWR?" H 8250 875 50  0001 C CNN
+F 1 "GND" H 8250 975 50  0000 C CNN
+F 2 "" H 8250 1125 50  0000 C CNN
+F 3 "" H 8250 1125 50  0000 C CNN
+	1    8250 1125
+	1    0    0    -1
+$EndComp
 $EndSCHEMATC

Commit message: parts swap
Parts:
- renumbered FACTORY1 to SW1, REBOOT1 to SW2, PROG1 to SW3
Changed lines of the file:
@@
 $EndComp
 $Comp
-L open-automation:SW_PUSH FACTORY1
+L open-automation:SW_PUSH SW1
 U 1 1 5B15E1FC
 P 2100 5625
-F 0 "FACTORY1" H 2100 5800 50  0000 C CNN
+F 0 "SW1" H 2100 5800 50  0000 C CNN
 F 1 "SW_PUSH" H 2100 5545 50  0000 C CNN
 F 2 "Buttons_Switches_SMD:SW_SPST_KMR2" H 2100 5625 50  0001 C CNN
@@
 $EndComp
 $Comp
-L open-automation:SW_PUSH REBOOT1
+L open-automation:SW_PUSH SW2
 U 1 1 5B15E1FF
 P 3050 5625
-F 0 "REBOOT1" H 3050 5800 50  0000 C CNN
+F 0 "SW2" H 3050 5800 50  0000 C CNN
 F 1 "SW_PUSH" H 3050 5545 50  0000 C CNN
 F 2 "Buttons_Switches_SMD:SW_SPST_KMR2" H 3050 5625 50  0001 C CNN
@@
 $EndComp
 $Comp
-L open-automation:SW_PUSH PROG1
+L open-automation:SW_PUSH SW3
 U 1 1 5B15E203
 P 3875 5625
-F 0 "PROG1" H 3875 5800 50  0000 C CNN
+F 0 "SW3" H 3875 5800 50  0000 C CNN
 F 1 "SW_PUSH" H 3875 5545 50  0000 C CNN
 F 2 "Buttons_Switches_SMD:SW_SPST_KMR2" H 3875 5625 50  0001 C CNN

Commit message: added softpower circuit
Parts:
- added Q6: Q_NPN_BEC, Package_TO_SOT_SMD:SOT-23, symbol open-automation:Q_NPN_BEC
- added R51, R52, R53: R_1k, Resistor_SMD:R_0603_1608Metric_Pad0.99x1.00mm_HandSolder, symbol open-automation:R_1k
- SW1, SW2, SW3: footprint Buttons_Switches_SMD:SW_SPST_KMR2 -> Button_Switch_SMD:SW_SPST_KMR2
Connections:
- wire segments 70 -> 79
Changed lines of the file:
@@
 F 0 "SW1" H 2100 5800 50  0000 C CNN
 F 1 "SW_PUSH" H 2100 5545 50  0000 C CNN
-F 2 "Buttons_Switches_SMD:SW_SPST_KMR2" H 2100 5625 50  0001 C CNN
+F 2 "Button_Switch_SMD:SW_SPST_KMR2" H 2100 5625 50  0001 C CNN
 F 3 "http://www.mouser.com/ds/2/60/KMR2_9aug12-25127.pdf" H 2100 5625 50  0001 C CNN
 F 4 "KMR211NG LFS" H 2100 5625 60  0001 C CNN "Part Number"
@@
 F 0 "SW2" H 3050 5800 50  0000 C CNN
 F 1 "SW_PUSH" H 3050 5545 50  0000 C CNN
-F 2 "Buttons_Switches_SMD:SW_SPST_KMR2" H 3050 5625 50  0001 C CNN
+F 2 "Button_Switch_SMD:SW_SPST_KMR2" H 3050 5625 50  0001 C CNN
 F 3 "http://www.mouser.com/ds/2/60/KMR2_9aug12-25127.pdf" H 3050 5625 50  0001 C CNN
 F 4 "KMR211NG LFS" H 3050 5625 60  0001 C CNN "Part Number"
@@
 F 0 "SW3" H 3875 5800 50  0000 C CNN
 F 1 "SW_PUSH" H 3875 5545 50  0000 C CNN
-F 2 "Buttons_Switches_SMD:SW_SPST_KMR2" H 3875 5625 50  0001 C CNN
+F 2 "Button_Switch_SMD:SW_SPST_KMR2" H 3875 5625 50  0001 C CNN
 F 3 "http://www.mouser.com/ds/2/60/KMR2_9aug12-25127.pdf" H 3875 5625 50  0001 C CNN
 F 4 "KMR211NG LFS" H 3875 5625 60  0001 C CNN "Part Number"
@@
 Wire Wire Line
 	6550 2425 6650 2425
-Text HLabel 6550 2525 0    50   Output ~ 0
+Text HLabel 4950 2775 0    50   Output ~ 0
 SOFT_POWER
-Wire Wire Line
-	6550 2525 6650 2525
 Text HLabel 7300 3650 0    60   Input ~ 0
 L_MAIN_AUDIO
@@
 	1    0    0    -1
 $EndComp
+$Comp
+L open-automation:R_1k R52
+U 1 1 5B1B9666
+P 5225 2775
+F 0 "R52" V 5018 2775 50  0000 C CNN
+F 1 "R_1k" V 5109 2775 50  0000 C CNN
+F 2 "Resistor_SMD:R_0603_1608Metric_Pad0.99x1.00mm_HandSolder" V 5155 2775 50  0001 C CNN
+F 3 "https://www.digikey.com/product-detail/en/panasonic-electronic-components/ERJ-3GEYJ102V/P1.0KGDKR-ND/577615" V 5305 2775 50  0001 C CNN
+F 4 "ERJ-3GEYJ102V" V 5405 2875 60  0001 C CNN "Part Number"
+	1    5225 2775
+	0    1    1    0
+$EndComp
+$Comp
+L open-automation:R_1k R51
+U 1 1 5B1BAEB5
+P 5025 2950
+F 0 "R51" H 5095 2996 50  0000 L CNN
+F 1 "R_1k" H 5095 2905 50  0000 L CNN
+F 2 "Resistor_SMD:R_0603_1608Metric_Pad0.99x1.00mm_HandSolder" V 4955 2950 50  0001 C CNN
+F 3 "https://www.digikey.com/product-detail/en/panasonic-electronic-components/ERJ-3GEYJ102V/P1.0KGDKR-ND/577615" V 5105 2950 50  0001 C CNN
+F 4 "ERJ-3GEYJ102V" V 5205 3050 60  0001 C CNN "Part Number"
+	1    5025 2950
+	1    0    0    -1
+$EndComp
+$Comp
+L open-automation:R_1k R53
+U 1 1 5B1BB164
+P 5700 2350
+F 0 "R53" H 5500 2425 50  0000 L CNN
+F 1 "R_1k" H 5475 2350 50  0000 L CNN
+F 2 "Resistor_SMD:R_0603_1608Metric_Pad0.99x1.00mm_HandSolder" V 5630 2350 50  0001 C CNN
+F 3 "https://www.digikey.com/product-detail/en/panasonic-electronic-components/ERJ-3GEYJ102V/P1.0KGDKR-ND/577615" V 5780 2350 50  0001 C CNN
+F 4 "ERJ-3GEYJ102V" V 5880 2450 60  0001 C CNN "Part Number"
+	1    5700 2350
+	1    0    0    -1
+$EndComp
+Wire Wire Line
+	5700 2525 6650 2525
+Wire Wire Line
+	5700 2975 5700 3125
+$Comp
+L open-automation:GND #PWR0124
+U 1 1 5B1CB05C
+P 5025 3125
+F 0 "#PWR0124" H 5025 2875 50  0001 C CNN
+F 1 "GND" H 5030 2952 50  0000 C CNN
+F 2 "" H 5025 3125 50  0000 C CNN
+F 3 "" H 5025 3125 50  0000 C CNN
+	1    5025 3125
+	1    0    0    -1
+$EndComp
+$Comp
+L open-automation:GND #PWR0125
+U 1 1 5B1CB0C0
+P 5700 3125
+F 0 "#PWR0125" H 5700 2875 50  0001 C CNN
+F 1 "GND" H 5705 2952 50  0000 C CNN
+F 2 "" H 5700 3125 50  0000 C CNN
+F 3 "" H 5700 3125 50  0000 C CNN
+	1    5700 3125
+	1    0    0    -1
+$EndComp
+Wire Wire Line
+	5700 2575 5700 2525
+Wire Wire Line
+	5400 2775 5375 2775
+Wire Wire Line
+	5025 2775 5075 2775
+Wire Wire Line
+	5025 3125 5025 3100
+Wire Wire Line
+	5025 2775 5025 2800
+Wire Wire Line
+	5025 2775 4950 2775
+Connection ~ 5025 2775
+Wire Wire Line
+	5700 2525 5700 2500
+Connection ~ 5700 2525
+Wire Wire Line
+	5700 2200 5700 2175
+Text HLabel 5700 2175 1    60   Input ~ 0
+3v3
+$Comp
+L open-automation:Q_NPN_BEC Q6
+U 1 1 5B1F6997
+P 5600 2775
+F 0 "Q6" H 5791 2821 50  0000 L CNN
+F 1 "Q_NPN_BEC" H 5791 2730 50  0000 L CNN
+F 2 "Package_TO_SOT_SMD:SOT-23" H 5800 2875 50  0001 C CNN
+F 3 "https://www.digikey.com/product-detail/en/on-semiconductor/KST10MTF/KST10MTFCT-ND/965649" H 5800 2825 50  0001 C CNN
+F 4 "KST10MTF" H 5900 2925 50  0001 C CNN "Part Number"
+	1    5600 2775
+	1    0    0    -1
+$EndComp

Commit message: corrections day 1
Parts:
- removed D10, D11, D12: LED, LED_SMD:LED_0603_1608Metric_Pad0.82x1.00mm_HandSolder, symbol open-dash-daughterboard-rescue:LED-open-automation
- added D? (x3): LED-0603-R, LED_SMD:LED_0603_1608Metric_Pad0.82x1.00mm_HandSolder, symbol open-automation:LED-0603-R
- added J?: Conn_02x08_Counter_Clockwise, Connector_Molex:Molex_Mini-Fit_Jr_5566-16A2_2x08_P4.20mm_Vertical, symbol Connector_Generic:Conn_02x08_Counter_Clockwise
- added J?: Conn_02x08_Counter_Clockwise, symbol Connector_Generic:Conn_02x08_Counter_Clockwise
Changed lines of the file:
@@
 FL_AUDIO_OUT-
-$Comp
-L open-dash-daughterboard-rescue:LED-open-automation D10
-U 1 1 5B1799AD
-P 2100 4775
-F 0 "D10" V 2075 4875 50  0000 C CNN
-F 1 "LED" V 2200 4700 50  0000 C CNN
-F 2 "LED_SMD:LED_0603_1608Metric_Pad0.82x1.00mm_HandSolder" H 2100 4775 50  0001 C CNN
-F 3 "http://www.osram-os.com/Graphics/XPic9/00128792_0.pdf" H 2100 4775 50  0001 C CNN
-F 4 "475-2512-2-ND" H 2100 4775 60  0001 C CNN "Part Number"
-	1    2100 4775
-	0    -1   -1   0
-$EndComp
 $Comp
 L open-automation:SW_PUSH SW1
@@
 Connection ~ 2100 5300
 $Comp
-L open-dash-daughterboard-rescue:LED-open-automation D11
-U 1 1 5B15E1FE
-P 3050 4775
-F 0 "D11" V 3025 4875 50  0000 C CNN
-F 1 "LED" V 3150 4700 50  0000 C CNN
-F 2 "LED_SMD:LED_0603_1608Metric_Pad0.82x1.00mm_HandSolder" H 3050 4775 50  0001 C CNN
-F 3 "http://www.osram-os.com/Graphics/XPic9/00128792_0.pdf" H 3050 4775 50  0001 C CNN
-F 4 "475-2512-2-ND" H 3050 4775 60  0001 C CNN "Part Number"
-	1    3050 4775
-	0    -1   -1   0
-$EndComp
-$Comp
 L open-automation:SW_PUSH SW2
 U 1 1 5B15E1FF
@@
 	3175 5300 3050 5300
 Connection ~ 3050 5300
-$Comp
-L open-dash-daughterboard-rescue:LED-open-automation D12
-U 1 1 5B15E202
-P 3875 4775
-F 0 "D12" V 3850 4875 50  0000 C CNN
-F 1 "LED" V 3975 4700 50  0000 C CNN
-F 2 "LED_SMD:LED_0603_1608Metric_Pad0.82x1.00mm_HandSolder" H 3875 4775 50  0001 C CNN
-F 3 "http://www.osram-os.com/Graphics/XPic9/00128792_0.pdf" H 3875 4775 50  0001 C CNN
-F 4 "475-2512-2-ND" H 3875 4775 60  0001 C CNN "Part Number"
-	1    3875 4775
-	0    -1   -1   0
-$EndComp
 $Comp
 L open-automation:SW_PUSH SW3
@@
 	1    0    0    -1
 $EndComp
+$Comp
+L open-automation:LED-0603-R D?
+U 1 1 5B35FE49
+P 2100 4775
+F 0 "D?" V 2138 4658 50  0000 R CNN
+F 1 "LED-0603-R" V 2047 4658 50  0000 R CNN
+F 2 "LED_SMD:LED_0603_1608Metric_Pad0.82x1.00mm_HandSolder" H 2000 4775 50  0001 C CNN
+F 3 "https://www.digikey.com/products/en?keywords=475-2512-2-ND" H 2100 4875 50  0001 C CNN
+F 4 "LS Q976-NR-1" H 2200 4975 50  0001 C CNN "Part Number"
+	1    2100 4775
+	0    -1   -1   0
+$EndComp
+$Comp
+L open-automation:LED-0603-R D?
+U 1 1 5B35FF8B
+P 3050 4775
+F 0 "D?" V 3088 4658 50  0000 R CNN
+F 1 "LED-0603-R" V 2997 4658 50  0000 R CNN
+F 2 "LED_SMD:LED_0603_1608Metric_Pad0.82x1.00mm_HandSolder" H 2950 4775 50  0001 C CNN
+F 3 "https://www.digikey.com/products/en?keywords=475-2512-2-ND" H 3050 4875 50  0001 C CNN
+F 4 "LS Q976-NR-1" H 3150 4975 50  0001 C CNN "Part Number"
+	1    3050 4775
+	0    -1   -1   0
+$EndComp
+$Comp
+L open-automation:LED-0603-R D?
+U 1 1 5B3600BD
+P 3875 4775
+F 0 "D?" V 3913 4658 50  0000 R CNN
+F 1 "LED-0603-R" V 3822 4658 50  0000 R CNN
+F 2 "LED_SMD:LED_0603_1608Metric_Pad0.82x1.00mm_HandSolder" H 3775 4775 50  0001 C CNN
+F 3 "https://www.digikey.com/products/en?keywords=475-2512-2-ND" H 3875 4875 50  0001 C CNN
+F 4 "LS Q976-NR-1" H 3975 4975 50  0001 C CNN "Part Number"
+	1    3875 4775
+	0    -1   -1   0
+$EndComp
+$Comp
+L Connector_Generic:Conn_02x08_Counter_Clockwise J?
+U 1 1 5B5067C0
+P 7150 5150
+F 0 "J?" H 7200 5667 50  0000 C CNN
+F 1 "Conn_02x08_Counter_Clockwise" H 7200 5576 50  0000 C CNN
+F 2 "Connector_Molex:Molex_Mini-Fit_Jr_5566-16A2_2x08_P4.20mm_Vertical" H 7150 5150 50  0001 C CNN
+F 3 "https://www.digikey.com/product-detail/en/molex-llc/0015978162/WM7202-ND/3044417" H 7150 5150 50  0001 C CNN
+F 4 "https://www.digikey.com/product-detail/en/molex-llc/0015978162/WM7202-ND/3044417" H 7150 5150 50  0001 C CNN "Part Number"
+	1    7150 5150
+	1    0    0    -1
+$EndComp
+$Comp
+L Connector_Generic:Conn_02x08_Counter_Clockwise J?
+U 1 1 5B506A12
+P 8575 5200
+F 0 "J?" H 8625 5717 50  0000 C CNN
+F 1 "Conn_02x08_Counter_Clockwise" H 8625 5626 50  0000 C CNN
+F 2 "" H 8575 5200 50  0001 C CNN
+F 3 "https://www.digikey.com/product-detail/en/molex-llc/0015975161/WM2595-ND/2405484" H 8575 5200 50  0001 C CNN
+F 4 "0015975161" H 8575 5200 50  0001 C CNN "Part Number"
+	1    8575 5200
+	1    0    0    -1
+$EndComp

Commit message: corrections
Parts:
- removed AUDIO_IN1: Conn_01x02, Connector_PinHeader_2.54mm:PinHeader_1x03_P2.54mm_Vertical, symbol Connector_Generic:Conn_01x03
- added J?: Barrel_Jack, Connector_BarrelJack:BarrelJack_Horizontal, symbol Connector:Barrel_Jack
- J?: Part Number https://www.digikey.com/product-detail/en/molex-llc/0015978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 -> 0015978162
Connections:
- wire segments 79 -> 76
Changed lines of the file:
@@
 Wire Wire Line
 	7100 2225 7125 2225
-Wire Wire Line
-	7050 2425 7100 2425
-Wire Wire Line
-	7100 2425 7100 2325
-Connection ~ 7100 2325
-Text HLabel 6550 2425 0    60   Input ~ 0
-5V
-Wire Wire Line
-	6550 2425 6650 2425
-Text HLabel 4950 2775 0    50   Output ~ 0
+Text HLabel 4950 2675 0    50   Output ~ 0
 SOFT_POWER
-Text HLabel 7300 3650 0    60   Input ~ 0
+Text HLabel 7150 2425 2    60   Input ~ 0
 L_MAIN_AUDIO
-Text HLabel 7300 3750 0    60   Input ~ 0
+Text HLabel 7150 2525 2    60   Input ~ 0
 R_MAIN_AUDIO
-$Comp
-L open-automation:GND #PWR0120
-U 1 1 5B1495DE
-P 7325 3500
-F 0 "#PWR0120" H 7325 3250 50  0001 C CNN
-F 1 "GND" H 7325 3350 50  0000 C CNN
-F 2 "" H 7325 3500 50  0000 C CNN
-F 3 "" H 7325 3500 50  0000 C CNN
-	1    7325 3500
-	-1   0    0    1
-$EndComp
-$Comp
-L Connector_Generic:Conn_01x03 AUDIO_IN1
-U 1 1 5B16C30A
-P 7575 3650
-F 0 "AUDIO_IN1" H 7655 3642 50  0000 L CNN
-F 1 "Conn_01x02" H 7655 3551 50  0000 L CNN
-F 2 "Connector_PinHeader_2.54mm:PinHeader_1x03_P2.54mm_Vertical" H 7575 3650 50  0001 C CNN
-F 3 "~" H 7575 3650 50  0001 C CNN
-	1    7575 3650
-	1    0    0    -1
-$EndComp
-Wire Wire Line
-	7325 3500 7325 3550
-Wire Wire Line
-	7325 3550 7375 3550
-Wire Wire Line
-	7375 3650 7300 3650
-Wire Wire Line
-	7300 3750 7375 3750
 $Comp
 L open-automation:molex-2x4-5.7mm U14
@@
 L open-automation:R_1k R52
 U 1 1 5B1B9666
-P 5225 2775
-F 0 "R52" V 5018 2775 50  0000 C CNN
-F 1 "R_1k" V 5109 2775 50  0000 C CNN
-F 2 "Resistor_SMD:R_0603_1608Metric_Pad0.99x1.00mm_HandSolder" V 5155 2775 50  0001 C CNN
-F 3 "https://www.digikey.com/product-detail/en/panasonic-electronic-components/ERJ-3GEYJ102V/P1.0KGDKR-ND/577615" V 5305 2775 50  0001 C CNN
-F 4 "ERJ-3GEYJ102V" V 5405 2875 60  0001 C CNN "Part Number"
-	1    5225 2775
+P 5225 2675
+F 0 "R52" V 5018 2675 50  0000 C CNN
+F 1 "R_1k" V 5109 2675 50  0000 C CNN
+F 2 "Resistor_SMD:R_0603_1608Metric_Pad0.99x1.00mm_HandSolder" V 5155 2675 50  0001 C CNN
+F 3 "https://www.digikey.com/product-detail/en/panasonic-electronic-components/ERJ-3GEYJ102V/P1.0KGDKR-ND/577615" V 5305 2675 50  0001 C CNN
+F 4 "ERJ-3GEYJ102V" V 5405 2775 60  0001 C CNN "Part Number"
+	1    5225 2675
 	0    1    1    0
 $EndComp
@@
 L open-automation:R_1k R51
 U 1 1 5B1BAEB5
-P 5025 2950
-F 0 "R51" H 5095 2996 50  0000 L CNN
-F 1 "R_1k" H 5095 2905 50  0000 L CNN
-F 2 "Resistor_SMD:R_0603_1608Metric_Pad0.99x1.00mm_HandSolder" V 4955 2950 50  0001 C CNN
-F 3 "https://www.digikey.com/product-detail/en/panasonic-electronic-components/ERJ-3GEYJ102V/P1.0KGDKR-ND/577615" V 5105 2950 50  0001 C CNN
-F 4 "ERJ-3GEYJ102V" V 5205 3050 60  0001 C CNN "Part Number"
-	1    5025 2950
+P 5025 2850
+F 0 "R51" H 5095 2896 50  0000 L CNN
+F 1 "R_1k" H 5095 2805 50  0000 L CNN
+F 2 "Resistor_SMD:R_0603_1608Metric_Pad0.99x1.00mm_HandSolder" V 4955 2850 50  0001 C CNN
+F 3 "https://www.digikey.com/product-detail/en/panasonic-electronic-components/ERJ-3GEYJ102V/P1.0KGDKR-ND/577615" V 5105 2850 50  0001 C CNN
+F 4 "ERJ-3GEYJ102V" V 5205 2950 60  0001 C CNN "Part Number"
+	1    5025 2850
 	1    0    0    -1
 $EndComp
@@
 L open-automation:R_1k R53
 U 1 1 5B1BB164
-P 5700 2350
-F 0 "R53" H 5500 2425 50  0000 L CNN
-F 1 "R_1k" H 5475 2350 50  0000 L CNN
-F 2 "Resistor_SMD:R_0603_1608Metric_Pad0.99x1.00mm_HandSolder" V 5630 2350 50  0001 C CNN
-F 3 "https://www.digikey.com/product-detail/en/panasonic-electronic-components/ERJ-3GEYJ102V/P1.0KGDKR-ND/577615" V 5780 2350 50  0001 C CNN
-F 4 "ERJ-3GEYJ102V" V 5880 2450 60  0001 C CNN "Part Number"
-	1    5700 2350
-	1    0    0    -1
-$EndComp
-Wire Wire Line
-	5700 2525 6650 2525
-Wire Wire Line
-	5700 2975 5700 3125
+P 5700 2250
+F 0 "R53" H 5500 2325 50  0000 L CNN
+F 1 "R_1k" H 5475 2250 50  0000 L CNN
+F 2 "Resistor_SMD:R_0603_1608Metric_Pad0.99x1.00mm_HandSolder" V 5630 2250 50  0001 C CNN
+F 3 "https://www.digikey.com/product-detail/en/panasonic-electronic-components/ERJ-3GEYJ102V/P1.0KGDKR-ND/577615" V 5780 2250 50  0001 C CNN
+F 4 "ERJ-3GEYJ102V" V 5880 2350 60  0001 C CNN "Part Number"
+	1    5700 2250
+	1    0    0    -1
+$EndComp
+Wire Wire Line
+	5700 2425 6650 2425
+Wire Wire Line
+	5700 2875 5700 3025
 $Comp
 L open-automation:GND #PWR0124
 U 1 1 5B1CB05C
-P 5025 3125
-F 0 "#PWR0124" H 5025 2875 50  0001 C CNN
-F 1 "GND" H 5030 2952 50  0000 C CNN
-F 2 "" H 5025 3125 50  0000 C CNN
-F 3 "" H 5025 3125 50  0000 C CNN
-	1    5025 3125
+P 5025 3025
+F 0 "#PWR0124" H 5025 2775 50  0001 C CNN
+F 1 "GND" H 5030 2852 50  0000 C CNN
+F 2 "" H 5025 3025 50  0000 C CNN
+F 3 "" H 5025 3025 50  0000 C CNN
+	1    5025 3025
 	1    0    0    -1
 $EndComp
@@
 L open-automation:GND #PWR0125
 U 1 1 5B1CB0C0
-P 5700 3125
-F 0 "#PWR0125" H 5700 2875 50  0001 C CNN
-F 1 "GND" H 5705 2952 50  0000 C CNN
-F 2 "" H 5700 3125 50  0000 C CNN
-F 3 "" H 5700 3125 50  0000 C CNN
-	1    5700 3125
-	1    0    0    -1
-$EndComp
-Wire Wire Line
-	5700 2575 5700 2525
-Wire Wire Line
-	5400 2775 5375 2775
-Wire Wire Line
-	5025 2775 5075 2775
-Wire Wire Line
-	5025 3125 5025 3100
-Wire Wire Line
-	5025 2775 5025 2800
-Wire Wire Line
-	5025 2775 4950 2775
-Connection ~ 5025 2775
-Wire Wire Line
-	5700 2525 5700 2500
-Connection ~ 5700 2525
-Wire Wire Line
-	5700 2200 5700 2175
-Text HLabel 5700 2175 1    60   Input ~ 0
+P 5700 3025
+F 0 "#PWR0125" H 5700 2775 50  0001 C CNN
+F 1 "GND" H 5705 2852 50  0000 C CNN
+F 2 "" H 5700 3025 50  0000 C CNN
+F 3 "" H 5700 3025 50  0000 C CNN
+	1    5700 3025
+	1    0    0    -1
+$EndComp
+Wire Wire Line
+	5700 2475 5700 2425
+Wire Wire Line
+	5400 2675 5375 2675
+Wire Wire Line
+	5025 2675 5075 2675
+Wire Wire Line
+	5025 3025 5025 3000
+Wire Wire Line
+	5025 2675 5025 2700
+Wire Wire Line
+	5025 2675 4950 2675
+Connection ~ 5025 2675
+Wire Wire Line
+	5700 2425 5700 2400
+Connection ~ 5700 2425
+Wire Wire Line
+	5700 2100 5700 2075
+Text HLabel 5700 2075 1    60   Input ~ 0
 3v3
 $Comp
 L open-automation:Q_NPN_BEC Q6
 U 1 1 5B1F6997
-P 5600 2775
-F 0 "Q6" H 5791 2821 50  0000 L CNN
-F 1 "Q_NPN_BEC" H 5791 2730 50  0000 L CNN
-F 2 "Package_TO_SOT_SMD:SOT-23" H 5800 2875 50  0001 C CNN
-F 3 "https://www.digikey.com/product-detail/en/on-semiconductor/KST10MTF/KST10MTFCT-ND/965649" H 5800 2825 50  0001 C CNN
-F 4 "KST10MTF" H 5900 2925 50  0001 C CNN "Part Number"
-	1    5600 2775
+P 5600 2675
+F 0 "Q6" H 5791 2721 50  0000 L CNN
+F 1 "Q_NPN_BEC" H 5791 2630 50  0000 L CNN
+F 2 "Package_TO_SOT_SMD:SOT-23" H 5800 2775 50  0001 C CNN
+F 3 "https://www.digikey.com/product-detail/en/on-semiconductor/KST10MTF/KST10MTFCT-ND/965649" H 5800 2725 50  0001 C CNN
+F 4 "KST10MTF" H 5900 2825 50  0001 C CNN "Part Number"
+	1    5600 2675
 	1    0    0    -1
 $EndComp
@@
 F 2 "Connector_Molex:Molex_Mini-Fit_Jr_5566-16A2_2x08_P4.20mm_Vertical" H 7150 5150 50  0001 C CNN
 F 3 "https://www.digikey.com/product-detail/en/molex-llc/0015978162/WM7202-ND/3044417" H 7150 5150 50  0001 C CNN
-F 4 "https://www.digikey.com/product-detail/en/molex-llc/0015978162/WM7202-ND/3044417" H 7150 5150 50  0001 C CNN "Part Number"
+F 4 "0015978162" H 7150 5150 50  0001 C CNN "Part Number"
 	1    7150 5150
 	1    0    0    -1
@@
 	1    0    0    -1
 $EndComp
+Wire Wire Line
+	7150 2425 7050 2425
+Wire Wire Line
+	7150 2525 7050 2525
+$Comp
+L open-automation:GND #PWR?
+U 1 1 5B4B0C05
+P 6475 2575
+F 0 "#PWR?" H 6475 2325 50  0001 C CNN
+F 1 "GND" H 6475 2425 50  0000 C CNN
+F 2 "" H 6475 2575 50  0000 C CNN
+F 3 "" H 6475 2575 50  0000 C CNN
+	1    6475 2575
+	1    0    0    -1
+$EndComp
+Wire Wire Line
+	6650 2525 6475 2525
+Wire Wire Line
+	6475 2525 6475 2575
+$Comp
+L Connector:Barrel_Jack J?
+U 1 1 5B4B4D04
+P 6875 3400
+F 0 "J?" H 6953 3725 50  0000 C CNN
+F 1 "Barrel_Jack" H 6953 3634 50  0000 C CNN
+F 2 "Connector_BarrelJack:BarrelJack_Horizontal" H 6925 3360 50  0001 C CNN
+F 3 "https://www.digikey.com/product-detail/en/cui-inc/RCJ-021/CP-1406-ND/408493" H 6925 3360 50  0001 C CNN
+F 4 "RCJ-021" H 6875 3400 50  0001 C CNN "Part Number"
+	1    6875 3400
+	1    0    0    -1
+$EndComp
