File: GPS-interface.sch (KiCad schematic (older format))
At the start: 11 parts

Commit message: organizing
Parts:
- gave numbers to parts that had none: 11
Connections:
- net labels added: GPS_Antenna
- net labels removed: GPS_Ant
Changed lines of the file:
@@
 $EndDescr
 $Comp
-L Connector_Generic:Conn_01x04 J?
+L Connector_Generic:Conn_01x04 J3
 U 1 1 5AE2E72E
 P 5350 3500
-F 0 "J?" H 5430 3492 50  0000 L CNN
+F 0 "J3" H 5430 3492 50  0000 L CNN
 F 1 "Conn_01x04" H 5430 3401 50  0000 L CNN
 F 2 "" H 5350 3500 50  0001 C CNN
@@
 SCL
 $Comp
-L open-automation:GND #PWR?
+L open-automation:GND #PWR0137
 U 1 1 5AE2E7DF
 P 3550 3800
-F 0 "#PWR?" H 3550 3550 50  0001 C CNN
+F 0 "#PWR0137" H 3550 3550 50  0001 C CNN
 F 1 "GND" H 3555 3627 50  0000 C CNN
 F 2 "" H 3550 3800 50  0000 C CNN
@@
 	3550 3700 3550 3800
 $Comp
-L Connector_Generic:Conn_01x04 J?
+L Connector_Generic:Conn_01x04 J4
 U 1 1 5AE2E8B5
 P 6650 3500
-F 0 "J?" H 6730 3492 50  0000 L CNN
+F 0 "J4" H 6730 3492 50  0000 L CNN
 F 1 "Conn_01x04" H 6730 3401 50  0000 L CNN
 F 2 "" H 6650 3500 50  0001 C CNN
@@
 SCL
 $Comp
-L open-automation:A2235-H-dk_RF-Receivers U?
+L open-automation:A2235-H-dk_RF-Receivers U12
 U 1 1 5AE2F0AB
 P 9150 3250
-F 0 "U?" H 9250 4050 60  0000 C CNN
+F 0 "U12" H 9250 4050 60  0000 C CNN
 F 1 "A2235-H" H 9250 3944 60  0000 C CNN
 F 2 "digikey-footprints:GSM_Module_17.8x16.5mm_A2235-H" H 9350 3450 60  0001 L CNN
@@
 	6850 3600 8200 3600
 Text HLabel 8050 3850 0    50   Input ~ 0
-GPS_Ant
+GPS_Antenna
 Wire Wire Line
 	8350 3850 8050 3850
@@
 3v3
 $Comp
-L Device:R R?
+L Device:R R33
 U 1 1 5AEA67C5
 P 5000 3050
-F 0 "R?" H 5070 3096 50  0000 L CNN
+F 0 "R33" H 5070 3096 50  0000 L CNN
 F 1 "Jumper" H 5070 3005 50  0000 L CNN
 F 2 "" V 4930 3050 50  0001 C CNN
@@
 $EndComp
 $Comp
-L Device:R R?
+L Device:R R32
 U 1 1 5AEA683D
 P 4600 3050
-F 0 "R?" H 4670 3096 50  0000 L CNN
+F 0 "R32" H 4670 3096 50  0000 L CNN
 F 1 "Jumper" H 4670 3005 50  0000 L CNN
 F 2 "" V 4530 3050 50  0001 C CNN
@@
 $EndComp
 $Comp
-L Device:R R?
+L Device:R R31
 U 1 1 5AEA685D
 P 4200 3050
-F 0 "R?" H 4270 3096 50  0000 L CNN
+F 0 "R31" H 4270 3096 50  0000 L CNN
 F 1 "Jumper" H 4270 3005 50  0000 L CNN
 F 2 "" V 4130 3050 50  0001 C CNN
@@
 $EndComp
 $Comp
-L Device:R R?
+L Device:R R30
 U 1 1 5AEA687F
 P 3800 3050
-F 0 "R?" H 3870 3096 50  0000 L CNN
+F 0 "R30" H 3870 3096 50  0000 L CNN
 F 1 "Jumper" H 3870 3005 50  0000 L CNN
 F 2 "" V 3730 3050 50  0001 C CNN
@@
 	8050 3950 8350 3950
 $Comp
-L Device:C C?
+L Device:C C41
 U 1 1 5AEADD26
 P 7850 2550
-F 0 "C?" H 7965 2596 50  0000 L CNN
+F 0 "C41" H 7965 2596 50  0000 L CNN
 F 1 "C" H 7965 2505 50  0000 L CNN
 F 2 "" H 7888 2400 50  0001 C CNN
@@
 $EndComp
 $Comp
-L Device:C C?
+L Device:C C43
 U 1 1 5AEADD96
 P 8200 2550
-F 0 "C?" H 8315 2596 50  0000 L CNN
+F 0 "C43" H 8315 2596 50  0000 L CNN
 F 1 "C" H 8315 2505 50  0000 L CNN
 F 2 "" H 8238 2400 50  0001 C CNN
@@
 Connection ~ 8200 2800
 $Comp
-L Device:C C?
+L Device:C C44
 U 1 1 5AEB1B71
 P 10150 3350
-F 0 "C?" V 9898 3350 50  0000 C CNN
+F 0 "C44" V 9898 3350 50  0000 C CNN
 F 1 "C" V 9989 3350 50  0000 C CNN
 F 2 "" H 10188 3200 50  0001 C CNN
@@
 $EndComp
 $Comp
-L Device:C C?
+L Device:C C42
 U 1 1 5AEB1C00
 P 8100 2950
-F 0 "C?" V 7848 2950 50  0000 C CNN
+F 0 "C42" V 7848 2950 50  0000 C CNN
 F 1 "C" V 7939 2950 50  0000 C CNN
 F 2 "" H 8138 2800 50  0001 C CNN

Commit message: update
Parts:
- R33: renamed from R30; footprint (none) -> Resistor_SMD:R_0603_1608Metric_Pad0.99x1.00mm_HandSolder
- R34: renamed from R31; footprint (none) -> Resistor_SMD:R_0603_1608Metric_Pad0.99x1.00mm_HandSolder
- R35: renamed from R32; footprint (none) -> Resistor_SMD:R_0603_1608Metric_Pad0.99x1.00mm_HandSolder
- R36: renamed from R33; footprint (none) -> Resistor_SMD:R_0603_1608Metric_Pad0.99x1.00mm_HandSolder
- renumbered C41 to C42, C42 to C43, C43 to C44, C44 to C45, J3 to J1, J4 to J2, U12 to U13
Changed lines of the file:
@@
 $Descr A4 11693 8268
 encoding utf-8
-Sheet 13 14
+Sheet 11 13
 Title ""
 Date ""
@@
 $EndDescr
 $Comp
-L Connector_Generic:Conn_01x04 J3
+L Connector_Generic:Conn_01x04 J1
 U 1 1 5AE2E72E
 P 5350 3500
-F 0 "J3" H 5430 3492 50  0000 L CNN
+F 0 "J1" H 5430 3492 50  0000 L CNN
 F 1 "Conn_01x04" H 5430 3401 50  0000 L CNN
 F 2 "" H 5350 3500 50  0001 C CNN
@@
 SCL
 $Comp
-L open-automation:GND #PWR0137
+L open-automation:GND #PWR064
 U 1 1 5AE2E7DF
 P 3550 3800
-F 0 "#PWR0137" H 3550 3550 50  0001 C CNN
+F 0 "#PWR064" H 3550 3550 50  0001 C CNN
 F 1 "GND" H 3555 3627 50  0000 C CNN
 F 2 "" H 3550 3800 50  0000 C CNN
@@
 	3550 3700 3550 3800
 $Comp
-L Connector_Generic:Conn_01x04 J4
+L Connector_Generic:Conn_01x04 J2
 U 1 1 5AE2E8B5
 P 6650 3500
-F 0 "J4" H 6730 3492 50  0000 L CNN
+F 0 "J2" H 6730 3492 50  0000 L CNN
 F 1 "Conn_01x04" H 6730 3401 50  0000 L CNN
 F 2 "" H 6650 3500 50  0001 C CNN
@@
 SCL
 $Comp
-L open-automation:A2235-H-dk_RF-Receivers U12
+L open-automation:A2235-H-dk_RF-Receivers U13
 U 1 1 5AE2F0AB
 P 9150 3250
-F 0 "U12" H 9250 4050 60  0000 C CNN
+F 0 "U13" H 9250 4050 60  0000 C CNN
 F 1 "A2235-H" H 9250 3944 60  0000 C CNN
 F 2 "digikey-footprints:GSM_Module_17.8x16.5mm_A2235-H" H 9350 3450 60  0001 L CNN
@@
 3v3
 $Comp
-L Device:R R33
+L Device:R R36
 U 1 1 5AEA67C5
 P 5000 3050
-F 0 "R33" H 5070 3096 50  0000 L CNN
+F 0 "R36" H 5070 3096 50  0000 L CNN
 F 1 "Jumper" H 5070 3005 50  0000 L CNN
-F 2 "" V 4930 3050 50  0001 C CNN
+F 2 "Resistor_SMD:R_0603_1608Metric_Pad0.99x1.00mm_HandSolder" V 4930 3050 50  0001 C CNN
 F 3 "~" H 5000 3050 50  0001 C CNN
 	1    5000 3050
@@
 $EndComp
 $Comp
-L Device:R R32
+L Device:R R35
 U 1 1 5AEA683D
 P 4600 3050
-F 0 "R32" H 4670 3096 50  0000 L CNN
+F 0 "R35" H 4670 3096 50  0000 L CNN
 F 1 "Jumper" H 4670 3005 50  0000 L CNN
-F 2 "" V 4530 3050 50  0001 C CNN
+F 2 "Resistor_SMD:R_0603_1608Metric_Pad0.99x1.00mm_HandSolder" V 4530 3050 50  0001 C CNN
 F 3 "~" H 4600 3050 50  0001 C CNN
 	1    4600 3050
@@
 $EndComp
 $Comp
-L Device:R R31
+L Device:R R34
 U 1 1 5AEA685D
 P 4200 3050
-F 0 "R31" H 4270 3096 50  0000 L CNN
+F 0 "R34" H 4270 3096 50  0000 L CNN
 F 1 "Jumper" H 4270 3005 50  0000 L CNN
-F 2 "" V 4130 3050 50  0001 C CNN
+F 2 "Resistor_SMD:R_0603_1608Metric_Pad0.99x1.00mm_HandSolder" V 4130 3050 50  0001 C CNN
 F 3 "~" H 4200 3050 50  0001 C CNN
 	1    4200 3050
@@
 $EndComp
 $Comp
-L Device:R R30
+L Device:R R33
 U 1 1 5AEA687F
 P 3800 3050
-F 0 "R30" H 3870 3096 50  0000 L CNN
+F 0 "R33" H 3870 3096 50  0000 L CNN
 F 1 "Jumper" H 3870 3005 50  0000 L CNN
-F 2 "" V 3730 3050 50  0001 C CNN
+F 2 "Resistor_SMD:R_0603_1608Metric_Pad0.99x1.00mm_HandSolder" V 3730 3050 50  0001 C CNN
 F 3 "~" H 3800 3050 50  0001 C CNN
 	1    3800 3050
@@
 	8050 3950 8350 3950
 $Comp
-L Device:C C41
+L Device:C C42
 U 1 1 5AEADD26
 P 7850 2550
-F 0 "C41" H 7965 2596 50  0000 L CNN
+F 0 "C42" H 7965 2596 50  0000 L CNN
 F 1 "C" H 7965 2505 50  0000 L CNN
 F 2 "" H 7888 2400 50  0001 C CNN
@@
 $EndComp
 $Comp
-L Device:C C43
+L Device:C C44
 U 1 1 5AEADD96
 P 8200 2550
-F 0 "C43" H 8315 2596 50  0000 L CNN
+F 0 "C44" H 8315 2596 50  0000 L CNN
 F 1 "C" H 8315 2505 50  0000 L CNN
 F 2 "" H 8238 2400 50  0001 C CNN
@@
 Connection ~ 8200 2800
 $Comp
-L Device:C C44
+L Device:C C45
 U 1 1 5AEB1B71
 P 10150 3350
-F 0 "C44" V 9898 3350 50  0000 C CNN
+F 0 "C45" V 9898 3350 50  0000 C CNN
 F 1 "C" V 9989 3350 50  0000 C CNN
 F 2 "" H 10188 3200 50  0001 C CNN
@@
 $EndComp
 $Comp
-L Device:C C42
+L Device:C C43
 U 1 1 5AEB1C00
 P 8100 2950
-F 0 "C42" V 7848 2950 50  0000 C CNN
+F 0 "C43" V 7848 2950 50  0000 C CNN
 F 1 "C" V 7939 2950 50  0000 C CNN
 F 2 "" H 8138 2800 50  0001 C CNN

Commit message: update
Parts:
- removed C42, C43, C44, C45: C, symbol Device:C
- removed J1, J2: Conn_01x04, symbol Connector_Generic:Conn_01x04
- removed R33, R34, R35, R36: Jumper, Resistor_SMD:R_0603_1608Metric_Pad0.99x1.00mm_HandSolder, symbol Device:R
- added C42: C_1uF, Capacitors_SMD:C_0603, symbol open-automation:C_1uF
- added C43: C_0.1uF, Capacitors_SMD:C_0603, symbol open-automation:C_0.1uF
Connections:
- net labels removed: GND_Plane, GPS_Antenna, SCL, SDA
- wire segments 45 -> 23
Other:
- note removed: "This block will be a piece that can be either left on the board and the antenna can be installed, or can be broken off and wired up to the bezel \n"

Commit message: update
Parts:
- added R33, R34, R35, R36, R42: R_10k, Resistor_SMD:R_0603_1608Metric_Pad0.99x1.00mm_HandSolder, symbol open-automation:R_10k
- added RX_TX1: CONN_01X02, Connector_PinHeader_2.54mm:PinHeader_1x02_P2.54mm_Vertical, symbol open-automation:CONN_01X02
Connections:
- net labels added: ANT_SW, EN_I2C, GPS_Antenna, RST_GPS, SCL, SDA, Vout, WAKEUP
- wire segments 23 -> 46
Other:
- moved on the sheet: U13

Commit message: update
Parts:
- removed U13: A2235-H, digikey-footprints:GSM_Module_17.8x16.5mm_A2235-H, symbol open-automation:A2235-H-dk_RF-Receivers
- added U13: GPS-A2235-H, digikey-footprints:GSM_Module_17.8x16.5mm_A2235-H, symbol open-automation:GPS-A2235-H
- C42, C43: footprint Capacitors_SMD:C_0603 -> Capacitor_SMD:C_0603_1608Metric_Pad0.99x1.00mm_HandSolder
Changed lines of the file:
@@
 Comment4 ""
 $EndDescr
-$Comp
-L open-automation:A2235-H-dk_RF-Receivers U13
-U 1 1 5AE2F0AB
-P 7025 3150
-F 0 "U13" H 7550 3600 60  0000 C CNN
-F 1 "A2235-H" H 6825 3600 60  0000 C CNN
-F 2 "digikey-footprints:GSM_Module_17.8x16.5mm_A2235-H" H 7225 3350 60  0001 L CNN
-F 3 "http://update.maestro-wireless.com/GNSS/A2235-H/Maestro_A2135_HA2235_H_v11.pdf" H 7225 3450 60  0001 L CNN
-F 4 "1530-1011-1-ND" H 7225 3550 60  0001 L CNN "Digi-Key_PN"
-F 5 "A2235-H" H 7225 3650 60  0001 L CNN "MPN"
-F 6 "RF/IF and RFID" H 7225 3750 60  0001 L CNN "Category"
-F 7 "RF Receivers" H 7225 3850 60  0001 L CNN "Family"
-F 8 "http://update.maestro-wireless.com/GNSS/A2235-H/Maestro_A2135_HA2235_H_v11.pdf" H 7225 3950 60  0001 L CNN "DK_Datasheet_Link"
-F 9 "/product-detail/en/maestro-wireless-solutions/A2235-H/1530-1011-1-ND/4898055" H 7225 4050 60  0001 L CNN "DK_Detail_Page"
-F 10 "MODULE GPS SIRFSTARIV" H 7225 4150 60  0001 L CNN "Description"
-F 11 "Maestro Wireless Solutions" H 7225 4250 60  0001 L CNN "Manufacturer"
-F 12 "Active" H 7225 4350 60  0001 L CNN "Status"
-	1    7025 3150
-	-1   0    0    -1
-$EndComp
 Wire Wire Line
 	6225 3750 5925 3750
@@
 F 0 "C42" H 3375 3000 50  0000 L CNN
 F 1 "C_1uF" H 3250 2800 50  0000 L CNN
-F 2 "Capacitors_SMD:C_0603" H 3575 3200 50  0001 C CNN
+F 2 "Capacitor_SMD:C_0603_1608Metric_Pad0.99x1.00mm_HandSolder" H 3575 3200 50  0001 C CNN
 F 3 "https://www.digikey.com/product-detail/en/yageo/CC0603ZRY5V7BB105/311-1372-1-ND/2103156" H 3475 2650 50  0001 C CNN
 F 4 "CC0603ZRY5V7BB105" H 3600 3100 60  0001 C CNN "Part Number"
@@
 F 0 "C43" H 3850 2975 50  0000 L CNN
 F 1 "C_0.1uF" H 3850 2800 50  0000 L CNN
-F 2 "Capacitors_SMD:C_0603" H 3925 3200 50  0001 C CNN
+F 2 "Capacitor_SMD:C_0603_1608Metric_Pad0.99x1.00mm_HandSolder" H 3925 3200 50  0001 C CNN
 F 3 "https://www.digikey.com/product-detail/en/kemet/C0603C104K5RACTU/399-5089-1-ND/1465623" H 3825 2650 50  0001 C CNN
 F 4 "C0603C104K5RACTU" H 3950 3100 60  0001 C CNN "Part Number"
@@
 Wire Wire Line
 	2050 2675 2050 2750
+$Comp
+L open-automation:GPS-A2235-H U13
+U 1 1 5B1940C2
+P 7025 3150
+F 0 "U13" H 6700 2100 60  0000 C CNN
+F 1 "GPS-A2235-H" H 6775 3600 60  0000 C CNN
+F 2 "digikey-footprints:GSM_Module_17.8x16.5mm_A2235-H" H 7225 3350 60  0001 L CNN
+F 3 "https://www.digikey.com/product-detail/en/maestro-wireless-solutions/A2235-H/1530-1011-1-ND/4898055" H 7225 3450 60  0001 L CNN
+F 4 "A2235-H" H 7225 3650 60  0001 L CNN "Part Number"
+	1    7025 3150
+	-1   0    0    -1
+$EndComp
 $EndSCHEMATC

Commit message: parts swap
Parts:
- removed C42: C_1uF, Capacitor_SMD:C_0603_1608Metric_Pad0.99x1.00mm_HandSolder, symbol open-automation:C_1uF
- added C49: C_1uF, Capacitor_SMD:C_0603_1608Metric_Pad0.99x1.00mm_HandSolder, symbol open-automation:C_1uF
- C43: Part Number C0603C104K5RACTU -> C1608X8R1H104K080AB
Changed lines of the file:
@@
 Wire Wire Line
 	6225 3750 5925 3750
-Wire Wire Line
-	3475 2750 3475 2700
-Wire Wire Line
-	3475 2700 3650 2700
-Wire Wire Line
-	3475 3050 3475 3150
-Wire Wire Line
-	3475 3150 3625 3150
-$Comp
-L open-automation:C_1uF C42
-U 1 1 5B14A0F4
-P 3475 2900
-F 0 "C42" H 3375 3000 50  0000 L CNN
-F 1 "C_1uF" H 3250 2800 50  0000 L CNN
-F 2 "Capacitor_SMD:C_0603_1608Metric_Pad0.99x1.00mm_HandSolder" H 3575 3200 50  0001 C CNN
-F 3 "https://www.digikey.com/product-detail/en/yageo/CC0603ZRY5V7BB105/311-1372-1-ND/2103156" H 3475 2650 50  0001 C CNN
-F 4 "CC0603ZRY5V7BB105" H 3600 3100 60  0001 C CNN "Part Number"
-	1    3475 2900
-	1    0    0    -1
-$EndComp
-$Comp
-L open-automation:C_0.1uF C43
-U 1 1 5B14A2C2
-P 3825 2900
-F 0 "C43" H 3850 2975 50  0000 L CNN
-F 1 "C_0.1uF" H 3850 2800 50  0000 L CNN
-F 2 "Capacitor_SMD:C_0603_1608Metric_Pad0.99x1.00mm_HandSolder" H 3925 3200 50  0001 C CNN
-F 3 "https://www.digikey.com/product-detail/en/kemet/C0603C104K5RACTU/399-5089-1-ND/1465623" H 3825 2650 50  0001 C CNN
-F 4 "C0603C104K5RACTU" H 3950 3100 60  0001 C CNN "Part Number"
-	1    3825 2900
-	1    0    0    -1
-$EndComp
 $Comp
 L open-automation:GND #PWR0109
@@
 Wire Wire Line
 	3625 3200 3625 3150
-Wire Wire Line
-	3625 3150 3825 3150
-Connection ~ 3625 3150
 $Comp
 L open-automation:GND #PWR0110
@@
 EN_I2C
 Wire Wire Line
-	3825 2750 3825 2700
-Wire Wire Line
-	3825 3050 3825 3150
-Wire Wire Line
 	6925 2550 6925 2475
 Text HLabel 3650 2650 1    50   Input ~ 0
@@
 Wire Wire Line
 	3650 2650 3650 2700
-Connection ~ 3650 2700
-Wire Wire Line
-	3650 2700 3825 2700
 Wire Wire Line
 	2525 2625 2525 2725
@@
 L open-automation:GPS-A2235-H U13
 U 1 1 5B1940C2
-P 7025 3150
-F 0 "U13" H 6700 2100 60  0000 C CNN
-F 1 "GPS-A2235-H" H 6775 3600 60  0000 C CNN
-F 2 "digikey-footprints:GSM_Module_17.8x16.5mm_A2235-H" H 7225 3350 60  0001 L CNN
-F 3 "https://www.digikey.com/product-detail/en/maestro-wireless-solutions/A2235-H/1530-1011-1-ND/4898055" H 7225 3450 60  0001 L CNN
-F 4 "A2235-H" H 7225 3650 60  0001 L CNN "Part Number"
-	1    7025 3150
+P 6950 3075
+F 0 "U13" H 6625 2025 60  0000 C CNN
+F 1 "GPS-A2235-H" H 6700 3525 60  0000 C CNN
+F 2 "digikey-footprints:GSM_Module_17.8x16.5mm_A2235-H" H 7150 3275 60  0001 L CNN
+F 3 "https://www.digikey.com/product-detail/en/maestro-wireless-solutions/A2235-H/1530-1011-1-ND/4898055" H 7150 3375 60  0001 L CNN
+F 4 "A2235-H" H 7150 3575 60  0001 L CNN "Part Number"
+	1    6950 3075
 	-1   0    0    -1
 $EndComp
+Wire Wire Line
+	3650 2700 3825 2700
+Wire Wire Line
+	3825 2750 3825 2700
+Wire Wire Line
+	3825 3050 3825 3150
+Entry Wire Line
+	6800 3650 6900 3750
+Entry Wire Line
+	6800 3650 6900 3750
+Wire Wire Line
+	3450 3050 3450 3150
+Wire Wire Line
+	3450 3150 3625 3150
+Connection ~ 3625 3150
+Wire Wire Line
+	3625 3150 3825 3150
+Wire Wire Line
+	3650 2700 3450 2700
+Wire Wire Line
+	3450 2700 3450 2750
+Connection ~ 3650 2700
+$Comp
+L open-automation:C_0.1uF C43
+U 1 1 5B27EDBD
+P 3825 2900
+F 0 "C43" H 3940 2946 50  0000 L CNN
+F 1 "C_0.1uF" H 3940 2855 50  0000 L CNN
+F 2 "Capacitor_SMD:C_0603_1608Metric_Pad0.99x1.00mm_HandSolder" H 3925 3200 50  0001 C CNN
+F 3 "https://www.digikey.com/product-detail/en/tdk-corporation/C1608X8R1H104K080AB/445-8818-1-ND/3248223" H 3825 2650 50  0001 C CNN
+F 4 "C1608X8R1H104K080AB" H 3950 3100 60  0001 C CNN "Part Number"
+	1    3825 2900
+	1    0    0    -1
+$EndComp
+$Comp
+L open-automation:C_1uF C49
+U 1 1 5B2CB9BD
+P 3450 2900
+F 0 "C49" H 3565 2946 50  0000 L CNN
+F 1 "C_1uF" H 3565 2855 50  0000 L CNN
+F 2 "Capacitor_SMD:C_0603_1608Metric_Pad0.99x1.00mm_HandSolder" H 3550 3200 50  0001 C CNN
+F 3 "https://www.digikey.com/product-detail/en/tdk-corporation/CGA3E1X7R1C105M080AC/445-12540-1-ND/3954206" H 3450 2650 50  0001 C CNN
+F 4 "CGA3E1X7R1C105M080AC" H 3575 3100 60  0001 C CNN "Part Number"
+	1    3450 2900
+	1    0    0    -1
+$EndComp
 $EndSCHEMATC

Commit message: added softpower circuit
Parts:
- removed U13: GPS-A2235-H, digikey-footprints:GSM_Module_17.8x16.5mm_A2235-H, symbol open-automation:GPS-A2235-H
- added U13: A2235-H, digikey-footprints:GSM_Module_17.8x16.5mm_A2235-H, symbol open-automation:A2235-H
Connections:
- wire segments 46 -> 53
Changed lines of the file:
@@
 $EndComp
 Wire Wire Line
-	7625 2950 7700 2950
+	7625 2950 7650 2950
 Wire Wire Line
 	7700 2950 7700 2900
@@
 	8100 3050 8000 3050
 Wire Wire Line
-	7700 3050 7625 3050
+	7700 3050 7650 3050
 Text HLabel 6150 3250 0    50   Input ~ 0
 SCL
@@
 $EndComp
 Wire Wire Line
-	7750 3750 7625 3750
-Wire Wire Line
-	7625 3850 7750 3850
+	7750 3750 7650 3750
+Wire Wire Line
+	7625 3850 7650 3850
 Text Label 7750 3550 0    50   ~ 0
 WAKEUP
 Wire Wire Line
-	7750 3550 7625 3550
+	7750 3550 7650 3550
 Text Label 5925 3050 0    50   ~ 0
 WAKEUP
@@
 	7675 3175 7675 3150
 Wire Wire Line
-	7675 3150 7625 3150
+	7675 3150 7650 3150
 Text Label 2525 2625 1    50   ~ 0
 EN_I2C
@@
 	7675 3275 7675 3250
 Wire Wire Line
-	7675 3250 7625 3250
+	7675 3250 7650 3250
 Text Label 2050 2675 1    50   ~ 0
 ANT_SW
@@
 Wire Wire Line
 	2050 2675 2050 2750
-$Comp
-L open-automation:GPS-A2235-H U13
-U 1 1 5B1940C2
-P 6950 3075
-F 0 "U13" H 6625 2025 60  0000 C CNN
-F 1 "GPS-A2235-H" H 6700 3525 60  0000 C CNN
-F 2 "digikey-footprints:GSM_Module_17.8x16.5mm_A2235-H" H 7150 3275 60  0001 L CNN
-F 3 "https://www.digikey.com/product-detail/en/maestro-wireless-solutions/A2235-H/1530-1011-1-ND/4898055" H 7150 3375 60  0001 L CNN
-F 4 "A2235-H" H 7150 3575 60  0001 L CNN "Part Number"
-	1    6950 3075
-	-1   0    0    -1
-$EndComp
 Wire Wire Line
 	3650 2700 3825 2700
@@
 Wire Wire Line
 	3825 3050 3825 3150
-Entry Wire Line
-	6800 3650 6900 3750
-Entry Wire Line
-	6800 3650 6900 3750
 Wire Wire Line
 	3450 3050 3450 3150
@@
 	1    0    0    -1
 $EndComp
+$Comp
+L open-automation:A2235-H U13
+U 1 1 5B1FACC9
+P 7025 3150
+F 0 "U13" H 6700 3600 60  0000 C CNN
+F 1 "A2235-H" H 6850 2100 60  0000 C CNN
+F 2 "digikey-footprints:GSM_Module_17.8x16.5mm_A2235-H" H 7225 3350 60  0001 L CNN
+F 3 "https://www.digikey.com/product-detail/en/maestro-wireless-solutions/A2235-H/1530-1011-1-ND/4898055" H 7225 3450 60  0001 L CNN
+F 4 "A2235-H" H 7225 3650 60  0001 L CNN "Part Number"
+	1    7025 3150
+	-1   0    0    -1
+$EndComp
+Connection ~ 7650 2950
+Wire Wire Line
+	7650 2950 7700 2950
+Connection ~ 7650 3250
+Wire Wire Line
+	7650 3250 7625 3250
+Connection ~ 7650 3550
+Wire Wire Line
+	7650 3550 7625 3550
+Connection ~ 7650 3650
+Connection ~ 7650 3750
+Wire Wire Line
+	7650 3750 7625 3750
+Connection ~ 7650 3850
+Wire Wire Line
+	7650 3850 7750 3850
+Connection ~ 7650 3050
+Wire Wire Line
+	7650 3050 7625 3050
+Connection ~ 7650 3150
+Wire Wire Line
+	7650 3150 7625 3150
 $EndSCHEMATC
