File: GPS-interface.sch (KiCad schematic (older format))
At the start: 9 parts, among them U13 A2235-H

Commit message: corrections day 1
Connections:
- wire segments 53 -> 46
Changed lines of the file:
@@
 $EndComp
-Wire Wire Line
-	7625 2950 7650 2950
 Wire Wire Line
 	7700 2950 7700 2900
@@
 Wire Wire Line
 	8100 3050 8000 3050
-Wire Wire Line
-	7700 3050 7650 3050
 Text HLabel 6150 3250 0    50   Input ~ 0
 SCL
@@
 	1    0    0    -1
 $EndComp
-Wire Wire Line
-	7750 3750 7650 3750
-Wire Wire Line
-	7625 3850 7650 3850
 Text Label 7750 3550 0    50   ~ 0
 WAKEUP
-Wire Wire Line
-	7750 3550 7650 3550
 Text Label 5925 3050 0    50   ~ 0
 WAKEUP
@@
 Wire Wire Line
 	7675 3175 7675 3150
-Wire Wire Line
-	7675 3150 7650 3150
 Text Label 2525 2625 1    50   ~ 0
 EN_I2C
@@
 Wire Wire Line
 	7675 3275 7675 3250
-Wire Wire Line
-	7675 3250 7650 3250
 Text Label 2050 2675 1    50   ~ 0
 ANT_SW
@@
 	-1   0    0    -1
 $EndComp
-Connection ~ 7650 2950
-Wire Wire Line
-	7650 2950 7700 2950
-Connection ~ 7650 3250
-Wire Wire Line
-	7650 3250 7625 3250
-Connection ~ 7650 3550
-Wire Wire Line
-	7650 3550 7625 3550
-Connection ~ 7650 3650
-Connection ~ 7650 3750
-Wire Wire Line
-	7650 3750 7625 3750
-Connection ~ 7650 3850
-Wire Wire Line
-	7650 3850 7750 3850
-Connection ~ 7650 3050
-Wire Wire Line
-	7650 3050 7625 3050
-Connection ~ 7650 3150
-Wire Wire Line
-	7650 3150 7625 3150
+Wire Wire Line
+	7625 2950 7700 2950
+Wire Wire Line
+	7625 3050 7700 3050
+Wire Wire Line
+	7625 3750 7750 3750
+Wire Wire Line
+	7625 3850 7750 3850
+Wire Wire Line
+	7625 3550 7750 3550
+Wire Wire Line
+	7625 3150 7675 3150
+Wire Wire Line
+	7625 3250 7675 3250
 $EndSCHEMATC

Commit message: almost there
Parts:
- renumbered C49 to C65, C43 to C66, R33 to R54, R34 to R55, R35 to R56, R36 to R57, R42 to R58, U13 to U15
Changed lines of the file:
@@
 $Descr A4 11693 8268
 encoding utf-8
-Sheet 11 13
+Sheet 11 12
 Title ""
 Date ""
@@
 	6225 3750 5925 3750
 $Comp
-L open-automation:GND #PWR0109
+L open-automation:GND #PWR094
 U 1 1 5B14A58A
 P 3625 3200
-F 0 "#PWR0109" H 3625 2950 50  0001 C CNN
+F 0 "#PWR094" H 3625 2950 50  0001 C CNN
 F 1 "GND" H 3630 3027 50  0000 C CNN
 F 2 "" H 3625 3200 50  0000 C CNN
@@
 	3625 3200 3625 3150
 $Comp
-L open-automation:GND #PWR0110
+L open-automation:GND #PWR095
 U 1 1 5B14BBD1
 P 6825 4450
-F 0 "#PWR0110" H 6825 4200 50  0001 C CNN
+F 0 "#PWR095" H 6825 4200 50  0001 C CNN
 F 1 "GND" H 6830 4277 50  0000 C CNN
 F 2 "" H 6825 4450 50  0000 C CNN
@@
 GPS_Antenna
 $Comp
-L open-automation:R_10k R35
+L open-automation:R_10k R56
 U 1 1 5B16C9C4
 P 7700 2750
-F 0 "R35" V 7700 2700 50  0000 L CNN
+F 0 "R56" V 7700 2700 50  0000 L CNN
 F 1 "R_10k" H 7750 2800 50  0000 L CNN
 F 2 "Resistor_SMD:R_0603_1608Metric_Pad0.99x1.00mm_HandSolder" V 7630 2750 50  0001 C CNN
@@
 Vout
 $Comp
-L open-automation:R_10k R42
+L open-automation:R_10k R58
 U 1 1 5B16D38A
 P 7850 3050
-F 0 "R42" V 7850 3000 50  0000 L CNN
+F 0 "R58" V 7850 3000 50  0000 L CNN
 F 1 "R_10k" V 7775 2975 50  0000 L CNN
 F 2 "Resistor_SMD:R_0603_1608Metric_Pad0.99x1.00mm_HandSolder" V 7780 3050 50  0001 C CNN
@@
 	6150 3850 6225 3850
 $Comp
-L open-automation:R_10k R33
+L open-automation:R_10k R54
 U 1 1 5B1727D2
 P 2050 2900
-F 0 "R33" V 2050 2850 50  0000 L CNN
+F 0 "R54" V 2050 2850 50  0000 L CNN
 F 1 "R_10k" V 2125 2800 50  0000 L CNN
 F 2 "Resistor_SMD:R_0603_1608Metric_Pad0.99x1.00mm_HandSolder" V 1980 2900 50  0001 C CNN
@@
 	2050 3050 2050 3150
 $Comp
-L open-automation:R_10k R34
+L open-automation:R_10k R55
 U 1 1 5B173FED
 P 2525 2875
-F 0 "R34" V 2525 2825 50  0000 L CNN
+F 0 "R55" V 2525 2825 50  0000 L CNN
 F 1 "R_10k" H 2375 3050 50  0000 L CNN
 F 2 "Resistor_SMD:R_0603_1608Metric_Pad0.99x1.00mm_HandSolder" V 2455 2875 50  0001 C CNN
@@
 $EndComp
 $Comp
-L open-automation:GND #PWR0114
+L open-automation:GND #PWR093
 U 1 1 5B1746BB
 P 2525 3100
-F 0 "#PWR0114" H 2525 2850 50  0001 C CNN
+F 0 "#PWR093" H 2525 2850 50  0001 C CNN
 F 1 "GND" H 2530 2927 50  0000 C CNN
 F 2 "" H 2525 3100 50  0000 C CNN
@@
 	2525 2625 2525 2725
 $Comp
-L open-automation:GND #PWR0118
+L open-automation:GND #PWR092
 U 1 1 5B17E978
 P 2050 3150
-F 0 "#PWR0118" H 2050 2900 50  0001 C CNN
+F 0 "#PWR092" H 2050 2900 50  0001 C CNN
 F 1 "GND" H 2055 2977 50  0000 C CNN
 F 2 "" H 2050 3150 50  0000 C CNN
@@
 ANT_SW
 $Comp
-L open-automation:R_10k R36
+L open-automation:R_10k R57
 U 1 1 5B1812C6
 P 7800 3650
-F 0 "R36" V 7800 3600 50  0000 L CNN
+F 0 "R57" V 7800 3600 50  0000 L CNN
 F 1 "R_10k" V 7725 3575 50  0000 L CNN
 F 2 "Resistor_SMD:R_0603_1608Metric_Pad0.99x1.00mm_HandSolder" V 7730 3650 50  0001 C CNN
@@
 	7650 3650 7625 3650
 $Comp
-L open-automation:GND #PWR0119
+L open-automation:GND #PWR096
 U 1 1 5B181B4D
 P 8025 3650
-F 0 "#PWR0119" H 8025 3400 50  0001 C CNN
+F 0 "#PWR096" H 8025 3400 50  0001 C CNN
 F 1 "GND" V 8075 3500 50  0000 C CNN
 F 2 "" H 8025 3650 50  0000 C CNN
@@
 Connection ~ 3650 2700
 $Comp
-L open-automation:C_0.1uF C43
+L open-automation:C_0.1uF C66
 U 1 1 5B27EDBD
 P 3825 2900
-F 0 "C43" H 3940 2946 50  0000 L CNN
+F 0 "C66" H 3940 2946 50  0000 L CNN
 F 1 "C_0.1uF" H 3940 2855 50  0000 L CNN
 F 2 "Capacitor_SMD:C_0603_1608Metric_Pad0.99x1.00mm_HandSolder" H 3925 3200 50  0001 C CNN
@@
 $EndComp
 $Comp
-L open-automation:C_1uF C49
+L open-automation:C_1uF C65
 U 1 1 5B2CB9BD
 P 3450 2900
-F 0 "C49" H 3565 2946 50  0000 L CNN
+F 0 "C65" H 3565 2946 50  0000 L CNN
 F 1 "C_1uF" H 3565 2855 50  0000 L CNN
 F 2 "Capacitor_SMD:C_0603_1608Metric_Pad0.99x1.00mm_HandSolder" H 3550 3200 50  0001 C CNN
@@
 $EndComp
 $Comp
-L open-automation:A2235-H U13
+L open-automation:A2235-H U15
 U 1 1 5B1FACC9
 P 7025 3150
-F 0 "U13" H 6700 3600 60  0000 C CNN
+F 0 "U15" H 6700 3600 60  0000 C CNN
 F 1 "A2235-H" H 6850 2100 60  0000 C CNN
 F 2 "digikey-footprints:GSM_Module_17.8x16.5mm_A2235-H" H 7225 3350 60  0001 L CNN
