File: FM-radio.sch (KiCad schematic (older format))
At the start: 39 parts, among them Q1 Q_NPN_BEC, Q2 Q_NJFET_DGS, Q3 Q_NJFET_DGS, U12 Si4740, U18 74LVC1G17SE-7

Commit message: inductor update
Parts:
- removed L5, L6: 6.8uH, open-automation:Coilcraft_0805PS_Handsoldering, symbol Device:L
- removed L9: 220uH, open-automation:Coilcraft_1008PS_Handsoldering, symbol Device:L
- added L? (x2): L_6.8uH, Inductor_SMD:L_0603_1608Metric_Pad0.99x1.00mm_HandSolder, symbol open-automation:L_6.8uH
- added L?: L_220uH, Inductor_SMD:L_1206_3216Metric_Pad1.39x1.80mm_HandSolder, symbol open-automation:L_220uH
Changed lines of the file:
@@
 	1550 950  1750 950
-$Comp
-L Device:L L5
-U 1 1 5ADAF6D2
-P 1750 3500
-F 0 "L5" H 1803 3546 50  0000 L CNN
-F 1 "6.8uH" H 1803 3455 50  0000 L CNN
-F 2 "open-automation:Coilcraft_0805PS_Handsoldering" H 1750 3500 50  0001 C CNN
-F 3 "https://www.mouser.com/ProductDetail/Coilcraft/0805PS-682KLB?qs=sGAEpiMZZMsg%252by3WlYCkU2kWFds1hA9DACZH0%2fCmx5U%3d" H 1750 3500 50  0001 C CNN
-F 4 "Coilcraft" H 1750 3500 50  0001 C CNN "Manufacture"
-F 5 "0805PS-682KLB" H 1750 3500 50  0001 C CNN "Part number"
-	1    1750 3500
-	1    0    0    -1
-$EndComp
 $Comp
 L Device:C C26
@@
 Wire Wire Line
 	6600 4050 6600 3950
-$Comp
-L Device:L L9
-U 1 1 5ADB3533
-P 5550 2150
-F 0 "L9" H 5603 2196 50  0000 L CNN
-F 1 "220uH" H 5603 2105 50  0000 L CNN
-F 2 "open-automation:Coilcraft_1008PS_Handsoldering" H 5550 2150 50  0001 C CNN
-F 3 "https://www.mouser.com/ProductDetail/Coilcraft/1008PS-224KLB?qs=zCSbvcPd3pbbzsho0wjAGQ%3D%3D" H 5550 2150 50  0001 C CNN
-F 4 "1008PS-224KLB" H 5550 2150 50  0001 C CNN "Part Number"
-	1    5550 2150
-	1    0    0    -1
-$EndComp
 Wire Wire Line
 	5850 2450 5550 2450
@@
 Wire Wire Line
 	3225 5850 3525 5850
-$Comp
-L Device:L L6
-U 1 1 5AE3A452
-P 2050 3800
-F 0 "L6" H 2103 3846 50  0000 L CNN
-F 1 "6.8uH" H 2103 3755 50  0000 L CNN
-F 2 "open-automation:Coilcraft_0805PS_Handsoldering" H 2050 3800 50  0001 C CNN
-F 3 "https://www.mouser.com/ProductDetail/Coilcraft/0805PS-682KLB?qs=sGAEpiMZZMsg%252by3WlYCkU2kWFds1hA9DACZH0%2fCmx5U%3d" H 2050 3800 50  0001 C CNN
-F 4 "Coilcraft" H 2050 3800 50  0001 C CNN "Manufacture"
-F 5 "0805PS-682KLB" H 2050 3800 50  0001 C CNN "Part number"
-	1    2050 3800
-	0    -1   -1   0
-$EndComp
 Wire Wire Line
 	2200 3800 2650 3800
@@
 	0    1    1    0
 $EndComp
+$Comp
+L open-automation:L_6.8uH L?
+U 1 1 5B2ACCB3
+P 1750 3500
+F 0 "L?" H 1803 3546 50  0000 L CNN
+F 1 "L_6.8uH" H 1803 3455 50  0000 L CNN
+F 2 "Inductor_SMD:L_0603_1608Metric_Pad0.99x1.00mm_HandSolder" V 1600 3400 50  0001 C CNN
+F 3 "https://www.digikey.com/product-detail/en/tdk-corporation/GLFR1608T6R8M-LR/445-6156-1-ND/2465482" V 1700 3500 50  0001 C CNN
+F 4 "GLFR1608T6R8M-LR" V 1800 3600 50  0001 C CNN "Part Number"
+	1    1750 3500
+	1    0    0    -1
+$EndComp
+$Comp
+L open-automation:L_6.8uH L?
+U 1 1 5B2B1F69
+P 2050 3800
+F 0 "L?" V 2240 3800 50  0000 C CNN
+F 1 "L_6.8uH" V 2149 3800 50  0000 C CNN
+F 2 "Inductor_SMD:L_0603_1608Metric_Pad0.99x1.00mm_HandSolder" V 1900 3700 50  0001 C CNN
+F 3 "https://www.digikey.com/product-detail/en/tdk-corporation/GLFR1608T6R8M-LR/445-6156-1-ND/2465482" V 2000 3800 50  0001 C CNN
+F 4 "GLFR1608T6R8M-LR" V 2100 3900 50  0001 C CNN "Part Number"
+	1    2050 3800
+	0    -1   -1   0
+$EndComp
+$Comp
+L open-automation:L_220uH L?
+U 1 1 5B2CD872
+P 5550 2150
+F 0 "L?" H 5603 2196 50  0000 L CNN
+F 1 "L_220uH" H 5603 2105 50  0000 L CNN
+F 2 "Inductor_SMD:L_1206_3216Metric_Pad1.39x1.80mm_HandSolder" V 5400 2050 50  0001 C CNN
+F 3 "https://www.digikey.com/product-detail/en/taiyo-yuden/CB2518T221K/587-2193-1-ND/2002891" V 5500 2150 50  0001 C CNN
+F 4 "CB2518T221K" V 5600 2250 50  0001 C CNN "Part Number"
+	1    5550 2150
+	1    0    0    -1
+$EndComp
 $EndSCHEMATC

Commit message: corrections day 1
Parts:
- U12: footprint Housings_DFN_QFN:QFN-24-1EP_4x4mm_Pitch0.5mm -> open-automation:QFN-24_4x4mm_P0.5mm
Connections:
- wire segments 134 -> 136
Changed lines of the file:
@@
 	1    0    0    -1
 $EndComp
-Wire Wire Line
-	9650 2500 9650 2450
-Wire Wire Line
-	9650 2450 8950 2450
 NoConn ~ 8950 2850
 NoConn ~ 8950 2750
@@
 Wire Wire Line
 	10450 2750 10450 2850
-$Comp
-L open-automation:GND #PWR061
-U 1 1 5ADEBD94
-P 9650 2500
-F 0 "#PWR061" H 9650 2250 50  0001 C CNN
-F 1 "GND" H 9655 2327 50  0000 C CNN
-F 2 "" H 9650 2500 50  0000 C CNN
-F 3 "" H 9650 2500 50  0000 C CNN
-	1    9650 2500
-	1    0    0    -1
-$EndComp
 Connection ~ 10450 2350
 Wire Wire Line
@@
 Wire Wire Line
 	2700 950  3800 950
-$Comp
-L open-automation:Si4740 U12
-U 1 1 5B1B14DB
-P 7750 3300
-F 0 "U12" H 8991 4046 50  0000 L CNN
-F 1 "Si4740" H 8991 3955 50  0000 L CNN
-F 2 "Housings_DFN_QFN:QFN-24-1EP_4x4mm_Pitch0.5mm" H 7950 4050 50  0001 C CNN
-F 3 "https://www.digikey.com/product-detail/en/silicon-labs/SI4740-C10-GMR/336-4880-1-ND/8619844" H 7950 3850 50  0001 C CNN
-F 4 "SI4740-C10-GMR" H 7750 3300 50  0001 C CNN "Part Number"
-	1    7750 3300
-	1    0    0    -1
-$EndComp
 Text HLabel 1550 950  0    50   Input ~ 0
 AMF_Antenna
@@
 	1    0    0    -1
 $EndComp
+$Comp
+L open-automation:Si4740 U12
+U 1 1 5B1B14DB
+P 7750 3300
+F 0 "U12" H 8991 4046 50  0000 L CNN
+F 1 "Si4740" H 8991 3955 50  0000 L CNN
+F 2 "open-automation:QFN-24_4x4mm_P0.5mm" H 7950 4050 50  0001 C CNN
+F 3 "https://www.digikey.com/product-detail/en/silicon-labs/SI4740-C10-GMR/336-4880-1-ND/8619844" H 7950 3850 50  0001 C CNN
+F 4 "SI4740-C10-GMR" H 7750 3300 50  0001 C CNN "Part Number"
+	1    7750 3300
+	1    0    0    -1
+$EndComp
+Wire Wire Line
+	8950 2450 9025 2450
+Wire Wire Line
+	9025 2450 9025 3050
+Wire Wire Line
+	8950 3050 9025 3050
+Connection ~ 9025 3050
+Wire Wire Line
+	9025 3050 9025 3150
+$Comp
+L open-automation:GND #PWR?
+U 1 1 5B42E917
+P 9025 3150
+F 0 "#PWR?" H 9025 2900 50  0001 C CNN
+F 1 "GND" H 9030 2977 50  0000 C CNN
+F 2 "" H 9025 3150 50  0000 C CNN
+F 3 "" H 9025 3150 50  0000 C CNN
+	1    9025 3150
+	1    0    0    -1
+$EndComp

Commit message: corrections
Parts:
- R29: symbol open-automation:R_10 -> open-dash-daughterboard-rescue:R_10-open-automation
Changed lines of the file:
@@
 $EndComp
 $Comp
-L open-automation:R_10 R29
+L open-dash-daughterboard-rescue:R_10-open-automation R29
 U 1 1 5B292BF0
 P 5325 1500

Commit message: almost there
Parts:
- gave numbers to parts that had none: 3
- renumbered C26 to C49, C27 to C50, C42 to C51, C29 to C52, C30 to C53, C31 to C54, C32 to C55, C33 to C56, C34 to C57, C35 to C58, C36 to C59, C37 to C60, C38 to C61, C46 to C62, C40 to C63, C48 to C64, D8 to D13, D9 to D14, Q1 to Q3, Q2 to Q4, Q3 to Q5, R24 to R45, R25 to R46, R26 to R47, R27 to R48, R28 to R49, R29 to R50, R30 to R51, R31 to R52, R32 to R53, U18 to U13, U12 to U14

Commit message: updated corrections
Parts:
- D13, D14, Q3, Q4, Q5: footprint TO_SOT_Packages_SMD:SOT-23 -> Package_TO_SOT_SMD:SOT-23
- L10: footprint Inductors_SMD:L_7.3x7.3_H4.5 -> Inductor_SMD:L_7.3x7.3_H4.5
- L11: footprint Inductors_SMD:L_6.3x6.3_H3 -> Inductor_SMD:L_6.3x6.3_H3
- L7, L8: footprint Inductors_SMD:L_0603_HandSoldering -> Inductor_SMD:L_0603_1608Metric_Pad0.99x1.00mm_HandSolder
- U13: footprint TO_SOT_Packages_SMD:SOT-353_SC-70-5_Handsoldering -> Package_TO_SOT_SMD:SOT-353_SC-70-5_Handsoldering
- U14: footprint open-automation:QFN-24_4x4mm_P0.5mm -> Package_DFN_QFN:QFN-24-1EP_4x4mm_P0.5mm_EP2.7x2.6mm
Changed lines of the file:
@@
 F 0 "L8" H 2753 1296 50  0000 L CNN
 F 1 "122nH" H 2753 1205 50  0000 L CNN
-F 2 "Inductors_SMD:L_0603_HandSoldering" H 2700 1250 50  0001 C CNN
+F 2 "Inductor_SMD:L_0603_1608Metric_Pad0.99x1.00mm_HandSolder" H 2700 1250 50  0001 C CNN
 F 3 "https://www.digikey.com/product-detail/en/pulse-electronics-network/PE-0603CD121GTT/1840-1101-1-ND/8120509" H 2700 1250 50  0001 C CNN
 F 4 "PE-0603CD121GTT" H 2700 1250 50  0001 C CNN "Part Number"
@@
 F 0 "L7" V 2600 950 50  0000 C CNN
 F 1 "33nH" V 2525 950 50  0000 C CNN
-F 2 "Inductors_SMD:L_0603_HandSoldering" H 2450 950 50  0001 C CNN
+F 2 "Inductor_SMD:L_0603_1608Metric_Pad0.99x1.00mm_HandSolder" H 2450 950 50  0001 C CNN
 F 3 "https://www.digikey.com/product-detail/en/bourns-inc/CW160808-33NJ/CW160808-33NJCT-ND/3767866" H 2450 950 50  0001 C CNN
 F 4 "CW160808-33NJ" V 2450 950 50  0001 C CNN "Part Number"
@@
 F 0 "Q4" H 5650 2875 50  0000 L CNN
 F 1 "Q_NJFET_DGS" H 5650 2800 50  0000 L CNN
-F 2 "TO_SOT_Packages_SMD:SOT-23" H 5650 2850 50  0001 C CNN
+F 2 "Package_TO_SOT_SMD:SOT-23" H 5650 2850 50  0001 C CNN
 F 3 "https://www.digikey.com/product-detail/en/nxp-usa-inc/BF861C215/568-6169-1-ND/2531456" H 5450 2750 50  0001 C CNN
 F 4 "BF861C,215" H 5450 2750 50  0001 C CNN "Part Number"
@@
 F 0 "D14" H 4525 3875 60  0000 R CNN
 F 1 "D1213A-01SO-7" H 4525 3975 60  0000 R CNN
-F 2 "TO_SOT_Packages_SMD:SOT-23" H 4775 4350 60  0001 L CNN
+F 2 "Package_TO_SOT_SMD:SOT-23" H 4775 4350 60  0001 L CNN
 F 3 "https://www.digikey.com/product-detail/en/diodes-incorporated/D1213A-01SO-7/D1213A-01SO-7DICT-ND/3340430" H 4775 4450 60  0001 L CNN
 F 4 "D1213A-01SO-7" H 4775 4550 60  0001 L CNN "Part Number"
@@
 F 0 "L10" H 5603 4346 50  0000 L CNN
 F 1 "1mH" H 5603 4255 50  0000 L CNN
-F 2 "Inductors_SMD:L_7.3x7.3_H4.5" H 5550 4300 50  0001 C CNN
+F 2 "Inductor_SMD:L_7.3x7.3_H4.5" H 5550 4300 50  0001 C CNN
 F 3 "https://www.digikey.com/product-detail/en/bourns-inc/SRR0745A-102M/SRR0745A-102MCT-ND/5031149" H 5550 4300 50  0001 C CNN
 F 4 "SRR0745A-102M" H 5550 4300 50  0001 C CNN "Part Number"
@@
 F 0 "L11" H 6653 3846 50  0000 L CNN
 F 1 "33uH" H 6653 3755 50  0000 L CNN
-F 2 "Inductors_SMD:L_6.3x6.3_H3" H 6600 3800 50  0001 C CNN
+F 2 "Inductor_SMD:L_6.3x6.3_H3" H 6600 3800 50  0001 C CNN
 F 3 "https://www.digikey.com/product-detail/en/bourns-inc/SRR0604-330KL/SRR0604-330KLCT-ND/2352994" H 6600 3800 50  0001 C CNN
 F 4 "SRR0604-330KL" H 6600 3800 50  0001 C CNN "Part Number"
@@
 F 0 "Q5" H 5650 3925 50  0000 L CNN
 F 1 "Q_NJFET_DGS" H 5650 3850 50  0000 L CNN
-F 2 "TO_SOT_Packages_SMD:SOT-23" H 5650 3900 50  0001 C CNN
+F 2 "Package_TO_SOT_SMD:SOT-23" H 5650 3900 50  0001 C CNN
 F 3 "https://www.digikey.com/product-detail/en/nxp-usa-inc/BF861C215/568-6169-1-ND/2531456" H 5450 3800 50  0001 C CNN
 F 4 "BF861C,215" H 5450 3800 50  0001 C CNN "Part Number"
@@
 F 0 "Q3" H 3916 5896 50  0000 L CNN
 F 1 "Q_NPN_BEC" H 3916 5805 50  0000 L CNN
-F 2 "TO_SOT_Packages_SMD:SOT-23" H 3925 5950 50  0001 C CNN
+F 2 "Package_TO_SOT_SMD:SOT-23" H 3925 5950 50  0001 C CNN
 F 3 "https://www.digikey.com/product-detail/en/on-semiconductor/KST10MTF/KST10MTFCT-ND/965649" H 3725 5850 50  0001 C CNN
 F 4 "KST10MTF" H 3725 5850 50  0001 C CNN "Part Number"
@@
 F 0 "D13" H 3750 1025 60  0000 R CNN
 F 1 "D1213A-01SO-7" H 3750 1125 60  0000 R CNN
-F 2 "TO_SOT_Packages_SMD:SOT-23" H 4000 1500 60  0001 L CNN
+F 2 "Package_TO_SOT_SMD:SOT-23" H 4000 1500 60  0001 L CNN
 F 3 "https://www.digikey.com/product-detail/en/diodes-incorporated/D1213A-01SO-7/D1213A-01SO-7DICT-ND/3340430" H 4000 1600 60  0001 L CNN
 F 4 "D1213A-01SO-7" H 4000 1700 60  0001 L CNN "Part Number"
@@
 F 0 "U13" H 2375 5700 60  0000 L CNN
 F 1 "74LVC1G17SE-7" H 2350 5600 60  0000 L CNN
-F 2 "TO_SOT_Packages_SMD:SOT-353_SC-70-5_Handsoldering" H 2450 6150 60  0001 L CNN
+F 2 "Package_TO_SOT_SMD:SOT-353_SC-70-5_Handsoldering" H 2450 6150 60  0001 L CNN
 F 3 "https://www.digikey.com/product-detail/en/diodes-incorporated/74LVC1G17SE-7/74LVC1G17SE-7CT-ND/3829456" H 2450 6250 60  0001 L CNN
 F 4 "74LVC1G17SE-7" H 2450 6350 60  0001 L CNN "Part Number"
@@
 F 0 "U14" H 8991 4046 50  0000 L CNN
 F 1 "Si4740" H 8991 3955 50  0000 L CNN
-F 2 "open-automation:QFN-24_4x4mm_P0.5mm" H 7950 4050 50  0001 C CNN
+F 2 "Package_DFN_QFN:QFN-24-1EP_4x4mm_P0.5mm_EP2.7x2.6mm" H 7950 4050 50  0001 C CNN
 F 3 "https://www.digikey.com/product-detail/en/silicon-labs/SI4740-C10-GMR/336-4880-1-ND/8619844" H 7950 3850 50  0001 C CNN
 F 4 "SI4740-C10-GMR" H 7750 3300 50  0001 C CNN "Part Number"

Commit message: traces
Parts:
- added R69: R_10k, Resistor_SMD:R_0603_1608Metric_Pad0.99x1.00mm_HandSolder, symbol open-automation:R_10k
Connections:
- wire segments 136 -> 140
Changed lines of the file:
@@
 $EndComp
 Wire Wire Line
-	7750 3550 7750 3800
+	7750 3550 7750 3675
 Wire Wire Line
 	7950 3550 7950 3800
@@
 	1    0    0    -1
 $EndComp
+Wire Wire Line
+	7750 3675 7650 3675
+Connection ~ 7750 3675
+Wire Wire Line
+	7750 3675 7750 3800
+$Comp
+L open-automation:R_10k R69
+U 1 1 5B37BC7C
+P 7500 3675
+F 0 "R69" V 7293 3675 50  0000 C CNN
+F 1 "R_10k" V 7384 3675 50  0000 C CNN
+F 2 "Resistor_SMD:R_0603_1608Metric_Pad0.99x1.00mm_HandSolder" V 7430 3675 50  0001 C CNN
+F 3 "https://www.digikey.com/product-detail/en/yageo/RC0603JR-0710KL/311-10KGRCT-ND/729647" V 7580 3675 50  0001 C CNN
+F 4 "RC0603JR-0710KL" V 7680 3775 60  0001 C CNN "Part Number"
+	1    7500 3675
+	0    1    1    0
+$EndComp
+Wire Wire Line
+	7350 3675 7300 3675
+Wire Wire Line
+	7300 3675 7300 3550
+Text HLabel 7300 3550 1    60   Input ~ 0
+3v3
 $EndSCHEMATC
