File: canbus.sch (KiCad schematic (older format))
At the start: 13 parts

Commit message: Slight re-arrangment, and added datasheets for potential video options.
Parts:
- added R? (x2): Jumper 0ohm, symbol Device:R
Connections:
- net labels added: CAN_RX, CAN_TX
- wire segments 56 -> 64
Changed lines of the file:
@@
 	4625 2950 4625 2750
 Wire Wire Line
-	3950 2850 5325 2850
+	3950 2850 4300 2850
 Wire Wire Line
-	4625 2750 5325 2750
+	4625 2750 4700 2750
 $Comp
 L open-automation:R_10k R?
@@
 	1    0    0    -1
 $EndComp
+$Comp
+L Device:R R?
+U 1 1 5AE8F142
+P 4300 1800
+F 0 "R?" H 4230 1754 50  0000 R CNN
+F 1 "Jumper 0ohm" H 4230 1845 50  0000 R CNN
+F 2 "" V 4230 1800 50  0001 C CNN
+F 3 "~" H 4300 1800 50  0001 C CNN
+	1    4300 1800
+	1    0    0    1
+$EndComp
+$Comp
+L Device:R R?
+U 1 1 5AE8F18A
+P 4700 1800
+F 0 "R?" H 4770 1846 50  0000 L CNN
+F 1 "Jumper 0ohm" H 4770 1755 50  0000 L CNN
+F 2 "" V 4630 1800 50  0001 C CNN
+F 3 "~" H 4700 1800 50  0001 C CNN
+	1    4700 1800
+	1    0    0    -1
+$EndComp
+Wire Wire Line
+	4300 1950 4300 2850
+Connection ~ 4300 2850
+Wire Wire Line
+	4300 2850 5325 2850
+Wire Wire Line
+	4700 1950 4700 2750
+Connection ~ 4700 2750
+Wire Wire Line
+	4700 2750 5325 2750
+Text HLabel 4100 1450 0    50   Input ~ 0
+CAN_RX
+Text HLabel 4900 1450 2    50   Input ~ 0
+CAN_TX
+Wire Wire Line
+	4100 1450 4300 1450
+Wire Wire Line
+	4300 1450 4300 1650
+Wire Wire Line
+	4700 1650 4700 1450
+Wire Wire Line
+	4700 1450 4900 1450
 $EndSCHEMATC

Commit message: organizing
Parts:
- gave numbers to parts that had none: 15
Changed lines of the file:
@@
 $EndDescr
 $Comp
-L Interface_CAN_LIN:MCP2551-I-SN U?
+L Interface_CAN_LIN:MCP2551-I-SN U9
 U 1 1 5AD6C5A2
 P 5825 2950
-F 0 "U?" H 5950 3375 50  0000 C CNN
+F 0 "U9" H 5950 3375 50  0000 C CNN
 F 1 "MCP2551-I_SN" H 6200 3300 50  0000 C CNN
 F 2 "Housings_SOIC:SOIC-8_3.9x4.9mm_Pitch1.27mm" H 5825 2450 50  0001 C CIN
@@
 $EndComp
 $Comp
-L Interface_CAN_LIN:MCP2515-EST U?
+L Interface_CAN_LIN:MCP2515-EST U6
 U 1 1 5AD6C74D
 P 3350 3450
-F 0 "U?" H 3450 4300 50  0000 C CNN
+F 0 "U6" H 3450 4300 50  0000 C CNN
 F 1 "MCP2515-E_ST" H 3700 4225 50  0000 C CNN
 F 2 "Housings_SSOP:TSSOP-20_4.4x6.5mm_Pitch0.65mm" H 3350 2550 50  0001 C CIN
@@
 $EndComp
 $Comp
-L open-automation:R_10k R?
+L open-automation:R_10k R18
 U 1 1 5AD70852
 P 5100 3325
-F 0 "R?" H 5170 3371 50  0000 L CNN
+F 0 "R18" H 5170 3371 50  0000 L CNN
 F 1 "4.7k" H 5170 3280 50  0000 L CNN
 F 2 "Resistors_SMD:R_0603" V 5030 3325 50  0001 C CNN
@@
 	5650 1900 5825 1900
 $Comp
-L open-automation:R_10k R?
+L open-automation:R_10k R20
 U 1 1 5AD72887
 P 7100 3275
-F 0 "R?" H 7170 3321 50  0000 L CNN
+F 0 "R20" H 7170 3321 50  0000 L CNN
 F 1 "100" H 7170 3230 50  0000 L CNN
 F 2 "Resistors_SMD:R_0603" V 7030 3275 50  0001 C CNN
@@
 	7100 3500 7100 3425
 $Comp
-L Device:C C?
+L Device:C C21
 U 1 1 5AD73AF7
 P 6650 3650
-F 0 "C?" H 6375 3700 50  0000 L CNN
+F 0 "C21" H 6375 3700 50  0000 L CNN
 F 1 "560pF" H 6325 3625 50  0000 L CNN
 F 2 "Capacitors_SMD:C_0603_HandSoldering" H 6688 3500 50  0001 C CNN
@@
 	6650 3125 6650 3050
 $Comp
-L Power_Protection:SP0502BAHT D?
+L Power_Protection:SP0502BAHT D6
 U 1 1 5AD76474
 P 7850 3350
-F 0 "D?" H 8055 3396 50  0000 L CNN
+F 0 "D6" H 8055 3396 50  0000 L CNN
 F 1 "PESD1CAN" H 8055 3305 50  0000 L CNN
 F 2 "TO_SOT_Packages_SMD:SOT-323_SC-70" H 8075 3300 50  0001 L CNN
@@
 $EndComp
 $Comp
-L Device:C C?
+L Device:C C19
 U 1 1 5AD7FDFC
 P 3175 2200
-F 0 "C?" H 2900 2250 50  0000 L CNN
+F 0 "C19" H 2900 2250 50  0000 L CNN
 F 1 "0.1uF" H 2875 2175 50  0000 L CNN
 F 2 "Capacitors_SMD:C_0603_HandSoldering" H 3213 2050 50  0001 C CNN
@@
 	3175 2000 3350 2000
 $Comp
-L Device:Crystal_Small Y?
+L Device:Crystal_Small Y1
 U 1 1 5AD8276F
 P 2300 3650
-F 0 "Y?" V 2254 3738 50  0000 L CNN
+F 0 "Y1" V 2254 3738 50  0000 L CNN
 F 1 "16MHz" V 2345 3738 50  0000 L CNN
 F 2 "Crystals:Crystal_SMD_HC49-SD_HandSoldering" H 2300 3650 50  0001 C CNN
@@
 	2650 3650 2750 3650
 $Comp
-L Device:C C?
+L Device:C C10
 U 1 1 5AD85611
 P 2000 3500
-F 0 "C?" H 1725 3550 50  0000 L CNN
+F 0 "C10" H 1725 3550 50  0000 L CNN
 F 1 "22pF" H 1700 3475 50  0000 L CNN
 F 2 "Capacitors_SMD:C_0603_HandSoldering" H 2038 3350 50  0001 C CNN
@@
 	4625 2750 4700 2750
 $Comp
-L open-automation:R_10k R?
+L open-automation:R_10k R19
 U 1 1 5ADA3415
 P 6650 3275
-F 0 "R?" H 6720 3321 50  0000 L CNN
+F 0 "R19" H 6720 3321 50  0000 L CNN
 F 1 "100" H 6720 3230 50  0000 L CNN
 F 2 "Resistors_SMD:R_0603" V 6580 3275 50  0001 C CNN
@@
 $EndComp
 $Comp
-L Device:C C?
+L Device:C C20
 U 1 1 5ADA50A9
 P 5650 2100
-F 0 "C?" H 5375 2150 50  0000 L CNN
+F 0 "C20" H 5375 2150 50  0000 L CNN
 F 1 "0.1uF" H 5350 2075 50  0000 L CNN
 F 2 "Capacitors_SMD:C_0603_HandSoldering" H 5688 1950 50  0001 C CNN
@@
 $EndComp
 $Comp
-L Device:C C?
+L Device:C C22
 U 1 1 5ADA5772
 P 7100 3650
-F 0 "C?" H 6825 3700 50  0000 L CNN
+F 0 "C22" H 6825 3700 50  0000 L CNN
 F 1 "560pF" H 6775 3625 50  0000 L CNN
 F 2 "Capacitors_SMD:C_0603_HandSoldering" H 7138 3500 50  0001 C CNN
@@
 $EndComp
 $Comp
-L Device:C C?
+L Device:C C18
 U 1 1 5ADA6ADD
 P 2000 3825
-F 0 "C?" H 1725 3875 50  0000 L CNN
+F 0 "C18" H 1725 3875 50  0000 L CNN
 F 1 "22pF" H 1700 3800 50  0000 L CNN
 F 2 "Capacitors_SMD:C_0603_HandSoldering" H 2038 3675 50  0001 C CNN
@@
 $EndComp
 $Comp
-L power:GND #PWR?
+L power:GND #PWR0102
 U 1 1 5ADD5FFD
 P 1725 3925
-F 0 "#PWR?" H 1725 3675 50  0001 C CNN
+F 0 "#PWR0102" H 1725 3675 50  0001 C CNN
 F 1 "GND" H 1730 3752 50  0000 C CNN
 F 2 "" H 1725 3925 50  0001 C CNN
@@
 	3175 2350 3175 2425
 $Comp
-L power:GND #PWR?
+L power:GND #PWR0103
 U 1 1 5ADD74BB
 P 5100 3525
-F 0 "#PWR?" H 5100 3275 50  0001 C CNN
+F 0 "#PWR0103" H 5100 3275 50  0001 C CNN
 F 1 "GND" H 5105 3352 50  0000 C CNN
 F 2 "" H 5100 3525 50  0001 C CNN
@@
 $EndComp
 $Comp
-L power:GND #PWR?
+L power:GND #PWR0104
 U 1 1 5ADD757D
 P 5825 3525
-F 0 "#PWR?" H 5825 3275 50  0001 C CNN
+F 0 "#PWR0104" H 5825 3275 50  0001 C CNN
 F 1 "GND" H 5830 3352 50  0000 C CNN
 F 2 "" H 5825 3525 50  0001 C CNN
@@
 $EndComp
 $Comp
-L power:GND #PWR?
+L power:GND #PWR0105
 U 1 1 5ADD7680
 P 7100 3875
-F 0 "#PWR?" H 7100 3625 50  0001 C CNN
+F 0 "#PWR0105" H 7100 3625 50  0001 C CNN
 F 1 "GND" H 7105 3702 50  0000 C CNN
 F 2 "" H 7100 3875 50  0001 C CNN
@@
 $EndComp
 $Comp
-L power:GND #PWR?
+L power:GND #PWR0108
 U 1 1 5ADD76B3
 P 5650 2325
-F 0 "#PWR?" H 5650 2075 50  0001 C CNN
+F 0 "#PWR0108" H 5650 2075 50  0001 C CNN
 F 1 "GND" H 5655 2152 50  0000 C CNN
 F 2 "" H 5650 2325 50  0001 C CNN
@@
 $EndComp
 $Comp
-L Device:R R?
+L Device:R R16
 U 1 1 5AE8F142
 P 4300 1800
-F 0 "R?" H 4230 1754 50  0000 R CNN
+F 0 "R16" H 4230 1754 50  0000 R CNN
 F 1 "Jumper 0ohm" H 4230 1845 50  0000 R CNN
 F 2 "" V 4230 1800 50  0001 C CNN
@@
 $EndComp
 $Comp
-L Device:R R?
+L Device:R R17
 U 1 1 5AE8F18A
 P 4700 1800
-F 0 "R?" H 4770 1846 50  0000 L CNN
+F 0 "R17" H 4770 1846 50  0000 L CNN
 F 1 "Jumper 0ohm" H 4770 1755 50  0000 L CNN
 F 2 "" V 4630 1800 50  0001 C CNN

Commit message: update
Parts:
- removed C10, C18: 22pF, Capacitors_SMD:C_0603_HandSoldering, symbol Device:C
- removed C19: 0.1uF, Capacitors_SMD:C_0603_HandSoldering, symbol Device:C
- removed R16, R17: Jumper 0ohm, symbol Device:R
- removed U6: MCP2515-E_ST, Housings_SSOP:TSSOP-20_4.4x6.5mm_Pitch0.65mm, symbol Interface_CAN_LIN:MCP2515-EST
- removed Y1: 16MHz, Crystals:Crystal_SMD_HC49-SD_HandSoldering, symbol Device:Crystal_Small
- C15: renamed from C20; footprint Capacitors_SMD:C_0603_HandSoldering -> Capacitor_SMD:C_0603_1608Metric_Pad0.99x1.00mm_HandSolder
- C16: renamed from C21; footprint Capacitors_SMD:C_0603_HandSoldering -> Capacitor_SMD:C_0603_1608Metric_Pad0.99x1.00mm_HandSolder
- C17: renamed from C22; footprint Capacitors_SMD:C_0603_HandSoldering -> Capacitor_SMD:C_0603_1608Metric_Pad0.99x1.00mm_HandSolder
- R18, R19, R20: footprint Resistors_SMD:R_0603 -> Resistor_SMD:R_0603_1608Metric_Pad0.99x1.00mm_HandSolder
- renumbered D6 to D7, U9 to U8
Connections:
- net labels added: CAN+, CAN-
- net labels removed: CAN_CS, CAN_H, CAN_INT, CAN_L, CAN_RESET, MISO, MOSI, SPI_SCK
- wire segments 64 -> 28
- no-connect marks 7 -> 1

Commit message: update
Parts:
- D7: footprint TO_SOT_Packages_SMD:SOT-323_SC-70 -> Package_TO_SOT_SMD:SOT-323_SC-70_Handsoldering
- U8: footprint Housings_SOIC:SOIC-8_3.9x4.9mm_Pitch1.27mm -> Package_SO:SOIC-8_3.9x4.9mm_P1.27mm
Changed lines of the file:
@@
 F 0 "U8" H 5950 3375 50  0000 C CNN
 F 1 "MCP2551-I_SN" H 6200 3300 50  0000 C CNN
-F 2 "Housings_SOIC:SOIC-8_3.9x4.9mm_Pitch1.27mm" H 5825 2450 50  0001 C CIN
+F 2 "Package_SO:SOIC-8_3.9x4.9mm_P1.27mm" H 5825 2450 50  0001 C CIN
 F 3 "https://www.digikey.com/product-detail/en/microchip-technology/MCP2551-I-SN/MCP2551-I-SN-ND/509452" H 5825 2950 50  0001 C CNN
 F 4 "MCP2551-I/SN" H 5825 2950 50  0001 C CNN "Part Number"
@@
 F 0 "D7" H 8055 3396 50  0000 L CNN
 F 1 "PESD1CAN" H 8055 3305 50  0000 L CNN
-F 2 "TO_SOT_Packages_SMD:SOT-323_SC-70" H 8075 3300 50  0001 L CNN
+F 2 "Package_TO_SOT_SMD:SOT-323_SC-70_Handsoldering" H 8075 3300 50  0001 L CNN
 F 3 "https://www.digikey.com/product-detail/en/nexperia-usa-inc/PESD1CAN-UX/1727-1306-1-ND/4386316" H 7975 3475 50  0001 C CNN
 F 4 "PESD1CAN-UX" H 7850 3350 50  0001 C CNN "Part Number"
