File: usb-interface.sch (KiCad schematic (older format))
At the start: 8 parts

Commit message: update
Parts:
- removed J?: USB_B, open-automation:USB_B-B1HSB6, symbol open-automation:USB_B
- removed P?: USB_A_2, open-automation:USB_A_2, symbol open-automation:USB_A_2
- added C46: C_1uF, Capacitors_SMD:C_0603, symbol open-automation:C_1uF
- added P4: CONN_01X04, Connector_PinHeader_2.54mm:PinHeader_2x04_P2.54mm_Vertical, symbol Connector_Generic:Conn_02x04_Odd_Even
- added R40, R41: R_12k, Resistor_SMD:R_0603_1608Metric_Pad0.99x1.00mm_HandSolder, symbol open-automation:R_12k
- Q4: renamed from Q?; footprint (none) -> Package_TO_SOT_SMD:SOT-23; Part Number (none) -> MMSS8050-H-TP
- U17: renamed from U?; footprint Package_DFN_QFN:QFN-20-1EP_3x3mm_P0.45mm_EP1.6x1.6mm -> Package_DFN_QFN:QFN-24-1EP_3x3mm_P0.45mm_EP1.6x1.6mm
- gave numbers to parts that had none: 4
Connections:
- net labels added: DCD, DSR, EN_ESP, PROG
- wire segments 33 -> 49

Commit message: update
Parts:
- U17: footprint Package_DFN_QFN:QFN-24-1EP_3x3mm_P0.45mm_EP1.6x1.6mm -> Housings_DFN_QFN:QFN-24-1EP_3x3mm_Pitch0.4mm
Changed lines of the file:
@@
 F 0 "U17" H 5800 4100 50  0000 C CNN
 F 1 "USB_IC-CP2104" H 4875 4125 50  0000 C CNN
-F 2 "Package_DFN_QFN:QFN-24-1EP_3x3mm_P0.45mm_EP1.6x1.6mm" H 5425 4125 50  0001 L CNN
+F 2 "Housings_DFN_QFN:QFN-24-1EP_3x3mm_Pitch0.4mm" H 5425 4125 50  0001 L CNN
 F 3 "https://www.digikey.com/product-detail/en/silicon-labs/CP2102N-A01-GQFN20/336-3692-ND/6012517" H 4725 6325 50  0001 C CNN
 F 4 "CP2102N-A01-GQFN20" H 5275 3807 50  0001 C CNN "Part Number"

Commit message: update
Parts:
- C13, C14, C46: footprint Capacitors_SMD:C_0603 -> Capacitor_SMD:C_0603_1608Metric_Pad0.99x1.00mm_HandSolder
- R37: footprint Resistors_SMD:R_0603 -> Resistor_SMD:R_0603_1608Metric_Pad0.99x1.00mm_HandSolder
Changed lines of the file:
@@
 F 0 "C13" H 3675 4700 50  0000 L CNN
 F 1 "C_10uF" H 3500 4550 50  0000 L CNN
-F 2 "Capacitors_SMD:C_0603" H 3875 4925 50  0001 C CNN
+F 2 "Capacitor_SMD:C_0603_1608Metric_Pad0.99x1.00mm_HandSolder" H 3875 4925 50  0001 C CNN
 F 3 "https://www.digikey.com/product-detail/en/murata-electronics-north-america/GRM188R61A106ME69D/490-10475-1-ND/5026393" H 3775 4375 50  0001 C CNN
 F 4 "GRM188R61A106ME69D" H 3900 4825 60  0001 C CNN "Part Number"
@@
 F 0 "C14" H 4115 4671 50  0000 L CNN
 F 1 "C_0.1uF" H 4115 4580 50  0000 L CNN
-F 2 "Capacitors_SMD:C_0603" H 4100 4925 50  0001 C CNN
+F 2 "Capacitor_SMD:C_0603_1608Metric_Pad0.99x1.00mm_HandSolder" H 4100 4925 50  0001 C CNN
 F 3 "https://www.digikey.com/product-detail/en/kemet/C0603C104K5RACTU/399-5089-1-ND/1465623" H 4000 4375 50  0001 C CNN
 F 4 "C0603C104K5RACTU" H 4125 4825 60  0001 C CNN "Part Number"
@@
 F 0 "R37" V 6225 4975 50  0000 C CNN
 F 1 "R_470" V 6150 4975 50  0000 C CNN
-F 2 "Resistors_SMD:R_0603" V 6155 4975 50  0001 C CNN
+F 2 "Resistor_SMD:R_0603_1608Metric_Pad0.99x1.00mm_HandSolder" V 6155 4975 50  0001 C CNN
 F 3 "https://www.digikey.com/product-detail/en/yageo/RC0603FR-07470RL/311-470HRCT-ND/730203" V 6305 4975 50  0001 C CNN
 F 4 "RC0603FR-07470RL" V 6405 5075 60  0001 C CNN "Part Number"
@@
 F 0 "C46" H 5300 4050 50  0000 L CNN
 F 1 "C_1uF" H 5300 3850 50  0000 L CNN
-F 2 "Capacitors_SMD:C_0603" H 5375 4250 50  0001 C CNN
+F 2 "Capacitor_SMD:C_0603_1608Metric_Pad0.99x1.00mm_HandSolder" H 5375 4250 50  0001 C CNN
 F 3 "https://www.digikey.com/product-detail/en/yageo/CC0603ZRY5V7BB105/311-1372-1-ND/2103156" H 5275 3700 50  0001 C CNN
 F 4 "CC0603ZRY5V7BB105" H 5400 4150 60  0001 C CNN "Part Number"

Commit message: update
Connections:
- wire segments 49 -> 52
Changed lines of the file:
@@
 $EndComp
 Wire Wire Line
-	5275 6075 5275 6125
+	5275 6075 5275 6100
 Text HLabel 3425 4475 0    60   Input ~ 0
 5V
@@
 Wire Wire Line
 	9400 2350 9350 2350
+Wire Wire Line
+	5375 6075 5375 6100
+Wire Wire Line
+	5375 6100 5275 6100
+Connection ~ 5275 6100
+Wire Wire Line
+	5275 6100 5275 6125
 $EndSCHEMATC

Commit message: parts swap
Parts:
- removed C13: C_10uF, Capacitor_SMD:C_0603_1608Metric_Pad0.99x1.00mm_HandSolder, symbol open-automation:C_10uF
- removed C46: C_1uF, Capacitor_SMD:C_0603_1608Metric_Pad0.99x1.00mm_HandSolder, symbol open-automation:C_1uF
- added C50: C_1uF, Capacitor_SMD:C_0603_1608Metric_Pad0.99x1.00mm_HandSolder, symbol open-automation:C_1uF
- added C52: C_10uF, Capacitor_SMD:C_0603_1608Metric_Pad0.99x1.00mm_HandSolder, symbol open-automation:C_10uF
- C14: Part Number C0603C104K5RACTU -> C1608X8R1H104K080AB
Changed lines of the file:
@@
 Text HLabel 3425 4475 0    60   Input ~ 0
 5V
-$Comp
-L open-automation:C_10uF C13
-U 1 1 5B160737
-P 3775 4625
-F 0 "C13" H 3675 4700 50  0000 L CNN
-F 1 "C_10uF" H 3500 4550 50  0000 L CNN
-F 2 "Capacitor_SMD:C_0603_1608Metric_Pad0.99x1.00mm_HandSolder" H 3875 4925 50  0001 C CNN
-F 3 "https://www.digikey.com/product-detail/en/murata-electronics-north-america/GRM188R61A106ME69D/490-10475-1-ND/5026393" H 3775 4375 50  0001 C CNN
-F 4 "GRM188R61A106ME69D" H 3900 4825 60  0001 C CNN "Part Number"
-	1    3775 4625
-	1    0    0    -1
-$EndComp
-$Comp
-L open-automation:C_0.1uF C14
-U 1 1 5B1608B3
-P 4000 4625
-F 0 "C14" H 4115 4671 50  0000 L CNN
-F 1 "C_0.1uF" H 4115 4580 50  0000 L CNN
-F 2 "Capacitor_SMD:C_0603_1608Metric_Pad0.99x1.00mm_HandSolder" H 4100 4925 50  0001 C CNN
-F 3 "https://www.digikey.com/product-detail/en/kemet/C0603C104K5RACTU/399-5089-1-ND/1465623" H 4000 4375 50  0001 C CNN
-F 4 "C0603C104K5RACTU" H 4125 4825 60  0001 C CNN "Part Number"
-	1    4000 4625
-	1    0    0    -1
-$EndComp
-Wire Wire Line
-	3425 4475 3775 4475
-Wire Wire Line
-	3775 4475 4000 4475
-Connection ~ 3775 4475
-Wire Wire Line
-	4000 4475 4475 4475
-Connection ~ 4000 4475
-Wire Wire Line
-	4000 4775 4000 4825
-Wire Wire Line
-	4000 4825 3900 4825
 Wire Wire Line
 	3775 4825 3775 4775
@@
 $EndComp
 Wire Wire Line
-	3900 4825 3900 4875
-Connection ~ 3900 4825
-Wire Wire Line
 	3900 4825 3775 4825
 Text Label 4400 4975 0    50   ~ 0
@@
 Wire Wire Line
 	4475 4675 4475 4475
-Connection ~ 4475 4475
 Wire Wire Line
 	4475 4475 4575 4475
@@
 Wire Wire Line
 	7400 4175 7425 4175
-$Comp
-L open-automation:C_1uF C46
-U 1 1 5B17F58C
-P 5275 3950
-F 0 "C46" H 5300 4050 50  0000 L CNN
-F 1 "C_1uF" H 5300 3850 50  0000 L CNN
-F 2 "Capacitor_SMD:C_0603_1608Metric_Pad0.99x1.00mm_HandSolder" H 5375 4250 50  0001 C CNN
-F 3 "https://www.digikey.com/product-detail/en/yageo/CC0603ZRY5V7BB105/311-1372-1-ND/2103156" H 5275 3700 50  0001 C CNN
-F 4 "CC0603ZRY5V7BB105" H 5400 4150 60  0001 C CNN "Part Number"
-	1    5275 3950
-	1    0    0    -1
-$EndComp
 Wire Wire Line
 	5275 4100 5275 4175
@@
 Wire Wire Line
 	5275 6100 5275 6125
+Connection ~ 4475 4475
+Wire Wire Line
+	3900 4825 3900 4875
+Connection ~ 3900 4825
+Wire Wire Line
+	4000 4825 3900 4825
+Wire Wire Line
+	4000 4775 4000 4825
+Wire Wire Line
+	4000 4475 4475 4475
+Connection ~ 4000 4475
+$Comp
+L open-automation:C_0.1uF C14
+U 1 1 5B1608B3
+P 4000 4625
+F 0 "C14" H 4115 4671 50  0000 L CNN
+F 1 "C_0.1uF" H 4115 4580 50  0000 L CNN
+F 2 "Capacitor_SMD:C_0603_1608Metric_Pad0.99x1.00mm_HandSolder" H 4100 4925 50  0001 C CNN
+F 3 "https://www.digikey.com/product-detail/en/tdk-corporation/C1608X7S0J475K080AC/445-9120-1-ND/3661604" H 4000 4375 50  0001 C CNN
+F 4 "C1608X8R1H104K080AB" H 4125 4825 60  0001 C CNN "Part Number"
+	1    4000 4625
+	1    0    0    -1
+$EndComp
+Wire Wire Line
+	3425 4475 3775 4475
+$Comp
+L open-automation:C_10uF C52
+U 1 1 5B27C012
+P 3775 4625
+F 0 "C52" H 3890 4671 50  0000 L CNN
+F 1 "C_10uF" H 3890 4580 50  0000 L CNN
+F 2 "Capacitor_SMD:C_0603_1608Metric_Pad0.99x1.00mm_HandSolder" H 3875 4925 50  0001 C CNN
+F 3 "https://www.digikey.com/product-detail/en/samsung-electro-mechanics/CL10A106MP8NNNC/1276-1871-1-ND/3889957" H 3775 4375 50  0001 C CNN
+F 4 "CL10A106MP8NNNC" H 3900 4825 60  0001 C CNN "Part Number"
+	1    3775 4625
+	1    0    0    -1
+$EndComp
+Connection ~ 3775 4475
+Wire Wire Line
+	3775 4475 4000 4475
+$Comp
+L open-automation:C_1uF C50
+U 1 1 5B2C9FB8
+P 5275 3950
+F 0 "C50" H 5390 3996 50  0000 L CNN
+F 1 "C_1uF" H 5390 3905 50  0000 L CNN
+F 2 "Capacitor_SMD:C_0603_1608Metric_Pad0.99x1.00mm_HandSolder" H 5375 4250 50  0001 C CNN
+F 3 "https://www.digikey.com/product-detail/en/tdk-corporation/CGA3E1X7R1C105M080AC/445-12540-1-ND/3954206" H 5275 3700 50  0001 C CNN
+F 4 "CGA3E1X7R1C105M080AC" H 5400 4150 60  0001 C CNN "Part Number"
+	1    5275 3950
+	1    0    0    -1
+$EndComp
 $EndSCHEMATC

Commit message: starting next revision - 0.2
Connections:
- wire segments 52 -> 50
Changed lines of the file:
@@
-EESchema Schematic File Version 4
+EESchema Schematic File Version 5
 LIBS:open-dash-daughterboard-cache
-EELAYER 26 0
+EELAYER 29 0
 EELAYER END
 $Descr A4 11693 8268
@@
 Wire Wire Line
 	4000 4775 4000 4825
-Wire Wire Line
-	4000 4475 4475 4475
-Connection ~ 4000 4475
 $Comp
 L open-automation:C_0.1uF C14
@@
 	1    0    0    -1
 $EndComp
-Wire Wire Line
-	3425 4475 3775 4475
 $Comp
 L open-automation:C_10uF C52
@@
 	1    0    0    -1
 $EndComp
-Connection ~ 3775 4475
-Wire Wire Line
-	3775 4475 4000 4475
 $Comp
 L open-automation:C_1uF C50
@@
 	1    0    0    -1
 $EndComp
+Wire Wire Line
+	3425 4475 4475 4475
 $EndSCHEMATC
