File: usb-interface-old.sch (KiCad schematic (older format))
At the start: 10 parts, among them P4 CONN_01X04, Q4 Q_NPN_BCE, Q5 Q_PNP_BCE, U17 USB_IC-CP2104

Commit message: finished schematic, starting layout
Changed lines of the file:
@@
 $Descr A4 11693 8268
 encoding utf-8
-Sheet 13 13
+Sheet 7 7
 Title ""
 Date ""
@@
 L Device:Q_NPN_BCE Q4
 U 1 1 5B167526
-P 8025 3575
-F 0 "Q4" H 8216 3621 50  0000 L CNN
-F 1 "Q_NPN_BCE" H 8216 3530 50  0000 L CNN
-F 2 "Package_TO_SOT_SMD:SOT-23" H 8225 3675 50  0001 C CNN
-F 3 "https://www.digikey.com/product-detail/en/micro-commercial-co/MMSS8050-H-TP/MMSS8050-H-TPMSCT-ND/2825945" H 8025 3575 50  0001 C CNN
-F 4 "MMSS8050-H-TP" H 8025 3575 50  0001 C CNN "Part Number"
-	1    8025 3575
+P 2775 3225
+F 0 "Q4" H 2966 3271 50  0000 L CNN
+F 1 "Q_NPN_BCE" H 2966 3180 50  0000 L CNN
+F 2 "Package_TO_SOT_SMD:SOT-23" H 2975 3325 50  0001 C CNN
+F 3 "https://www.digikey.com/product-detail/en/micro-commercial-co/MMSS8050-H-TP/MMSS8050-H-TPMSCT-ND/2825945" H 2775 3225 50  0001 C CNN
+F 4 "MMSS8050-H-TP" H 2775 3225 50  0001 C CNN "Part Number"
+	1    2775 3225
 	1    0    0    -1
 $EndComp
@@
 L Device:Q_PNP_BEC Q5
 U 1 1 5B16769F
-P 8025 4175
-F 0 "Q5" H 8216 4221 50  0000 L CNN
-F 1 "Q_PNP_BCE" H 8216 4130 50  0000 L CNN
-F 2 "Package_TO_SOT_SMD:SOT-23" H 8225 4275 50  0001 C CNN
-F 3 "https://www.digikey.com/product-detail/en/micro-commercial-co/MMSS8550-L-TP/MMSS8550-L-TPMSCT-ND/2827205" H 8025 4175 50  0001 C CNN
-F 4 "MMSS8550-L-TP" H 8025 4175 50  0001 C CNN "Part Number"
-	1    8025 4175
+P 2775 3825
+F 0 "Q5" H 2966 3871 50  0000 L CNN
+F 1 "Q_PNP_BCE" H 2966 3780 50  0000 L CNN
+F 2 "Package_TO_SOT_SMD:SOT-23" H 2975 3925 50  0001 C CNN
+F 3 "https://www.digikey.com/product-detail/en/micro-commercial-co/MMSS8550-L-TP/MMSS8550-L-TPMSCT-ND/2827205" H 2775 3825 50  0001 C CNN
+F 4 "MMSS8550-L-TP" H 2775 3825 50  0001 C CNN "Part Number"
+	1    2775 3825
 	1    0    0    -1
 $EndComp
@@
 L Connector_Generic:Conn_02x04_Odd_Even P4
 U 1 1 5B1561A8
-P 9050 2150
-F 0 "P4" H 9100 2467 50  0000 C CNN
-F 1 "CONN_01X04" H 9100 2376 50  0000 C CNN
-F 2 "Connector_PinHeader_2.54mm:PinHeader_2x04_P2.54mm_Vertical" H 9127 2054 50  0001 L CNN
-F 3 "https://www.digikey.com/products/en?keywords=88738-8000" H 9128 2054 50  0001 L CNN
-F 4 "0887388000" H 9050 2150 50  0001 C CNN "Part Number"
-	1    9050 2150
+P 3800 1800
+F 0 "P4" H 3850 2117 50  0000 C CNN
+F 1 "CONN_01X04" H 3850 2026 50  0000 C CNN
+F 2 "Connector_PinHeader_2.54mm:PinHeader_2x04_P2.54mm_Vertical" H 3877 1704 50  0001 L CNN
+F 3 "https://www.digikey.com/products/en?keywords=88738-8000" H 3878 1704 50  0001 L CNN
+F 4 "0887388000" H 3800 1800 50  0001 C CNN "Part Number"
+	1    3800 1800
 	1    0    0    -1
 $EndComp
@@
 L open-automation:GND #PWR0117
 U 1 1 5B156693
-P 8800 2400
-F 0 "#PWR0117" H 8800 2150 50  0001 C CNN
-F 1 "GND" H 8800 2250 50  0000 C CNN
-F 2 "" H 8800 2400 50  0000 C CNN
-F 3 "" H 8800 2400 50  0000 C CNN
-	1    8800 2400
-	1    0    0    -1
-$EndComp
-Wire Wire Line
-	8800 2400 8800 2350
-Wire Wire Line
-	8800 2350 8850 2350
-Text HLabel 8820 2010 1    60   Input ~ 0
+P 3550 2050
+F 0 "#PWR0117" H 3550 1800 50  0001 C CNN
+F 1 "GND" H 3550 1900 50  0000 C CNN
+F 2 "" H 3550 2050 50  0000 C CNN
+F 3 "" H 3550 2050 50  0000 C CNN
+	1    3550 2050
+	1    0    0    -1
+$EndComp
+Wire Wire Line
+	3550 2050 3550 2000
+Wire Wire Line
+	3550 2000 3600 2000
+Text HLabel 3570 1660 1    60   Input ~ 0
 5V
-Text Label 8700 2150 0    50   ~ 0
+Text Label 3450 1800 0    50   ~ 0
 D_N
-Text Label 8700 2250 0    50   ~ 0
+Text Label 3450 1900 0    50   ~ 0
 D_P
 Wire Wire Line
-	8820 2010 8820 2050
-Wire Wire Line
-	8820 2050 8850 2050
-Wire Wire Line
-	8700 2150 8850 2150
-Wire Wire Line
-	8850 2250 8700 2250
+	3570 1660 3570 1700
+Wire Wire Line
+	3570 1700 3600 1700
+Wire Wire Line
+	3450 1800 3600 1800
+Wire Wire Line
+	3600 1900 3450 1900
 $Comp
 L open-automation:R_12k R40
 U 1 1 5B178943
-P 7575 3575
-F 0 "R40" V 7575 3575 50  0000 C CNN
-F 1 "R_12k" V 7500 3575 50  0000 C CNN
-F 2 "Resistor_SMD:R_0603_1608Metric_Pad0.99x1.00mm_HandSolder" V 7505 3575 50  0001 C CNN
-F 3 "https://www.digikey.com/product-detail/en/yageo/RC0603JR-0712KL/311-12KGRCT-ND/729656" V 7655 3575 50  0001 C CNN
-F 4 "RC0603JR-0712KL" V 7755 3675 60  0001 C CNN "Part Number"
-	1    7575 3575
+P 2325 3225
+F 0 "R40" V 2325 3225 50  0000 C CNN
+F 1 "R_12k" V 2250 3225 50  0000 C CNN
+F 2 "Resistor_SMD:R_0603_1608Metric_Pad0.99x1.00mm_HandSolder" V 2255 3225 50  0001 C CNN
+F 3 "https://www.digikey.com/product-detail/en/yageo/RC0603JR-0712KL/311-12KGRCT-ND/729656" V 2405 3225 50  0001 C CNN
+F 4 "RC0603JR-0712KL" V 2505 3325 60  0001 C CNN "Part Number"
+	1    2325 3225
 	0    1    1    0
 $EndComp
@@
 L open-automation:R_12k R41
 U 1 1 5B178CF5
-P 7575 4175
-F 0 "R41" V 7575 4175 50  0000 C CNN
-F 1 "R_12k" V 7500 4175 50  0000 C CNN
-F 2 "Resistor_SMD:R_0603_1608Metric_Pad0.99x1.00mm_HandSolder" V 7505 4175 50  0001 C CNN
-F 3 "https://www.digikey.com/product-detail/en/yageo/RC0603JR-0712KL/311-12KGRCT-ND/729656" V 7655 4175 50  0001 C CNN
-F 4 "RC0603JR-0712KL" V 7755 4275 60  0001 C CNN "Part Number"
-	1    7575 4175
+P 2325 3825
+F 0 "R41" V 2325 3825 50  0000 C CNN
+F 1 "R_12k" V 2250 3825 50  0000 C CNN
+F 2 "Resistor_SMD:R_0603_1608Metric_Pad0.99x1.00mm_HandSolder" V 2255 3825 50  0001 C CNN
+F 3 "https://www.digikey.com/product-detail/en/yageo/RC0603JR-0712KL/311-12KGRCT-ND/729656" V 2405 3825 50  0001 C CNN
+F 4 "RC0603JR-0712KL" V 2505 3925 60  0001 C CNN "Part Number"
+	1    2325 3825
 	0    1    1    0
 $EndComp
 Wire Wire Line
-	7725 4175 7825 4175
-Wire Wire Line
-	7825 3575 7725 3575
-Text HLabel 8150 3250 2    60   Input ~ 0
+	2475 3825 2575 3825
+Wire Wire Line
+	2575 3225 2475 3225
+Text HLabel 2900 2900 2    60   Input ~ 0
 EN_ESP
 Wire Wire Line
-	8150 3250 8125 3250
-Wire Wire Line
-	8125 3250 8125 3375
-Text HLabel 8150 4500 2    60   Input ~ 0
+	2900 2900 2875 2900
+Wire Wire Line
+	2875 2900 2875 3025
+Text HLabel 2900 4150 2    60   Input ~ 0
 PROG
 Wire Wire Line
-	8150 4500 8125 4500
-Wire Wire Line
-	8125 4500 8125 4375
-Text Label 7150 3575 0    50   ~ 0
+	2900 4150 2875 4150
+Wire Wire Line
+	2875 4150 2875 4025
+Text Label 1900 3225 0    50   ~ 0
 DTR
 Wire Wire Line
-	7150 3575 7350 3575
-Text Label 7150 4175 0    50   ~ 0
+	1900 3225 2100 3225
+Text Label 1900 3825 0    50   ~ 0
 RTS
 Wire Wire Line
-	7150 4175 7400 4175
-Wire Wire Line
-	8125 3975 8125 3925
-Wire Wire Line
-	8125 3925 7350 3925
-Wire Wire Line
-	7350 3925 7350 3575
-Connection ~ 7350 3575
-Wire Wire Line
-	7350 3575 7425 3575
-Wire Wire Line
-	8125 3775 8125 3825
-Wire Wire Line
-	8125 3825 7400 3825
-Wire Wire Line
-	7400 3825 7400 4175
-Connection ~ 7400 4175
-Wire Wire Line
-	7400 4175 7425 4175
+	1900 3825 2150 3825
+Wire Wire Line
+	2875 3625 2875 3575
+Wire Wire Line
+	2875 3575 2100 3575
+Wire Wire Line
+	2100 3575 2100 3225
+Connection ~ 2100 3225
+Wire Wire Line
+	2100 3225 2175 3225
+Wire Wire Line
+	2875 3425 2875 3475
+Wire Wire Line
+	2875 3475 2150 3475
+Wire Wire Line
+	2150 3475 2150 3825
+Connection ~ 2150 3825
+Wire Wire Line
+	2150 3825 2175 3825
 Wire Wire Line
 	5275 4100 5275 4175
@@
 Wire Wire Line
 	6025 4575 5975 4575
-Text Label 9400 2050 0    50   ~ 0
+Text Label 4150 1700 0    50   ~ 0
 DCD
-Text Label 9400 2150 0    50   ~ 0
+Text Label 4150 1800 0    50   ~ 0
 DTR
-Text Label 9400 2250 0    50   ~ 0
+Text Label 4150 1900 0    50   ~ 0
 DSR
 Wire Wire Line
-	9400 2250 9350 2250
-Wire Wire Line
-	9400 2150 9350 2150
-Wire Wire Line
-	9400 2050 9350 2050
-Text Label 9400 2350 0    50   ~ 0
+	4150 1900 4100 1900
+Wire Wire Line
+	4150 1800 4100 1800
+Wire Wire Line
+	4150 1700 4100 1700
+Text Label 4150 2000 0    50   ~ 0
 RTS
 Wire Wire Line
-	9400 2350 9350 2350
+	4150 2000 4100 2000
 Wire Wire Line
 	5375 6075 5375 6100
@@
 U 1 1 5B1608B3
 P 4000 4625
-F 0 "C14" H 4115 4671 50  0000 L CNN
-F 1 "C_0.1uF" H 4115 4580 50  0000 L CNN
+F 0 "C14" H 4100 4650 50  0000 L CNN
+F 1 "C_0.1uF" H 4000 4550 50  0000 L CNN
 F 2 "Capacitor_SMD:C_0603_1608Metric_Pad0.99x1.00mm_HandSolder" H 4100 4925 50  0001 C CNN
 F 3 "https://www.digikey.com/product-detail/en/tdk-corporation/C1608X7S0J475K080AC/445-9120-1-ND/3661604" H 4000 4375 50  0001 C CNN
@@
 U 1 1 5B27C012
 P 3775 4625
-F 0 "C52" H 3890 4671 50  0000 L CNN
-F 1 "C_10uF" H 3890 4580 50  0000 L CNN
+F 0 "C52" H 3500 4650 50  0000 L CNN
+F 1 "C_10uF" H 3500 4550 50  0000 L CNN
 F 2 "Capacitor_SMD:C_0603_1608Metric_Pad0.99x1.00mm_HandSolder" H 3875 4925 50  0001 C CNN
 F 3 "https://www.digikey.com/product-detail/en/samsung-electro-mechanics/CL10A106MP8NNNC/1276-1871-1-ND/3889957" H 3775 4375 50  0001 C CNN
