File: usb.sch (KiCad schematic (older format))
At the start: 15 parts, among them J4 USB_MINI_B, Q1 Q_NPN_BCE, Q2 Q_PNP_BCE, U7 FT231XS

Commit message: Finished layout (v0.2), sent to board house
Parts:
- removed C1: C_47pF, Capacitor_SMD:C_0603_1608Metric_Pad1.05x0.95mm_HandSolder, symbol open-automation:C_47pF
- removed R1, R2: R_27, Resistor_SMD:R_0603_1608Metric_Pad1.05x0.95mm_HandSolder, symbol open-automation:R_27
- removed R3, R4: R_10k, Resistor_SMD:R_0603_1608Metric_Pad1.05x0.95mm_HandSolder, symbol open-automation:R_10k
- removed R5: R_10k, Resistor_SMD:R_0603_1608Metric_Pad0.99x1.00mm_HandSolder, symbol open-automation:R_10k
- added C4: C_47pF, Capacitor_SMD:C_0603_1608Metric_Pad1.05x0.95mm_HandSolder, symbol open-automation:C_47pF
- added R4, R5: R_27, Resistor_SMD:R_0603_1608Metric_Pad1.05x0.95mm_HandSolder, symbol open-automation:R_27
- added R6, R7, R8: R_10K, Resistor_SMD:R_0603_1608Metric_Pad1.05x0.95mm_HandSolder, symbol open-automation:R_10K
- C5: renamed from C2; Part Number GRM188R60G476ME15D -> GCM1885C2A470FA16D; Website (none) -> https://www.digikey.com/product-detail/en/murata-electronic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
- C6: renamed from C3; Part Number CL10F104ZO8NNNC -> C1608X8R1H104K080AB
- C8: renamed from C5; Part Number CL10F104ZO8NNNC -> C1608X8R1H104K080AB
- renumbered C4 to C7, R6 to R9, U7 to U6

Commit message: 0.2 revisions
Connections:
- net labels added: USB_RXD, USB_TXD
- wire segments 46 -> 47
Changed lines of the file:
@@
 Text Label 3650 3800 2    50   ~ 0
 USBDP
+Text Label 2950 1300 0    50   ~ 0
+USBDM
+Wire Wire Line
+	2950 1400 2900 1400
 Text Label 2950 1400 0    50   ~ 0
-USBDM
-Wire Wire Line
-	2950 1400 2900 1400
-Text Label 2950 1300 0    50   ~ 0
 USBDP
 Wire Wire Line
@@
 	5500 3400 5450 3400
 Text Label 5500 3400 0    50   ~ 0
-TXD
+USB_TXD
 Text Label 5500 3500 0    50   ~ 0
-RXD
+USB_RXD
 Wire Wire Line
 	1350 1150 1400 1150
 Wire Wire Line
 	1400 1050 1350 1050
+Text Label 1400 1150 0    50   ~ 0
+USB_TXD
 Text Label 1400 1050 0    50   ~ 0
-TXD
-Text Label 1400 1150 0    50   ~ 0
-RXD
+USB_RXD
 Wire Wire Line
 	4850 3050 4850 3100
@@
 	1    0    0    -1
 $EndComp
+Text Label 4000 3400 2    50   ~ 0
+3V3OUT
+Wire Wire Line
+	4000 3400 4050 3400
 $EndSCHEMATC

Commit message: sent 0.2 revision to pcb house
Parts:
- removed R8: R_10K, Resistor_SMD:R_0603_1608Metric_Pad1.05x0.95mm_HandSolder, symbol open-automation:R_10K
- removed R9: R_4K7, Resistor_SMD:R_0603_1608Metric_Pad1.05x0.95mm_HandSolder, symbol open-automation:R_4K7
- added D7: D_1N5819HW, Diode_SMD:D_SOD-123, symbol open-automation:D_1N5819HW
Connections:
- net labels removed: VBUS
- wire segments 47 -> 44
Changed lines of the file:
@@
 Text Label 1400 1250 0    50   ~ 0
 5V
-Text Label 2950 1100 0    50   ~ 0
-VBUS
 Wire Wire Line
 	4000 4000 4050 4000
@@
 Wire Wire Line
 	5500 4300 5450 4300
-Text Label 8350 4000 0    50   ~ 0
-VSENSE
-Wire Wire Line
-	8350 3950 8350 4000
-Wire Wire Line
-	8350 3500 8350 3550
-Text Label 8350 3500 0    50   ~ 0
-VBUS
-Wire Wire Line
-	8350 4450 8350 4400
-$Comp
-L open-automation:GND #PWR021
-U 1 1 5CC969CC
-P 8350 4450
-AR Path="/5B15E02A/5CC969CC" Ref="#PWR021"  Part="1"
-AR Path="/5C04BFCE/5CC969CC" Ref="#PWR?"  Part="1"
-F 0 "#PWR021" H 8350 4200 50  0001 C CNN
-F 1 "GND" H 8355 4277 50  0000 C CNN
-F 2 "" H 8350 4450 50  0000 C CNN
-F 3 "" H 8350 4450 50  0000 C CNN
-	1    8350 4450
-	1    0    0    -1
-$EndComp
-$Comp
-L open-automation:R_4K7 R9
-U 1 1 5CC82187
-P 8600 3750
-F 0 "R9" V 8600 4050 50  0000 R CNN
-F 1 "R_4K7" V 8600 4300 50  0000 R CNN
-F 2 "Resistor_SMD:R_0603_1608Metric_Pad1.05x0.95mm_HandSolder" H 8575 3575 50  0001 C CNN
-F 3 "https://industrial.panasonic.com/ww/products/resistors/chip-resistors/general-purpose-chip-resistors/thick-film-chip-resistors/ERJ3GEYJ472V" H 8600 3500 50  0001 C CNN
-F 4 "ERJ-3GEYJ472V" H 8600 3825 60  0001 C CNN "Part Number"
-F 5 "https://www.digikey.com/product-detail/en/panasonic-electronic-components/ERJ-3GEYJ472V/P4.7KGCT-ND/135199" H 8600 3750 50  0001 C CNN "Website"
-	1    8600 3750
-	0    -1   -1   0
-$EndComp
 Wire Wire Line
 	6500 4250 6500 3900
@@
 	1    6700 4250
 	0    -1   -1   0
-$EndComp
-$Comp
-L open-automation:R_10K R8
-U 1 1 5CC21EE4
-P 8350 4200
-F 0 "R8" H 8420 4246 50  0000 L CNN
-F 1 "R_10K" H 8420 4155 50  0000 L CNN
-F 2 "Resistor_SMD:R_0603_1608Metric_Pad1.05x0.95mm_HandSolder" V 8280 4200 50  0001 C CNN
-F 3 "" V 8430 4200 50  0001 C CNN
-F 4 "RC0603JR-0710KL" V 8530 4300 60  0001 C CNN "Part Number"
-	1    8350 4200
-	1    0    0    -1
 $EndComp
 $Comp
@@
 Wire Wire Line
 	4000 3400 4050 3400
+Text Label 3250 1100 0    50   ~ 0
+5V
+$Comp
+L open-automation:D_1N5819HW D7
+U 1 1 5CD8937E
+P 3100 1100
+F 0 "D7" H 3100 884 50  0000 C CNN
+F 1 "D_1N5819HW" H 3100 975 50  0000 C CNN
+F 2 "Diode_SMD:D_SOD-123" H 3100 925 50  0001 C CNN
+F 3 "http://www.diodes.com/_files/datasheets/ds23022.pdf" H 3100 1100 50  0001 C CNN
+F 4 "1N5819HW-7-F" H 3100 1400 50  0001 C CNN "Part Number"
+F 5 "https://www.digikey.com/product-detail/en/diodes-incorporated/1N5819HW-7-F/1N5819HW-FDICT-ND/815283" H 3200 1300 50  0001 C CNN "Website"
+	1    3100 1100
+	-1   0    0    1
+$EndComp
 $EndSCHEMATC
