File: open-dash-daughterboard/environment.sch (KiCad schematic (older format))
At the start: 4 parts, among them U2 TSL45315CL, U6 SI7020-A20

Commit message: updated to v5 kicad
Parts:
- C10, C9: symbol C_0.1uF -> open-automation:C_0.1uF
- U2: symbol TSL45315CL -> open-automation:TSL45315CL
- U6: symbol SI7020-A20 -> open-automation:SI7020-A20
Connections:
- wire segments 16 -> 18
Changed lines of the file:
@@
-EESchema Schematic File Version 2
-LIBS:ESP32-footprints-Shem-Lib
-LIBS:espressif-xess
-LIBS:dk_Interface-Drivers-Receivers-Transceivers
-LIBS:open-automation
+EESchema Schematic File Version 4
 LIBS:open-dash-daughterboard-cache
-EELAYER 25 0
+EELAYER 26 0
 EELAYER END
 $Descr A4 11693 8268
@@
 3V3
 $Comp
-L GND #PWR023
+L open-automation:GND #PWR023
 U 1 1 59C50BD3
 P 3850 3575
@@
 SDA
 $Comp
-L SI7020-A20 U6
+L open-automation:SI7020-A20 U6
 U 1 1 59C50BD4
 P 4350 3525
@@
 $EndComp
 $Comp
-L C_0.1uF C9
+L open-automation:C_0.1uF C9
 U 1 1 59C50BD5
 P 3550 3625
@@
 $EndComp
 $Comp
-L GND #PWR024
+L open-automation:GND #PWR024
 U 1 1 59C50BD6
 P 3550 3825
@@
 SCL
 $Comp
-L GND #PWR025
+L open-automation:GND #PWR025
 U 1 1 59C50BD8
 P 7425 3675
@@
 3V3
 $Comp
-L C_0.1uF C10
+L open-automation:C_0.1uF C10
 U 1 1 59C50BDA
 P 7200 3700
@@
 Temp-Humidty
 Wire Wire Line
-	3400 3425 3900 3425
+	3400 3425 3550 3425
 Wire Wire Line
 	3900 3525 3850 3525
@@
 	7425 3625 7475 3625
 Wire Wire Line
-	7100 3525 7475 3525
+	7100 3525 7200 3525
 Wire Wire Line
 	7200 3525 7200 3550
 $Comp
-L GND #PWR026
+L open-automation:GND #PWR026
 U 1 1 59E2A131
 P 7200 3900
@@
 	8375 3500 8425 3500
 $Comp
-L TSL45315CL U2
+L open-automation:TSL45315CL U2
 U 1 1 59E41F23
 P 7925 3625
@@
 	1    0    0    -1
 $EndComp
+Wire Wire Line
+	3550 3425 3900 3425
+Wire Wire Line
+	7200 3525 7475 3525
 $EndSCHEMATC
