File: open-dash-daughterboard/microcontroller.sch (KiCad schematic (older format))
At the start: 7 parts, among them J1 Conn_02x05_Odd_Even, U1 ESP-WROOM-32

Commit message: updated to v5 kicad
Parts:
- C4: symbol C_10uF -> open-automation:C_10uF
- C6: symbol C_1uF -> open-automation:C_1uF
- J1: symbol Conn_02x05_Odd_Even -> open-automation:Conn_02x05_Odd_Even
- R10, R6, R9: symbol R_10k -> open-automation:R_10k
- U1: symbol ESP-WROOM-32 -> open-automation:ESP-WROOM-32
Connections:
- wire segments 39 -> 42
Changed lines of the file:
@@
-EESchema Schematic File Version 2
-LIBS:ESP32-footprints-Shem-Lib
-LIBS:espressif-xess
-LIBS:dk_Interface-Drivers-Receivers-Transceivers
-LIBS:open-automation
+EESchema Schematic File Version 4
 LIBS:open-dash-daughterboard-cache
-EELAYER 25 0
+EELAYER 26 0
 EELAYER END
 $Descr A4 11693 8268
@@
 $EndDescr
 $Comp
-L GND #PWR01
+L open-automation:GND #PWR01
 U 1 1 59097974
 P 4825 2750
@@
 IO2
 $Comp
-L ESP-WROOM-32 U1
+L open-automation:ESP-WROOM-32 U1
 U 1 1 590979AF
 P 5775 3450
@@
 SDA
 $Comp
-L GND #PWR02
+L open-automation:GND #PWR02
 U 1 1 590979B0
 P 8150 3500
@@
 V_USB
 $Comp
-L GND #PWR03
+L open-automation:GND #PWR03
 U 1 1 590979B2
 P 8750 3500
@@
 	6625 4100 6725 4100
 Wire Wire Line
-	6175 4650 6175 4750
+	6175 4650 6175 4700
 Wire Wire Line
 	4775 3000 4875 3000
@@
 Microcontroller
 $Comp
-L C_1uF C6
+L open-automation:C_1uF C6
 U 1 1 59C55B03
 P 2825 3775
@@
 $EndComp
 $Comp
-L GND #PWR04
+L open-automation:GND #PWR04
 U 1 1 59C55B05
 P 2625 4025
@@
 	2425 3925 2425 3975
 Wire Wire Line
-	2425 3975 2825 3975
+	2425 3975 2625 3975
 Wire Wire Line
 	2825 3975 2825 3925
@@
 	8100 3750 8200 3750
 $Comp
-L R_10k R6
+L open-automation:R_10k R6
 U 1 1 59C609F8
 P 6400 4700
@@
 Connection ~ 6175 4700
 $Comp
-L GND #PWR05
+L open-automation:GND #PWR05
 U 1 1 59C60A9D
 P 6600 4700
@@
 	6725 3900 6625 3900
 $Comp
-L Conn_02x05_Odd_Even J1
+L open-automation:Conn_02x05_Odd_Even J1
 U 1 1 59C6C1C0
 P 8400 3750
@@
 SDA
 $Comp
-L R_10k R10
+L open-automation:R_10k R10
 U 1 1 59C83F25
 P 3450 3700
@@
 $EndComp
 $Comp
-L R_10k R9
+L open-automation:R_10k R9
 U 1 1 59C83F7C
 P 3350 3700
@@
 3V3
 $Comp
-L C_10uF C4
+L open-automation:C_10uF C4
 U 1 1 5A10664F
 P 2425 3775
@@
 	2425 3625 2425 3525
 Wire Wire Line
-	2425 3525 2825 3525
+	2425 3525 2625 3525
 Wire Wire Line
 	2625 3525 2625 3400
@@
 Wire Notes Line
 	3000 4275 2075 4275
+Wire Wire Line
+	2625 3975 2825 3975
+Wire Wire Line
+	6175 4700 6175 4750
+Wire Wire Line
+	2625 3525 2825 3525
 $EndSCHEMATC
