File: open-dash-daughterboard/power.sch (KiCad schematic (older format))
At the start: 17 parts, among them Q1 Q_NMOS_GSD_AOD4184A, U11 NCP1117LPST33T3G, U3 LM2576, U5 Power-Monitor-INA219

Commit message: merged in smart regulator
Parts:
- BATTERY1, PANEL1: symbol Conn_01x02 -> CONN_01X02
- C1: symbol CP -> C_100uF
- C2: symbol CP -> C_1000uF
Changed lines of the file:
@@
 LIBS:ESP32-footprints-Shem-Lib
 LIBS:espressif-xess
+LIBS:dk_Interface-Drivers-Receivers-Transceivers
+LIBS:open-automation
 LIBS:open-dash-daughterboard-cache
 EELAYER 25 0
@@
 V_USB
 $Comp
-L CP C1
+L C_100uF C1
 U 1 1 593709F5
 P 7900 3475
@@
 $EndComp
 $Comp
-L CP C2
+L C_1000uF C2
 U 1 1 5968D146
 P 9900 3825
@@
 V_MAIN
 $Comp
-L Conn_01x02 BATTERY1
+L CONN_01X02 BATTERY1
 U 1 1 597573B9
 P 5625 5775
@@
 V_MAIN
 $Comp
-L Conn_01x02 PANEL1
+L CONN_01X02 PANEL1
 U 1 1 59C5AB51
 P 5650 6275

Commit message: updated to v5 kicad
Parts:
- BATTERY1, PANEL1: symbol CONN_01X02 -> open-automation:CONN_01X02
- C1: symbol C_100uF -> open-automation:C_100uF
- C2: symbol C_1000uF -> open-automation:C_1000uF
- C3: symbol C -> open-automation:C
- C8: symbol C_0.1uF -> open-automation:C_0.1uF
- D1: symbol D_Schottky -> open-automation:D_Schottky
- D4: symbol LED -> open-automation:LED
- L1: symbol L -> open-automation:L
- Q1: symbol Q_NMOS_GSD_AOD4184A -> open-automation:Q_NMOS_GSD_AOD4184A
- R1: symbol R_10m -> open-automation:R_10m
- R11, R8: symbol R_10k -> open-automation:R_10k
- R7: symbol R -> open-automation:R
- U11: symbol NCP1117LPST33T3G -> open-automation:NCP1117LPST33T3G
- U3: symbol LM2576 -> open-automation:LM2576
- U5: symbol Power-Monitor-INA219 -> open-automation:Power-Monitor-INA219
Connections:
- wire segments 56 -> 67
Changed lines of the file:
@@
-EESchema Schematic File Version 2
-LIBS:ESP32-footprints-Shem-Lib
-LIBS:espressif-xess
-LIBS:dk_Interface-Drivers-Receivers-Transceivers
-LIBS:open-automation
+EESchema Schematic File Version 4
 LIBS:open-dash-daughterboard-cache
-EELAYER 25 0
+EELAYER 26 0
 EELAYER END
 $Descr A4 11693 8268
@@
 $EndDescr
 $Comp
-L LM2576 U3
+L open-automation:LM2576 U3
 U 1 1 5936E607
 P 8800 3675
@@
 V_USB
 $Comp
-L C_100uF C1
+L open-automation:C_100uF C1
 U 1 1 593709F5
 P 7900 3475
@@
 $EndComp
 $Comp
-L C_1000uF C2
+L open-automation:C_1000uF C2
 U 1 1 5968D146
 P 9900 3825
@@
 $EndComp
 $Comp
-L L L1
+L open-automation:L L1
 U 1 1 5969017D
 P 9650 3675
@@
 $EndComp
 $Comp
-L GND #PWR010
+L open-automation:GND #PWR010
 U 1 1 59690AC9
 P 9900 4025
@@
 $EndComp
 $Comp
-L GND #PWR011
+L open-automation:GND #PWR011
 U 1 1 59690B3F
 P 7700 3475
@@
 $EndComp
 $Comp
-L GND #PWR012
+L open-automation:GND #PWR012
 U 1 1 59690D86
 P 9450 4075
@@
 $EndComp
 $Comp
-L D_Schottky D1
+L open-automation:D_Schottky D1
 U 1 1 59690FC6
 P 9450 3875
@@
 V_MAIN
 $Comp
-L CONN_01X02 BATTERY1
+L open-automation:CONN_01X02 BATTERY1
 U 1 1 597573B9
 P 5625 5775
@@
 BATTERY
 $Comp
-L GND #PWR013
+L open-automation:GND #PWR013
 U 1 1 59757643
 P 5375 5875
@@
 3V3
 $Comp
-L GND #PWR014
+L open-automation:GND #PWR014
 U 1 1 598E598C
 P 8250 3825
@@
 power_EN
 $Comp
-L GND #PWR015
+L open-automation:GND #PWR015
 U 1 1 598F6B7D
 P 8225 5100
@@
 V_MAIN
 $Comp
-L C C3
+L open-automation:C C3
 U 1 1 598F70D3
 P 9125 5150
@@
 $EndComp
 $Comp
-L GND #PWR016
+L open-automation:GND #PWR016
 U 1 1 598F7252
 P 9125 5400
@@
 $EndComp
 $Comp
-L LED D4
+L open-automation:LED D4
 U 1 1 598F7872
 P 9525 5200
@@
 $EndComp
 $Comp
-L GND #PWR017
+L open-automation:GND #PWR017
 U 1 1 598F7A99
 P 9525 5750
@@
 $EndComp
 $Comp
-L GND #PWR018
+L open-automation:GND #PWR018
 U 1 1 59A20D2D
 P 8000 4075
@@
 3V3
 $Comp
-L C_0.1uF C8
+L open-automation:C_0.1uF C8
 U 1 1 59C52B59
 P 4275 4275
@@
 $EndComp
 $Comp
-L GND #PWR019
+L open-automation:GND #PWR019
 U 1 1 59C53560
 P 4075 4275
@@
 	8225 5100 8225 5050
 Wire Wire Line
-	9025 4950 9525 4950
+	9025 4950 9125 4950
 Wire Wire Line
 	9450 3725 9450 3675
@@
 Connection ~ 9850 3675
 Wire Wire Line
-	9850 3425 9850 3675
-Wire Wire Line
-	9800 3675 9900 3675
-Wire Wire Line
-	9400 3675 9500 3675
+	9850 3425 9850 3575
+Wire Wire Line
+	9800 3675 9850 3675
+Wire Wire Line
+	9400 3675 9450 3675
 Wire Wire Line
 	9400 3575 9850 3575
@@
 Connection ~ 8250 3475
 Wire Wire Line
-	8250 3375 8250 3575
+	8250 3375 8250 3475
 Wire Wire Line
 	7700 3475 7750 3475
@@
 	8250 3775 8300 3775
 Wire Wire Line
-	7750 3675 8300 3675
+	7750 3675 8000 3675
 Wire Wire Line
 	5375 5875 5375 5825
@@
 	4575 4875 4625 4875
 Wire Wire Line
-	4325 4950 4075 4950
+	4325 4950 4150 4950
 Wire Wire Line
 	4150 4950 4150 4875
@@
 Connection ~ 4150 4525
 Wire Wire Line
-	4500 4275 4425 4275
+	4500 4275 4450 4275
 Connection ~ 4450 4275
 Wire Wire Line
@@
 	5550 4575 5700 4575
 $Comp
-L GND #PWR020
+L open-automation:GND #PWR020
 U 1 1 59C52714
 P 4575 4900
@@
 V_MAIN
 $Comp
-L CONN_01X02 PANEL1
+L open-automation:CONN_01X02 PANEL1
 U 1 1 59C5AB51
 P 5650 6275
@@
 V_PANEL
 $Comp
-L GND #PWR021
+L open-automation:GND #PWR021
 U 1 1 59C5AB58
 P 5400 6375
@@
 	5350 6225 5450 6225
 $Comp
-L Power-Monitor-INA219 U5
+L open-automation:Power-Monitor-INA219 U5
 U 1 1 59C5E21B
 P 5100 4725
@@
 $EndComp
 $Comp
-L R_10k R8
+L open-automation:R_10k R8
 U 1 1 59C5FC56
 P 8000 3875
@@
 $EndComp
 $Comp
-L GND #PWR022
+L open-automation:GND #PWR022
 U 1 1 59C6263F
 P 5700 4550
@@
 	4525 3275 4675 3275
 $Comp
-L R R7
+L open-automation:R R7
 U 1 1 59E3D0E8
 P 4875 2725
@@
 	4875 2475 4875 2575
 Wire Wire Line
-	4875 2875 4875 2975
+	4875 2875 4875 2925
 Text GLabel 4725 2925 0    60   Input ~ 0
 PANEL_SW
@@
 Connection ~ 4875 2925
 Wire Wire Line
-	4325 4525 4075 4525
+	4325 4525 4150 4525
 Wire Wire Line
 	5200 3275 5075 3275
 $Comp
-L R_10k R11
+L open-automation:R_10k R11
 U 1 1 59E4131F
 P 9525 5550
@@
 	5675 4675 5550 4675
 $Comp
-L NCP1117LPST33T3G U11
+L open-automation:NCP1117LPST33T3G U11
 U 1 1 5A105FD6
 P 8675 4950
@@
 $EndComp
 $Comp
-L R_10m R1
+L open-automation:R_10m R1
 U 1 1 5A108421
 P 4150 4750
@@
 $EndComp
 $Comp
-L Q_NMOS_GSD_AOD4184A Q1
+L open-automation:Q_NMOS_GSD_AOD4184A Q1
 U 1 1 5A109055
 P 4800 3250
@@
 	0    1    1    0
 $EndComp
+Wire Wire Line
+	9425 4950 9525 4950
+Wire Wire Line
+	9125 4950 9425 4950
+Wire Wire Line
+	9450 3675 9500 3675
+Wire Wire Line
+	9850 3575 9850 3675
+Wire Wire Line
+	9850 3675 9900 3675
+Wire Wire Line
+	8250 3475 8250 3575
+Wire Wire Line
+	8000 3675 8300 3675
+Wire Wire Line
+	4150 4950 4075 4950
+Wire Wire Line
+	4150 4525 4075 4525
+Wire Wire Line
+	4450 4275 4425 4275
+Wire Wire Line
+	4875 2925 4875 2975
 $EndSCHEMATC
