File: open-dash-daughterboard/switches.sch (KiCad schematic (older format))
At the start: 12 parts, among them P5 USB_A_2, U10 touchpad, U4 housing-mounts

Commit message: merged in smart regulator
Parts:
- FACTORY1, PROG1, REBOOT1: symbol SW_Push -> SW_PUSH
Changed lines of the file:
@@
 LIBS:ESP32-footprints-Shem-Lib
 LIBS:espressif-xess
+LIBS:dk_Interface-Drivers-Receivers-Transceivers
+LIBS:open-automation
 LIBS:open-dash-daughterboard-cache
 EELAYER 25 0
@@
 $EndComp
 $Comp
-L SW_Push FACTORY1
+L SW_PUSH FACTORY1
 U 1 1 59C587B8
 P 3725 3975
@@
 3V3
 $Comp
-L SW_Push REBOOT1
+L SW_PUSH REBOOT1
 U 1 1 59E3EE49
 P 4675 3975
@@
 3V3
 $Comp
-L SW_Push PROG1
+L SW_PUSH PROG1
 U 1 1 59E3F1CB
 P 5450 3975

Commit message: updated to v5 kicad
Parts:
- D2, D3, D5: symbol LED -> open-automation:LED
- FACTORY1, PROG1, REBOOT1: symbol SW_PUSH -> open-automation:SW_PUSH
- P5: symbol USB_A_2 -> open-automation:USB_A_2
- R2, R3, R4: symbol R_10k -> open-automation:R_10k
- U10: symbol touchpad -> open-automation:touchpad
- U4: symbol housing-mounts -> open-automation:housing-mounts
Connections:
- wire segments 25 -> 29
Changed lines of the file:
@@
-EESchema Schematic File Version 2
-LIBS:ESP32-footprints-Shem-Lib
-LIBS:espressif-xess
-LIBS:dk_Interface-Drivers-Receivers-Transceivers
-LIBS:open-automation
+EESchema Schematic File Version 4
 LIBS:open-dash-daughterboard-cache
-EELAYER 25 0
+EELAYER 26 0
 EELAYER END
 $Descr A4 11693 8268
@@
 $EndDescr
 $Comp
-L LED D2
+L open-automation:LED D2
 U 1 1 59092D24
 P 3725 3125
@@
 	7975 4600 8075 4600
 $Comp
-L touchpad U10
+L open-automation:touchpad U10
 U 1 1 590F8D3B
 P 8475 4600
@@
 3V3
 $Comp
-L USB_A_2 P5
+L open-automation:USB_A_2 P5
 U 1 1 59693837
 P 8350 2800
@@
 $EndComp
 $Comp
-L GND #PWR06
+L open-automation:GND #PWR06
 U 1 1 5969393D
 P 8500 3200
@@
 $EndComp
 Wire Wire Line
-	8500 3100 8500 3200
+	8500 3100 8500 3150
 Wire Wire Line
 	8750 2700 8750 3150
@@
 	7900 3200 7850 3200
 $Comp
-L housing-mounts U4
+L open-automation:housing-mounts U4
 U 1 1 5978A2A6
 P 8425 4025
@@
 $EndComp
 $Comp
-L SW_PUSH FACTORY1
+L open-automation:SW_PUSH FACTORY1
 U 1 1 59C587B8
 P 3725 3975
@@
 FACTORY
 $Comp
-L GND #PWR07
+L open-automation:GND #PWR07
 U 1 1 59C59092
 P 3725 4350
@@
 	3725 4350 3725 4275
 $Comp
-L R_10k R2
+L open-automation:R_10k R2
 U 1 1 59E3E4D2
 P 3725 3475
@@
 	3725 2925 3725 2975
 Wire Wire Line
-	3725 3625 3725 3675
+	3725 3625 3725 3650
 Wire Wire Line
 	3850 3650 3725 3650
 Connection ~ 3725 3650
 $Comp
-L LED D3
+L open-automation:LED D3
 U 1 1 59E3EE41
 P 4675 3125
@@
 3V3
 $Comp
-L SW_PUSH REBOOT1
+L open-automation:SW_PUSH REBOOT1
 U 1 1 59E3EE49
 P 4675 3975
@@
 EN
 $Comp
-L GND #PWR08
+L open-automation:GND #PWR08
 U 1 1 59E3EE50
 P 4675 4350
@@
 	4675 4350 4675 4275
 $Comp
-L R_10k R3
+L open-automation:R_10k R3
 U 1 1 59E3EE58
 P 4675 3475
@@
 	4675 2925 4675 2975
 Wire Wire Line
-	4675 3625 4675 3675
+	4675 3625 4675 3650
 Wire Wire Line
 	4800 3650 4675 3650
 Connection ~ 4675 3650
 $Comp
-L LED D5
+L open-automation:LED D5
 U 1 1 59E3F1C3
 P 5450 3125
@@
 3V3
 $Comp
-L SW_PUSH PROG1
+L open-automation:SW_PUSH PROG1
 U 1 1 59E3F1CB
 P 5450 3975
@@
 PROG
 $Comp
-L GND #PWR09
+L open-automation:GND #PWR09
 U 1 1 59E3F1D2
 P 5450 4350
@@
 	5450 4350 5450 4275
 $Comp
-L R_10k R4
+L open-automation:R_10k R4
 U 1 1 59E3F1DA
 P 5450 3475
@@
 	5450 2925 5450 2975
 Wire Wire Line
-	5450 3625 5450 3675
+	5450 3625 5450 3650
 Wire Wire Line
 	5575 3650 5450 3650
@@
 Wire Wire Line
 	8050 3200 8050 3100
+Wire Wire Line
+	8500 3150 8500 3200
+Wire Wire Line
+	3725 3650 3725 3675
+Wire Wire Line
+	4675 3650 4675 3675
+Wire Wire Line
+	5450 3650 5450 3675
 $EndSCHEMATC
